Commit message: Description: Added camera links and optical links

File: orion_description/urdf/orion_cameras.urdf.xacro (robot description, xacro)
@@ -4,5 +4,5 @@
     <!--  //////////////////////// ASTRA_S CAM ///////////////////////////// -->
     <xacro:if value="${camera == 'astra_s'}">
-        <!-- Link Astra S -->
+        <!-- ....................... Astra S ............................... -->
         <link name="astra">
         <visual>
@@ -29,5 +29,4 @@
         </inertial>
         </link>
-        <!-- Joint Astra S -->
         <joint name="astra_joint" type="fixed">
             <parent link="${level_cam}"/>
@@ -35,8 +34,11 @@
             <origin xyz="0.023 0 0.0325" rpy="0 0 0"/>
         </joint>
+        <!-- ....................... Camera sensor defs ..................... -->
+        <xacro:camera_sensor x="0.02" y="0" z="0" R="${pi_2}" P="0" Y="${pi_2}"
+          parent="astra"/>
     </xacro:if>
     <!--  //////////////////////// OS30A CAM ///////////////////////////// -->
     <xacro:if value="${camera == 'os30a'}">
-        <!-- Link OS30A Support -->
+        <!-- ..................... OS30A Support .......................... -->
         <link name="os30a_sup">
         <visual>
@@ -63,5 +65,4 @@
         </inertial>
         </link>
-        <!-- Joint OS30A Support -->
         <joint name="os30a_sup_joint" type="fixed">
             <parent link="${level_cam}"/>
@@ -69,5 +70,5 @@
             <origin xyz="${0.0555 - 0.0285} 0 0.0025" rpy="0 0 0"/>
         </joint>
-        <!-- Link OS30A Support -->
+        <!-- .................... OS30A ............................. -->
         <link name="os30a">
         <visual>
@@ -94,5 +95,4 @@
         </inertial>
         </link>
-        <!-- Joint OS30A Support -->
         <joint name="os30a_joint" type="fixed">
             <parent link="os30a_sup"/>
@@ -100,8 +100,11 @@
             <origin xyz="0.025 0 0.0145" rpy="0 0 0"/>
         </joint>
+        <!-- ....................... Camera sensor defs ..................... -->
+        <xacro:camera_sensor x="0" y="0" z="0" R="${pi_2}" P="0" Y="${pi_2}"
+          parent="os30a"/>
     </xacro:if>
     <!--  //////////////////////// A010 CAM ///////////////////////////// -->
     <xacro:if value="${camera == 'a010'}">
-        <!-- Link Maixsense Support -->
+        <!-- ................... Maixsense Support ......................... -->
         <link name="maixsense_sup">
         <visual>
@@ -128,5 +131,4 @@
         </inertial>
         </link>
-        <!-- Joint Maixsense Support -->
         <joint name="maixsense_sup_joint" type="fixed">
             <parent link="${level_cam}"/>
@@ -134,5 +136,5 @@
             <origin xyz="0.038945 -0.030451 0.0125" rpy="0 0 0"/>
         </joint>
-        <!-- Link Maixsense -->
+        <!-- ................................ Maixsense ............................ -->
         <link name="maixsense">
         <visual>
@@ -159,5 +161,4 @@
         </inertial>
         </link>
-        <!-- Joint Maixsense -->
         <joint name="maixsense_joint" type="fixed">
             <parent link="maixsense_sup"/>
@@ -165,4 +166,5 @@
             <origin xyz="0 0 0.0205" rpy="0 0 0"/>
         </joint>
+        <!-- ......................... Usage of GMov ...................................  -->
         <xacro:if value="${g_mov}">
             <xacro:include filename="$(find g_mov_description)/urdf/g_mov_macros.urdf.xacro"/>
@@ -170,4 +172,7 @@
                 x="0.017825" y="0.035" z="0" joint_prefix="g_mov"/>
         </xacro:if>
+        <!-- ......................... Camera sensors links ............................ -->
+        <xacro:camera_sensor x="0.011" y="0" z="0.0025" R="${pi_2}" P="0" Y="${pi_2}"
+          parent="maixsense"/>
     </xacro:if>
 </robot>

File: orion_description/urdf/orion_macros.urdf.xacro (robot description, xacro)
@@ -884,3 +884,19 @@
             front="r" side="" x="${x - offset_x}" y="0" z="${z}"/>
     </xacro:macro>
+    <!-- ///////////////////// Cameras macros ////////////////////// -->
+    <xacro:macro name="camera_sensor" params="x y z R P Y parent">
+        <!-- ................... Camera sensors links .................. -->
+        <link name="camera_link"/>
+        <joint name="camera_joint" type="fixed">
+            <origin xyz="${x} ${y} ${z}" rpy="0 0 0"/>
+            <parent link="${parent}"/>
+            <child link="camera_link"/>
+        </joint>
+        <link name="camera_link_optical"/>
+        <joint name="optical_joint" type="fixed">
+            <origin xyz="0 0 0" rpy="${R} ${P} ${Y}"/>
+            <parent link="camera_link"/>
+            <child link="camera_link_optical"/>
+        </joint>
+    </xacro:macro>
 </robot>
