Commit message: Description: Added base platforms macros | Assets: Exploring usage of inertia calculator

File: orion_description/urdf/orion_base.urdf.xacro (robot description, xacro)
@@ -4,4 +4,16 @@
     <!-- FOR NOW IT IS EMPTY-->
     <link name="base_link"/>
-    <xacro:generic_base name="base1" parent="base_link" x="0" y="0" z="0"/>
+    <xacro:property name="level_height" value="0.08"/>
+    <xacro:property name="thickness" value="0.0025"/>
+    <xacro:com_base level="0" parent="base_link" x="0" y="0"
+        z="${level_height*0+ thickness*0}"/>
+    <xacro:com_base level="1" parent="base_link" x="0" y="0"
+        z="${level_height*1 + thickness*1}"/>
+    <xacro:com_base level="2" parent="base_link" x="0" y="0"
+        z="${level_height*2 + thickness*2}"/>
+    <xacro:com_base level="3" parent="base_link" x="0" y="0"
+        z="${level_height*3 + thickness*3}"/>
+    <xacro:half_base level="4" side="2" parent="base_link" x="0" y="0"
+        z="${level_height*4 + thickness*4}"/>
+    <xacro:spacer_10x80 front="1" side="1" level="0" x="${0.15/2 - 0.0275}" y="${0.21/2 - 0.010}" z="0"/>
 </robot>

File: orion_description/urdf/orion_macros.urdf.xacro (robot description, xacro)
@@ -91,5 +91,94 @@
         </joint>
     </xacro:macro>
-    <xacro:macro name="generic_base" params="name parent x y z">
+    <!--//////////////////// MATH AND NUMS MACROS ///////////////////////-->
+    <xacro:property name="pi_2" value="${pi / 2}"/>
+    <xacro:property name="pi_4" value="${pi / 4}"/>
+    <xacro:property name="pi_6" value="${pi / 6}"/>
+    <xacro:property name="pi_8" value="${pi / 8}"/>
+    <!--///////////////////// 10 x 80 SPACERS MACROS ///////////////////////-->
+    <!-- single custom spacer 10 x 80 mm -->
+    <xacro:macro name="spacer_10x80" params="front side level x y z">
+        <xacro:property name="muls" value="1"/>
+        <xacro:if value="${side == 2}">
+            <xacro:property name="muls" value="-1"/>
+        </xacro:if>
+        <xacro:property name="mulf" value="1"/>
+        <xacro:if value="${side == 2}">
+            <xacro:property name="mulf" value="-1"/>
+        </xacro:if>
+        <!-- Link -->
+        <link name="spacer_l${level}_${front}${side}">
+        <visual>
+            <origin xyz="0 0 0" rpy="0 0 ${muls*pi}"/>
+            <geometry>
+            <mesh filename="package://orion_description/meshes/spacer_10x80.stl"
+                scale="0.001 0.001 0.001"/>
+            </geometry>
+        </visual>
+        <collision>
+            <origin xyz="0 0 0" rpy="0 0 ${muls*pi}"/>
+            <geometry>
+            <mesh filename="package://orion_description/meshes/spacer_10x80.stl"
+                scale="0.001 0.001 0.001"/>
+            </geometry>
+        </collision>
+        <inertial>
+            <origin xyz="0 0 0"/>
+            <mass value="0.0053"/>
+            <inertia ixx="0.001" ixy="0.0" ixz="0.0"
+                    iyy="0.001" iyz="0.0"
+                    izz="0.001"/>
+        </inertial>
+        </link>
+        <joint name="spacer_l${level}_${front}${side}_joint" type="fixed">
+            <parent link="base_l${level}_s${side}"/>
+            <child link="spacer_l${level}_${front}${side}"/>
+            <origin xyz="${x*mulf} ${y*muls} ${z+0.0025}" rpy="0 0 0"/>
+        </joint>
+    </xacro:macro>
+    <!--//////////////////// BASES AND LEVELS MACROS ///////////////////////-->
+    <xacro:macro name="half_base" params="level side parent x y z">
+        <xacro:property name="mul" value="1"/>
+        <xacro:if value="${side == 2}">
+            <xacro:property name="mul" value="-1"/>
+        </xacro:if>
+        <!-- Link -->
+        <link name="base_l${level}_s${side}">
+        <visual>
+            <origin xyz="0 0 0" rpy="0 0 ${mul*pi_2}"/>
+            <geometry>
+            <mesh filename="package://orion_description/meshes/half_platform.stl"
+                scale="0.001 0.001 0.001"/>
+            </geometry>
+        </visual>
+        <collision>
+            <origin xyz="0 0 0" rpy="0 0 ${mul*pi_2}"/>
+            <geometry>
+            <mesh filename="package://orion_description/meshes/half_platform.stl"
+                scale="0.001 0.001 0.001"/>
+            </geometry>
+        </collision>
+        <inertial>
+            <origin xyz="0 0 0" rpy="0 0 ${mul*pi_2}"/>
+            <mass value="0.1"/>
+            <inertia ixx="0.001" ixy="0.0" ixz="0.0"
+                    iyy="0.001" iyz="0.0"
+                    izz="0.001"/>
+        </inertial>
+        </link>
+        <!-- Fixed Joint -->
+        <joint name="base_l${level}_s${side}_joint" type="fixed">
+        <parent link="${parent}"/>
+        <child link="base_l${level}_s${side}"/>
+        <origin xyz="${x + (mul*0.115/2)} ${y} ${z}" rpy="0 0 0"/>
+        </joint>
+    </xacro:macro>
+    <xacro:macro name="com_base" params="level parent x y z">
+        <xacro:half_base level="${level}" side="1" parent="base_link" x="${x}"
+            y="${y}" z="${z}"/>
+        <xacro:half_base level="${level}" side="2" parent="base_link" x="${x}"
+            y="${y}" z="${z}"/>
+    </xacro:macro>
+    <xacro:macro name="generic_sphere" params="name parent x y z">
     <!-- Link -->
         <link name="${name}">
@@ -97,13 +186,11 @@
             <origin xyz="0 0 0" rpy="0 0 0"/>
             <geometry>
-            <mesh filename="package://orion_description/meshes/half_platform.stl"
-                scale="0.001 0.001 0.001"/>
-            </geometry>
-        </visual>
-        <collision>
-            <origin xyz="0 0 0" rpy="0 0 0"/>
-            <geometry>
-            <mesh filename="package://orion_description/meshes/half_platform.stl"
-                scale="0.001 0.001 0.001"/>
+                <sphere radius="0.005"/>
+            </geometry>
+        </visual>
+        <collision>
+            <origin xyz="0 0 0" rpy="0 0 0"/>
+            <geometry>
+                <sphere radius="0.005"/>
             </geometry>
         </collision>

Commit message: Description: Fixing orientation of spacers_10x80

File: orion_description/urdf/orion_base.urdf.xacro (robot description, xacro)
@@ -16,4 +16,20 @@
     <xacro:half_base level="4" side="2" parent="base_link" x="0" y="0"
         z="${level_height*4 + thickness*4}"/>
-    <xacro:spacer_10x80 front="1" side="1" level="0" x="${0.15/2 - 0.0275}" y="${0.21/2 - 0.010}" z="0"/>
+    <xacro:double_spacer_10x80 front="1" level="0" x="${0.15/2 - 0.0275}"
+            y="${0.21/2 - 0.010}" z="0"/>
+    <xacro:double_spacer_10x80 front="2" level="0" x="${0.15/2 - 0.0275}"
+            y="${0.21/2 - 0.010}" z="0"/>
+    <xacro:double_spacer_10x80 front="1" level="1" x="${0.15/2 - 0.0275}"
+            y="${0.21/2 - 0.010}" z="0"/>
+    <xacro:double_spacer_10x80 front="2" level="1" x="${0.15/2 - 0.0275}"
+            y="${0.21/2 - 0.010}" z="0"/>
+    <xacro:double_spacer_10x80 front="1" level="2" x="${0.15/2 - 0.0275}"
+            y="${0.21/2 - 0.010}" z="0"/>
+    <xacro:double_spacer_10x80 front="2" level="2" x="${0.15/2 - 0.0275}"
+            y="${0.21/2 - 0.010}" z="0"/>
+    <xacro:double_spacer_10x80 front="2" level="3" x="${0.15/2 - 0.0275}"
+            y="${0.21/2 - 0.010}" z="0"/>
+    <xacro:double_spacer_10x80 front="1" level="3" x="${-0.15/2 + 0.0075}"
+            y="${0.21/2 - 0.010}" z="0"/>
+    <xacro:motor_dc front="1" side="1" x="0.005" y="0.0675" z="-0.0225"/>
 </robot>

File: orion_description/urdf/orion_macros.urdf.xacro (robot description, xacro)
@@ -99,4 +99,5 @@
     <!-- single custom spacer 10 x 80 mm -->
     <xacro:macro name="spacer_10x80" params="front side level x y z">
+        <!-- Orientation properties -->
         <xacro:property name="muls" value="1"/>
         <xacro:if value="${side == 2}">
@@ -104,18 +105,29 @@
         </xacro:if>
         <xacro:property name="mulf" value="1"/>
-        <xacro:if value="${side == 2}">
+        <xacro:if value="${front == 2}">
             <xacro:property name="mulf" value="-1"/>
         </xacro:if>
-        <!-- Link -->
+        <xacro:property name="gyro" value="${pi}"/>
+        <xacro:if value="${side == 2 and front == 1}">
+            <xacro:property name="gyro" value="${pi_2}"/>
+        </xacro:if>
+        <xacro:if value="${side == 1 and front == 2}">
+            <xacro:property name="gyro" value="${3*pi_2}"/>
+        </xacro:if>
+        <xacro:if value="${side == 2 and front == 2}">
+            <xacro:property name="gyro" value="0"/>
+        </xacro:if>
+        <!-- Link definition-->
         <link name="spacer_l${level}_${front}${side}">
         <visual>
-            <origin xyz="0 0 0" rpy="0 0 ${muls*pi}"/>
+            <origin xyz="0 0 0" rpy="0 0 ${gyro}"/>
             <geometry>
             <mesh filename="package://orion_description/meshes/spacer_10x80.stl"
                 scale="0.001 0.001 0.001"/>
             </geometry>
-        </visual>
-        <collision>
-            <origin xyz="0 0 0" rpy="0 0 ${muls*pi}"/>
+            <material name="SoftBlack"/>
+        </visual>
+        <collision>
+            <origin xyz="0 0 0" rpy="0 0 ${gyro}"/>
             <geometry>
             <mesh filename="package://orion_description/meshes/spacer_10x80.stl"
@@ -131,9 +143,16 @@
         </inertial>
         </link>
+        <!-- Joint definition -->
         <joint name="spacer_l${level}_${front}${side}_joint" type="fixed">
-            <parent link="base_l${level}_s${side}"/>
+            <parent link="base_l${level}_s${front}"/>
             <child link="spacer_l${level}_${front}${side}"/>
             <origin xyz="${x*mulf} ${y*muls} ${z+0.0025}" rpy="0 0 0"/>
         </joint>
+    </xacro:macro>
+    <xacro:macro name="double_spacer_10x80" params="front level x y z">
+        <xacro:spacer_10x80 front="${front}" side="1" level="${level}" x="${x}"
+            y="${y}" z="${z}"/>
+        <xacro:spacer_10x80 front="${front}" side="2" level="${level}" x="${x}"
+            y="${y}" z="${z}"/>
     </xacro:macro>
     <!--//////////////////// BASES AND LEVELS MACROS ///////////////////////-->
@@ -151,4 +170,5 @@
                 scale="0.001 0.001 0.001"/>
             </geometry>
+            <material name="SoftBlack"/>
         </visual>
         <collision>
@@ -208,4 +228,39 @@
         <child link="${name}"/>
         <origin xyz="${x} ${y} ${z}" rpy="0 0 0"/>
+        </joint>
+    </xacro:macro>
+    <!--  /////////////////// MOTOR DC MACROS ///////////////////////////////-->
+    <!--  Motor DC Component Kit -->
+    <xacro:macro name="motor_dc" params="front side x y z">
+        <!-- Link definition-->
+        <link name="motor_support_${front}${side}">
+        <visual>
+            <origin xyz="0 0 0" rpy="${pi} 0 0"/>
+            <geometry>
+            <mesh filename="package://orion_description/meshes/motor_mount.stl"
+                scale="0.001 0.001 0.001"/>
+            </geometry>
+            <material name="MetalGray"/>
+        </visual>
+        <collision>
+            <origin xyz="0 0 0" rpy="${pi} 0 0"/>
+            <geometry>
+            <mesh filename="package://orion_description/meshes/motor_mount.stl"
+                scale="0.001 0.001 0.001"/>
+            </geometry>
+        </collision>
+        <inertial>
+            <origin xyz="0 0 0"/>
+            <mass value="0.0053"/>
+            <inertia ixx="0.001" ixy="0.0" ixz="0.0"
+                    iyy="0.001" iyz="0.0"
+                    izz="0.001"/>
+        </inertial>
+        </link>
+        <!-- Joint definition -->
+        <joint name="motor_support_${front}${side}_joint" type="fixed">
+            <parent link="base_l0_s${front}"/>
+            <child link="motor_support_${front}${side}"/>
+            <origin xyz="${x} ${y} ${z+0.0025}" rpy="0 0 0"/>
         </joint>
     </xacro:macro>

File: orion_description/urdf/orion_materials.urdf.xacro (robot description, xacro)
@@ -16,5 +16,5 @@
     <!-- Equivalent to RGB(26, 26, 26) -->
     <material name="SoftBlack">
-        <color rgba="0.1 0.1 0.1 1.0"/>
+        <color rgba="0.2 0.2 0.2 1.0"/>
     </material>
     <!-- Equivalent to RGB(255, 255, 255) -->

Commit message: Description: Adding motor dc and its related components

File: orion_description/urdf/orion_base.urdf.xacro (robot description, xacro)
@@ -32,4 +32,7 @@
     <xacro:double_spacer_10x80 front="1" level="3" x="${-0.15/2 + 0.0075}"
             y="${0.21/2 - 0.010}" z="0"/>
-    <xacro:motor_dc front="1" side="1" x="0.005" y="0.0675" z="-0.0225"/>
+    <xacro:motor_dc front="1" side="1" x="-0.0025" y="${0.05718+0.036/2}"
+        z="-0.0225"/>
+    <xacro:motor_dc front="1" side="2" x="-0.0025" y="${0.05718+0.036/2}"
+        z="-0.0225"/>
 </robot>

File: orion_description/urdf/orion_macros.urdf.xacro (robot description, xacro)
@@ -233,8 +233,19 @@
     <!--  Motor DC Component Kit -->
     <xacro:macro name="motor_dc" params="front side x y z">
-        <!-- Link definition-->
+        <!-- Properties -->
+        <xacro:property name="mulf" value="1"/>
+        <xacro:if value="${front == 2}">
+            <xacro:property name="mulf" value="-1"/>
+        </xacro:if>
+        <xacro:property name="muls" value="1"/>
+        <xacro:property name="orin" value="0"/>
+        <xacro:if value="${side == 2}">
+            <xacro:property name="muls" value="-1"/>
+            <xacro:property name="orin" value="${pi}"/>
+        </xacro:if>
+        <!-- Link motor mount definition-->
         <link name="motor_support_${front}${side}">
         <visual>
-            <origin xyz="0 0 0" rpy="${pi} 0 0"/>
+            <origin xyz="0 0 0" rpy="${pi} 0 ${orin}"/>
             <geometry>
             <mesh filename="package://orion_description/meshes/motor_mount.stl"
@@ -244,5 +255,5 @@
         </visual>
         <collision>
-            <origin xyz="0 0 0" rpy="${pi} 0 0"/>
+            <origin xyz="0 0 0" rpy="${muls*pi} 0 0"/>
             <geometry>
             <mesh filename="package://orion_description/meshes/motor_mount.stl"
@@ -258,9 +269,134 @@
         </inertial>
         </link>
-        <!-- Joint definition -->
+        <!-- Joint motor mount definition-->
         <joint name="motor_support_${front}${side}_joint" type="fixed">
             <parent link="base_l0_s${front}"/>
             <child link="motor_support_${front}${side}"/>
-            <origin xyz="${x} ${y} ${z+0.0025}" rpy="0 0 0"/>
+            <origin xyz="${x*mulf} ${y*muls} ${z+0.0025}" rpy="0 0 0"/>
+        </joint>
+        <!-- Link motor dc definition-->
+        <link name="motor_dc_${front}${side}">
+        <visual>
+            <origin xyz="0 0 0" rpy="${-pi_2*muls} 0 0"/>
+            <geometry>
+            <mesh filename="package://orion_description/meshes/motor_dc.stl"
+                scale="0.001 0.001 0.001"/>
+            </geometry>
+            <material name="MetalGray"/>
+        </visual>
+        <collision>
+            <origin xyz="0 0 0" rpy="${-pi_2*muls} 0 0"/>
+            <geometry>
+            <mesh filename="package://orion_description/meshes/motor_dc.stl"
+                scale="0.001 0.001 0.001"/>
+            </geometry>
+        </collision>
+        <inertial>
+            <origin xyz="0 0 0"/>
+            <mass value="0.0053"/>
+            <inertia ixx="0.001" ixy="0.0" ixz="0.0"
+                    iyy="0.001" iyz="0.0"
+                    izz="0.001"/>
+        </inertial>
+        </link>
+        <!-- Joint motor dc definition-->
+        <joint name="motor_dc_${front}${side}_joint" type="fixed">
+            <parent link="motor_support_${front}${side}"/>
+            <child link="motor_dc_${front}${side}"/>
+            <origin xyz="0 ${-0.05625*muls} 0" rpy="0 0 0"/>
+        </joint>
+        <!-- Link coupling definition-->
+        <link name="coupling_${front}${side}">
+        <visual>
+            <origin xyz="0 0 0" rpy="0 0 ${pi_6*muls}"/>
+            <geometry>
+            <mesh filename="package://orion_description/meshes/coupling.stl"
+                scale="0.001 0.001 0.001"/>
+            </geometry>
+            <material name="Brass"/>
+        </visual>
+        <collision>
+            <origin xyz="0 0 0" rpy="0 0 ${pi_6*muls}"/>
+            <geometry>
+            <mesh filename="package://orion_description/meshes/coupling.stl"
+                scale="0.001 0.001 0.001"/>
+            </geometry>
+        </collision>
+        <inertial>
+            <origin xyz="0 0 0"/>
+            <mass value="0.0053"/>
+            <inertia ixx="0.001" ixy="0.0" ixz="0.0"
+                    iyy="0.001" iyz="0.0"
+                    izz="0.001"/>
+        </inertial>
+        </link>
+        <!-- Joint coupling definition-->
+        <joint name="coupling_${front}${side}_joint" type="continuous">
+            <axis xyz="0.0 0.0 1.0"/>
+            <parent link="motor_support_${front}${side}"/>
+            <child link="coupling_${front}${side}"/>
+            <origin xyz="0 ${(0.01120 + 0.000325)*muls} 0" rpy="${-pi_2*muls+orin} 0 0"/>
+        </joint>
+        <!-- Ring coupling definition-->
+        <link name="ring_${front}${side}">
+        <visual>
+            <origin xyz="0 0 0" rpy="0 ${-pi_2*muls} 0"/>
+            <geometry>
+            <mesh filename="package://orion_description/meshes/ring.stl"
+                scale="0.001 0.001 0.001"/>
+            </geometry>
+            <material name="ArduinoBlue"/>
+        </visual>
+        <collision>
+            <origin xyz="0 0 0" rpy="0 ${-pi_2*muls} 0"/>
+            <geometry>
+            <mesh filename="package://orion_description/meshes/ring.stl"
+                scale="0.001 0.001 0.001"/>
+            </geometry>
+        </collision>
+        <inertial>
+            <origin xyz="0 0 0"/>
+            <mass value="0.0053"/>
+            <inertia ixx="0.001" ixy="0.0" ixz="0.0"
+                    iyy="0.001" iyz="0.0"
+                    izz="0.001"/>
+        </inertial>
+        </link>
+        <!-- Ring coupling definition-->
+        <joint name="ring_${front}${side}_joint" type="fixed">
+            <parent link="coupling_${front}${side}"/>
+            <child link="ring_${front}${side}"/>
+            <origin xyz="0 0 ${0.0068*muls}" rpy="0 0 0"/>
+        </joint>
+        <!-- Link neumatic definition-->
+        <link name="neumatic_${front}${side}">
+        <visual>
+            <origin xyz="0 0 0" rpy="0 ${pi_2*muls} 0"/>
+            <geometry>
+            <mesh filename="package://orion_description/meshes/neumatic.stl"
+                scale="0.001 0.001 0.001"/>
+            </geometry>
+            <material name="SoftBlack"/>
+        </visual>
+        <collision>
+            <origin xyz="0 0 0" rpy="0 ${pi_2*muls} 0"/>
+            <geometry>
+            <mesh filename="package://orion_description/meshes/neumatic.stl"
+                scale="0.001 0.001 0.001"/>
+            </geometry>
+        </collision>
+        <inertial>
+            <origin xyz="0 0 0"/>
+            <mass value="0.0053"/>
+            <inertia ixx="0.001" ixy="0.0" ixz="0.0"
+                    iyy="0.001" iyz="0.0"
+                    izz="0.001"/>
+        </inertial>
+        </link>
+        <!-- Joint neumatic definition-->
+        <joint name="neumatic_${front}${side}_joint" type="fixed">
+            <parent link="ring_${front}${side}"/>
+            <child link="neumatic_${front}${side}"/>
+            <origin xyz="0 0 0" rpy="0 0 0"/>
         </joint>
     </xacro:macro>
