Commit message: Description: Added caster wheel and first hex spacers

File: orion_description/urdf/orion_base.urdf.xacro (robot description, xacro)
@@ -2,8 +2,10 @@
 <robot xmlns:xacro="http://www.ros.org/wiki/xacro">
     <!-- This xacro file aims for adding the mobile platform to the robot-->
-    <!-- FOR NOW IT IS EMPTY-->
+    <!-- ////////////////////////// BASE LINK //////////////////////////////-->
     <link name="base_link"/>
+    <!-- ///////////////////////// PROPERTIES //////////////////////////////-->
     <xacro:property name="level_height" value="0.08"/>
     <xacro:property name="thickness" value="0.0025"/>
+    <!-- /////////////////////////// LEVELS ///////////////////////////////-->
     <xacro:com_base level="0" parent="base_link" x="0" y="0"
         z="${level_height*0+ thickness*0}"/>
@@ -16,4 +18,5 @@
     <xacro:half_base level="4" side="2" parent="base_link" x="0" y="0"
         z="${level_height*4 + thickness*4}"/>
+    <!-- /////////////////////// LEVEL's SPACERS//////////////////////////-->
     <xacro:double_spacer_10x80 front="1" level="0" x="${0.15/2 - 0.0275}"
             y="${0.21/2 - 0.010}" z="0"/>
@@ -32,7 +35,47 @@
     <xacro:double_spacer_10x80 front="1" level="3" x="${-0.15/2 + 0.0075}"
             y="${0.21/2 - 0.010}" z="0"/>
+    <!-- //////////////////////// MOTORS DC ////////////////////////////-->
     <xacro:motor_dc front="1" side="1" x="-0.0025" y="${0.05718+0.036/2}"
         z="-0.0225"/>
     <xacro:motor_dc front="1" side="2" x="-0.0025" y="${0.05718+0.036/2}"
         z="-0.0225"/>
+    <!-- /////////////////////// CASTER WHEEL //////////////////////////-->
+    <xacro:x4xspacer_m4x17 id="hm4x17" element="caster" parent="base_l0_s2"
+        offset_x="0.012" offset_y="0.015" x="-0.022" y="0"
+        z="${-0.001 - 0.017}"/>
+    <xacro:caster_wheel parent="base_l0_s2" front="2" x="-0.022" y="0"
+        z="${-0.002 - 0.017}"/>
+    <!-- //////////////// FIRST FLOOR COMPONENTS ///////////////////// -->
+    <xacro:x6xspacer_m3x10 id="hm3x10" element="bathol" parent="base_l0_s1"
+        offset_x="${0.0855/2}" offset_y="${0.127/2}" x="0.005" y="0" z="0.0025"/>
+    <link name="bat_platform">
+        <visual>
+            <origin xyz="0 0 0" rpy="0 0 ${pi_2}"/>
+            <geometry>
+            <mesh filename="package://orion_description/meshes/bathold_support.stl"
+                scale="0.001 0.001 0.001"/>
+            </geometry>
+            <material name="PureWhite"/>
+        </visual>
+        <collision>
+            <origin xyz="0 0 0" rpy="0 0 ${pi_2}"/>
+            <geometry>
+            <mesh filename="package://orion_description/meshes/bathold_support.stl"
+                scale="0.001 0.001 0.001"/>
+            </geometry>
+        </collision>
+        <inertial>
+            <origin xyz="0 0 0" rpy="0 0 ${pi_2}"/>
+            <mass value="0.1"/>
+            <inertia ixx="0.001" ixy="0.0" ixz="0.0"
+                    iyy="0.001" iyz="0.0"
+                    izz="0.001"/>
+        </inertial>
+        </link>
+        <!-- Fixed Joint -->
+        <joint name="bat_platform_joint" type="fixed">
+            <parent link="base_l0_s1"/>
+            <child link="bat_platform"/>
+            <origin xyz="0.005 0 0.0125" rpy="0 0 0"/>
+        </joint>
 </robot>

File: orion_description/urdf/orion_macros.urdf.xacro (robot description, xacro)
@@ -170,5 +170,5 @@
                 scale="0.001 0.001 0.001"/>
             </geometry>
-            <material name="SoftBlack"/>
+            <material name="PureWhite"/>
         </visual>
         <collision>
@@ -189,7 +189,7 @@
         <!-- Fixed Joint -->
         <joint name="base_l${level}_s${side}_joint" type="fixed">
-        <parent link="${parent}"/>
-        <child link="base_l${level}_s${side}"/>
-        <origin xyz="${x + (mul*0.115/2)} ${y} ${z}" rpy="0 0 0"/>
+            <parent link="${parent}"/>
+            <child link="base_l${level}_s${side}"/>
+            <origin xyz="${x + (mul*0.115/2)} ${y} ${z}" rpy="0 0 0"/>
         </joint>
     </xacro:macro>
@@ -401,16 +401,115 @@
         </joint>
     </xacro:macro>
+    <!--////////////////////////// CASTER WHEEL ////////////////////////////-->
+    <xacro:macro name="caster_wheel" params="parent front x y z">
+        <!-- Link caster base definition-->
+        <link name="caster_base_${front}">
+        <visual>
+            <origin xyz="0 0 0" rpy="${pi} 0 ${pi_2}"/>
+            <geometry>
+            <mesh filename="package://orion_description/meshes/caster_base.stl"
+                scale="0.001 0.001 0.001"/>
+            </geometry>
+            <material name="MetalGray"/>
+        </visual>
+        <collision>
+            <origin xyz="0 0 0" rpy="${pi} 0 ${pi_2}"/>
+            <geometry>
+            <mesh filename="package://orion_description/meshes/caster_base.stl"
+                scale="0.001 0.001 0.001"/>
+            </geometry>
+        </collision>
+        <inertial>
+            <origin xyz="0 0 0"/>
+            <mass value="0.0053"/>
+            <inertia ixx="0.001" ixy="0.0" ixz="0.0"
+                    iyy="0.001" iyz="0.0"
+                    izz="0.001"/>
+        </inertial>
+        </link>
+        <!-- Joint caster base definition-->
+        <joint name="caster_base_${front}_joint" type="fixed">
+            <parent link="${parent}"/>
+            <child link="caster_base_${front}"/>
+            <origin xyz="${x} ${y} ${z}" rpy="0 0 0"/>
+        </joint>
+        <!-- Link caster middle definition-->
+        <link name="caster_middle_${front}">
+        <visual>
+            <origin xyz="0 0 0" rpy="0 0 ${-pi_2}"/>
+            <geometry>
+            <mesh filename="package://orion_description/meshes/caster_middle.stl"
+                scale="0.001 0.001 0.001"/>
+            </geometry>
+            <material name="MetalGray"/>
+        </visual>
+        <collision>
+            <origin xyz="0 0 0" rpy="0 0 ${-pi_2}"/>
+            <geometry>
+            <mesh filename="package://orion_description/meshes/caster_middle.stl"
+                scale="0.001 0.001 0.001"/>
+            </geometry>
+        </collision>
+        <inertial>
+            <origin xyz="0 0 0"/>
+            <mass value="0.0053"/>
+            <inertia ixx="0.001" ixy="0.0" ixz="0.0"
+                    iyy="0.001" iyz="0.0"
+                    izz="0.001"/>
+        </inertial>
+        </link>
+        <!-- Joint caster middle definition-->
+        <joint name="caster_middle_${front}_joint" type="continuous">
+            <axis xyz="0.0 0.0 1.0"/>
+            <parent link="caster_base_${front}"/>
+            <child link="caster_middle_${front}"/>
+            <origin xyz="0 0 -0.002" rpy="${pi} 0 0"/>
+        </joint>
+        <!-- Link caster wheel definition-->
+        <link name="caster_wheel_${front}">
+        <visual>
+            <origin xyz="0 0 0" rpy="${pi_2} 0 0"/>
+            <geometry>
+            <mesh filename="package://orion_description/meshes/caster_wheel.stl"
+                scale="0.001 0.001 0.001"/>
+            </geometry>
+            <material name="SoftBlack"/>
+        </visual>
+        <collision>
+            <origin xyz="0 0 0" rpy="${pi_2} 0 0"/>
+            <geometry>
+            <mesh filename="package://orion_description/meshes/caster_wheel.stl"
+                scale="0.001 0.001 0.001"/>
+            </geometry>
+        </collision>
+        <inertial>
+            <origin xyz="0 0 0"/>
+            <mass value="0.0053"/>
+            <inertia ixx="0.001" ixy="0.0" ixz="0.0"
+                    iyy="0.001" iyz="0.0"
+                    izz="0.001"/>
+        </inertial>
+        </link>
+        <!-- Joint caster wheel definition-->
+        <joint name="caster_wheel_${front}_joint" type="continuous">
+            <axis xyz="0.0 0.0 1.0"/>
+            <parent link="caster_middle_${front}"/>
+            <child link="caster_wheel_${front}"/>
+            <origin xyz="-0.0108 0 0.0185" rpy="${pi/2} 0 0"/>
+        </joint>
+    </xacro:macro>
     <!--///////////////////// M3 x 10 SPACERS MACROS ///////////////////////-->
     <!-- Hex spacer M3 x 10 macro -->
     <xacro:macro name="spacer_m3x10"
-            params="name parent element front side x y z">
+            params="id parent element front side x y z">
         <!-- Link -->
-        <link name="${name}_${element}_${front}${side}">
+        <link name="${id}_${element}_${front}${side}">
         <visual>
             <origin xyz="0 0 0" rpy="0 0 0"/>
             <geometry>
             <mesh filename="package://orion_description/meshes/spacer_m3x10.stl"
-                scale="1 1 1"/>
-            </geometry>
+                scale="0.001 0.001 0.001"/>
+            </geometry>
+            <material name="Brass"/>
         </visual>
         <collision>
@@ -418,23 +517,23 @@
             <geometry>
             <mesh filename="package://orion_description/meshes/spacer_m3x10.stl"
-                scale="1 1 1"/>
-            </geometry>
-        </collision>
-        <inertial>
-            <origin xyz="0 0 0"/>
-            <mass value="0.0053"/>
-            <inertia ixx="0.001" ixy="0.0" ixz="0.0"
-                    iyy="0.001" iyz="0.0"
-                    izz="0.001"/>
-        </inertial>
-        </link>
-        <joint name="${name}_${element}_${front}${side}_joint" type="fixed">
-        <parent link="${parent}"/>
-        <child link="${name}"/>
-        <origin xyz="${x} ${y} ${z}" rpy="0 0 0"/>
+                scale="0.001 0.001 0.001"/>
+            </geometry>
+        </collision>
+        <inertial>
+            <origin xyz="0 0 0"/>
+            <mass value="0.0053"/>
+            <inertia ixx="0.001" ixy="0.0" ixz="0.0"
+                    iyy="0.001" iyz="0.0"
+                    izz="0.001"/>
+        </inertial>
+        </link>
+        <joint name="${id}_${element}_${front}${side}_joint" type="fixed">
+            <parent link="${parent}"/>
+            <child link="${id}_${element}_${front}${side}"/>
+            <origin xyz="${x} ${y} ${z}" rpy="0 0 0"/>
         </joint>
     </xacro:macro>
     <!-- 2 symetric hex spacers by considering y axis -->
-    <xacro:macro name="2xspacer_m3x10"
+    <xacro:macro name="x2xspacer_m3x10"
                 params="name element parent offset_y x y z">
         <xacro:spacer_m3x10 name="${name}" parent="${parent}" element="${element}"
@@ -444,14 +543,85 @@
     </xacro:macro>
     <!-- 4 symetric hex spacers by considering x/y axis -->
-    <xacro:macro name="4xspacer_m3x10"
-                params="name element parent offset_x offset_y x y z">
-        <xacro:spacer_m3x10 name="${name}" parent="${parent}" element="${element}"
+    <xacro:macro name="x4xspacer_m3x10"
+                params="id element parent offset_x offset_y x y z">
+        <xacro:spacer_m3x10 id="${id}" parent="${parent}" element="${element}"
             front="f" side="r" x="${x + offset_x}" y="${y - offset_y}" z="${z}"/>
-        <xacro:spacer_m3x10 name="${name}" parent="${parent}" element="${element}"
+        <xacro:spacer_m3x10 id="${id}" parent="${parent}" element="${element}"
             front="f" side="l" x="${x + offset_x}" y="${y + offset_y}" z="${z}"/>
-        <xacro:spacer_m3x10 name="${name}" parent="${parent}" element="${element}"
+        <xacro:spacer_m3x10 id="${id}" parent="${parent}" element="${element}"
             front="r" side="r" x="${x - offset_x}" y="${y + offset_y}" z="${z}"/>
-        <xacro:spacer_m3x10 name="${name}" parent="${parent}" element="${element}"
+        <xacro:spacer_m3x10 id="${id}" parent="${parent}" element="${element}"
             front="r" side="l" x="${x - offset_x}" y="${y - offset_y}" z="${z}"/>
     </xacro:macro>
+    <!-- 6 symetric hex spacers by considering x/y axis -->
+    <xacro:macro name="x6xspacer_m3x10"
+                params="id element parent offset_x offset_y x y z">
+        <xacro:spacer_m3x10 id="${id}" parent="${parent}" element="${element}"
+            front="f" side="r" x="${x + offset_x}" y="${y - offset_y}" z="${z}"/>
+        <xacro:spacer_m3x10 id="${id}" parent="${parent}" element="${element}"
+            front="f" side="l" x="${x + offset_x}" y="${y + offset_y}" z="${z}"/>
+        <xacro:spacer_m3x10 id="${id}" parent="${parent}" element="${element}"
+            front="r" side="r" x="${x - offset_x}" y="${y + offset_y}" z="${z}"/>
+        <xacro:spacer_m3x10 id="${id}" parent="${parent}" element="${element}"
+            front="r" side="l" x="${x - offset_x}" y="${y - offset_y}" z="${z}"/>
+        <xacro:spacer_m3x10 id="${id}" parent="${parent}" element="${element}"
+            front="f" side="" x="${x + offset_x}" y="0" z="${z}"/>
+        <xacro:spacer_m3x10 id="${id}" parent="${parent}" element="${element}"
+            front="r" side="" x="${x - offset_x}" y="0" z="${z}"/>
+    </xacro:macro>
+    <!--///////////////////// M4 x 17 SPACERS MACROS ///////////////////////-->
+    <!-- Hex spacer M4 x 17 macro -->
+    <xacro:macro name="spacer_m4x17"
+            params="id parent element front side x y z">
+        <!-- Link -->
+        <link name="${id}_${element}_${front}${side}">
+        <visual>
+            <origin xyz="0 0 0" rpy="0 0 0"/>
+            <geometry>
+            <mesh filename="package://orion_description/meshes/spacer_m4x17.stl"
+                scale="0.001 0.001 0.001"/>
+            </geometry>
+            <material name="Brass"/>
+        </visual>
+        <collision>
+            <origin xyz="0 0 0" rpy="0 0 0"/>
+            <geometry>
+            <mesh filename="package://orion_description/meshes/spacer_m4x17.stl"
+                scale="0.001 0.001 0.001"/>
+            </geometry>
+        </collision>
+        <inertial>
+            <origin xyz="0 0 0"/>
+            <mass value="0.0053"/>
+            <inertia ixx="0.001" ixy="0.0" ixz="0.0"
+                    iyy="0.001" iyz="0.0"
+                    izz="0.001"/>
+        </inertial>
+        </link>
+        <joint name="${id}_${element}_${front}${side}_joint" type="fixed">
+        <parent link="${parent}"/>
+        <child link="${id}_${element}_${front}${side}"/>
+        <origin xyz="${x} ${y} ${z}" rpy="0 0 0"/>
+        </joint>
+    </xacro:macro>
+    <!-- 2 symetric hex spacers by considering y axis -->
+    <xacro:macro name="x2xspacer_m4x17"
+                params="id element parent offset_y x y z">
+        <xacro:spacer_m4x17 id="${id}" parent="${parent}" element="${element}"
+            front="" side="r" x="${x}" y="${y - offset_y}" z="${z}"/>
+        <xacro:spacer_m4x17 id="${id}" parent="${parent}" element="${element}"
+            front="" side="l" x="${x}" y="${y + offset_y}" z="${z}"/>
+    </xacro:macro>
+    <!-- 4 symetric hex spacers by considering x/y axis -->
+    <xacro:macro name="x4xspacer_m4x17"
+                params="id element parent offset_x offset_y x y z">
+        <xacro:spacer_m4x17 id="${id}" parent="${parent}" element="${element}"
+            front="f" side="r" x="${x + offset_x}" y="${y - offset_y}" z="${z}"/>
+        <xacro:spacer_m4x17 id="${id}" parent="${parent}" element="${element}"
+            front="f" side="l" x="${x + offset_x}" y="${y + offset_y}" z="${z}"/>
+        <xacro:spacer_m4x17 id="${id}" parent="${parent}" element="${element}"
+            front="r" side="r" x="${x - offset_x}" y="${y + offset_y}" z="${z}"/>
+        <xacro:spacer_m4x17 id="${id}" parent="${parent}" element="${element}"
+            front="r" side="l" x="${x - offset_x}" y="${y - offset_y}" z="${z}"/>
+    </xacro:macro>
 </robot>
