Commit message: Description: Added Batteries stacks, servo supports, driver and reg

File: orion_description/urdf/orion_base.urdf.xacro (robot description, xacro)
@@ -47,35 +47,207 @@
         z="${-0.002 - 0.017}"/>
     <!-- //////////////// FIRST FLOOR COMPONENTS ///////////////////// -->
+    <!-- Hex spacers for Battery Support -->
     <xacro:x6xspacer_m3x10 id="hm3x10" element="bathol" parent="base_l0_s1"
         offset_x="${0.0855/2}" offset_y="${0.127/2}" x="0.005" y="0" z="0.0025"/>
+    <!-- Link Battery Support-->
     <link name="bat_platform">
-        <visual>
-            <origin xyz="0 0 0" rpy="0 0 ${pi_2}"/>
-            <geometry>
-            <mesh filename="package://orion_description/meshes/bathold_support.stl"
-                scale="0.001 0.001 0.001"/>
-            </geometry>
-            <material name="PureWhite"/>
-        </visual>
-        <collision>
-            <origin xyz="0 0 0" rpy="0 0 ${pi_2}"/>
-            <geometry>
-            <mesh filename="package://orion_description/meshes/bathold_support.stl"
-                scale="0.001 0.001 0.001"/>
-            </geometry>
-        </collision>
-        <inertial>
-            <origin xyz="0 0 0" rpy="0 0 ${pi_2}"/>
-            <mass value="0.1"/>
-            <inertia ixx="0.001" ixy="0.0" ixz="0.0"
-                    iyy="0.001" iyz="0.0"
-                    izz="0.001"/>
-        </inertial>
-        </link>
-        <!-- Fixed Joint -->
-        <joint name="bat_platform_joint" type="fixed">
-            <parent link="base_l0_s1"/>
-            <child link="bat_platform"/>
-            <origin xyz="0.005 0 0.0125" rpy="0 0 0"/>
-        </joint>
+    <visual>
+        <origin xyz="0 0 0" rpy="0 0 ${pi_2}"/>
+        <geometry>
+        <mesh filename="package://orion_description/meshes/bathold_support.stl"
+            scale="0.001 0.001 0.001"/>
+        </geometry>
+        <material name="PureWhite"/>
+    </visual>
+    <collision>
+        <origin xyz="0 0 0" rpy="0 0 ${pi_2}"/>
+        <geometry>
+        <mesh filename="package://orion_description/meshes/bathold_support.stl"
+            scale="0.001 0.001 0.001"/>
+        </geometry>
+    </collision>
+    <inertial>
+        <origin xyz="0 0 0" rpy="0 0 ${pi_2}"/>
+        <mass value="0.1"/>
+        <inertia ixx="0.001" ixy="0.0" ixz="0.0"
+                iyy="0.001" iyz="0.0"
+                izz="0.001"/>
+    </inertial>
+    </link>
+    <!-- Joint Battery Support -->
+    <joint name="bat_platform_joint" type="fixed">
+        <parent link="base_l0_s1"/>
+        <child link="bat_platform"/>
+        <origin xyz="0.005 0 0.0125" rpy="0 0 0"/>
+    </joint>
+    <!-- Battery Stacks -->
+    <xacro:stack_bat parent="bat_platform" num="1" x="0" y="-0.023" z="0"/>
+    <xacro:stack_bat parent="bat_platform" num="2" x="0" y="${0.023+0.02}"
+        z="0"/>
+    <!-- Hex spacers for Motor Driver-->
+    <xacro:x4xspacer_m3x10 id="hm3x10" element="driver" parent="base_l0_s2"
+        offset_x="${0.03702/2}" offset_y="${-0.0368/2}" x="-0.023453"
+        y="0.031351" z="0.0025"/>
+    <!-- Link Motor Driver-->
+    <link name="driver_platform">
+    <visual>
+        <origin xyz="0 0 0" rpy="0 0 0"/>
+        <geometry>
+        <mesh filename="package://orion_description/meshes/driver.stl"
+            scale="0.001 0.001 0.001"/>
+        </geometry>
+        <material name="DriverRed"/>
+    </visual>
+    <collision>
+        <origin xyz="0 0 0" rpy="0 0 0"/>
+        <geometry>
+        <mesh filename="package://orion_description/meshes/driver.stl"
+            scale="0.001 0.001 0.001"/>
+        </geometry>
+    </collision>
+    <inertial>
+        <origin xyz="0 0 0" rpy="0 0 0"/>
+        <mass value="0.1"/>
+        <inertia ixx="0.001" ixy="0.0" ixz="0.0"
+                iyy="0.001" iyz="0.0"
+                izz="0.001"/>
+    </inertial>
+    </link>
+    <!-- Joint Motor Driver -->
+    <joint name="driver_platform" type="fixed">
+        <parent link="base_l0_s2"/>
+        <child link="driver_platform"/>
+        <origin xyz="-0.023453 0.031351 0.0125" rpy="0 0 0"/>
+    </joint>
+    <!-- Link Regulator Support-->
+    <link name="reg_support">
+    <visual>
+        <origin xyz="0 0 0" rpy="0 0 ${-pi_2}"/>
+        <geometry>
+        <mesh filename="package://orion_description/meshes/regulator_sup.stl"
+            scale="0.001 0.001 0.001"/>
+        </geometry>
+        <material name="SoftBlack"/>
+    </visual>
+    <collision>
+        <origin xyz="0 0 0" rpy="0 0 ${-pi_2}"/>
+        <geometry>
+        <mesh filename="package://orion_description/meshes/regulator_sup.stl"
+            scale="0.001 0.001 0.001"/>
+        </geometry>
+    </collision>
+    <inertial>
+        <origin xyz="0 0 0" rpy="0 0 ${-pi_2}"/>
+        <mass value="0.1"/>
+        <inertia ixx="0.001" ixy="0.0" ixz="0.0"
+                iyy="0.001" iyz="0.0"
+                izz="0.001"/>
+    </inertial>
+    </link>
+    <!-- Joint Regulator Support -->
+    <joint name="reg_support_joint" type="fixed">
+        <parent link="base_l0_s2"/>
+        <child link="reg_support"/>
+        <origin xyz="-0.036 -0.0275 0.0025" rpy="0 0 0"/>
+    </joint>
+    <!-- Link Regulator Support-->
+    <link name="regulator">
+    <visual>
+        <origin xyz="0 0 0" rpy="${pi_2} 0 ${-pi_2}"/>
+        <geometry>
+        <mesh filename="package://orion_description/meshes/regulator.stl"
+            scale="0.001 0.001 0.001"/>
+        </geometry>
+        <material name="ArduinoBlue"/>
+    </visual>
+    <collision>
+        <origin xyz="0 0 0" rpy="${pi_2} 0 ${-pi_2}"/>
+        <geometry>
+        <mesh filename="package://orion_description/meshes/regulator.stl"
+            scale="0.001 0.001 0.001"/>
+        </geometry>
+    </collision>
+    <inertial>
+        <origin xyz="0 0 0" rpy="${pi_2} 0 ${-pi_2}"/>
+        <mass value="0.1"/>
+        <inertia ixx="0.001" ixy="0.0" ixz="0.0"
+                iyy="0.001" iyz="0.0"
+                izz="0.001"/>
+    </inertial>
+    </link>
+    <!-- Joint Regulator -->
+    <joint name="reg_joint" type="fixed">
+        <parent link="reg_support"/>
+        <child link="regulator"/>
+        <origin xyz="-0.0025 0 ${0.06/2}" rpy="0 0 0"/>
+    </joint>
+    <xacro:servo_mounted parent="base_l1_s2" side="1" x="0.00275" y="0.0765"
+        z="-0.026"/>
+    <xacro:servo_mounted parent="base_l1_s2" side="2" x="0.00275" y="0.0765"
+        z="-0.026"/>
+    <!-- ///////////////// SECOND FLOOR COMPONENTS /////////////////////// -->
+    <xacro:x4xspacer_m3x10 id="hm3x10" element="espadapter" parent="base_l1_s1"
+        offset_x="${0.0577/2}" offset_y="${0.0607/2}" x="0" y="0" z="-0.01"/>
+    <!-- Link Esp32 Adapter -->
+    <link name="esp32_adapter">
+    <visual>
+        <origin xyz="0 0 0" rpy="${pi} 0 0"/>
+        <geometry>
+        <mesh filename="package://orion_description/meshes/esp32_adp.stl"
+            scale="0.001 0.001 0.001"/>
+        </geometry>
+        <material name="RaspberryGreen"/>
+    </visual>
+    <collision>
+        <origin xyz="0 0 0" rpy="${pi} 0 0"/>
+        <geometry>
+        <mesh filename="package://orion_description/meshes/esp32_adp.stl"
+            scale="0.001 0.001 0.001"/>
+        </geometry>
+    </collision>
+    <inertial>
+        <origin xyz="0 0 0" rpy="${pi} 0 0"/>
+        <mass value="0.1"/>
+        <inertia ixx="0.001" ixy="0.0" ixz="0.0"
+                iyy="0.001" iyz="0.0"
+                izz="0.001"/>
+    </inertial>
+    </link>
+    <!-- Joint Esp32 Adapter -->
+    <joint name="esp32_adapter_joint" type="fixed">
+        <parent link="base_l1_s1"/>
+        <child link="esp32_adapter"/>
+        <origin xyz="0 0 -0.01" rpy="0 0 0"/>
+    </joint>
+    <!-- Link Esp32 -->
+    <link name="esp32">
+    <visual>
+        <origin xyz="0 0 0" rpy="${pi} 0 ${-pi_2}"/>
+        <geometry>
+        <mesh filename="package://orion_description/meshes/esp32.stl"
+            scale="0.001 0.001 0.001"/>
+        </geometry>
+        <material name="SoftBlack"/>
+    </visual>
+    <collision>
+        <origin xyz="0 0 0" rpy="${pi} 0 ${-pi_2}"/>
+        <geometry>
+        <mesh filename="package://orion_description/meshes/esp32.stl"
+            scale="0.001 0.001 0.001"/>
+        </geometry>
+    </collision>
+    <inertial>
+        <origin xyz="0 0 0" rpy="${pi} 0 ${-pi_2}"/>
+        <mass value="0.1"/>
+        <inertia ixx="0.001" ixy="0.0" ixz="0.0"
+                iyy="0.001" iyz="0.0"
+                izz="0.001"/>
+    </inertial>
+    </link>
+    <!-- Joint Esp32 -->
+    <joint name="esp32_joint" type="fixed">
+        <parent link="esp32_adapter"/>
+        <child link="esp32"/>
+        <origin xyz="0.002 0 -0.01" rpy="0 0 0"/>
+    </joint>
 </robot>

File: orion_description/urdf/orion_macros.urdf.xacro (robot description, xacro)
@@ -255,5 +255,5 @@
         </visual>
         <collision>
-            <origin xyz="0 0 0" rpy="${muls*pi} 0 0"/>
+            <origin xyz="0 0 0" rpy="${pi} 0 ${orin}"/>
             <geometry>
             <mesh filename="package://orion_description/meshes/motor_mount.stl"
@@ -309,5 +309,5 @@
         <link name="coupling_${front}${side}">
         <visual>
-            <origin xyz="0 0 0" rpy="0 0 ${pi_6*muls}"/>
+            <origin xyz="0 0 0" rpy="${orin} 0 ${pi_6*muls}"/>
             <geometry>
             <mesh filename="package://orion_description/meshes/coupling.stl"
@@ -317,5 +317,5 @@
         </visual>
         <collision>
-            <origin xyz="0 0 0" rpy="0 0 ${pi_6*muls}"/>
+            <origin xyz="0 0 0" rpy="${orin} 0 ${pi_6*muls}"/>
             <geometry>
             <mesh filename="package://orion_description/meshes/coupling.stl"
@@ -338,5 +338,5 @@
             <origin xyz="0 ${(0.01120 + 0.000325)*muls} 0" rpy="${-pi_2*muls+orin} 0 0"/>
         </joint>
-        <!-- Ring coupling definition-->
+        <!-- LInk Ring  definition-->
         <link name="ring_${front}${side}">
         <visual>
@@ -363,5 +363,5 @@
         </inertial>
         </link>
-        <!-- Ring coupling definition-->
+        <!-- Joint ring definition-->
         <joint name="ring_${front}${side}_joint" type="fixed">
             <parent link="coupling_${front}${side}"/>
@@ -497,4 +497,129 @@
             <child link="caster_wheel_${front}"/>
             <origin xyz="-0.0108 0 0.0185" rpy="${pi/2} 0 0"/>
+        </joint>
+    </xacro:macro>
+    <!-- ///////////////////// BATTERIES MACROS ////////////////////////////-->
+    <!-- B18650 Macro-->
+    <xacro:macro name="b18650" params="parent element num x y z">
+        <xacro:property name="inv" value="1"/>
+        <xacro:property name="rot" value="${pi_2}"/>
+        <xacro:if value="${num == 2}">
+            <xacro:property name="rot" value="${pi_2*3}"/>
+            <xacro:property name="inv" value="-1"/>
+        </xacro:if>
+        <xacro:if value="${num == 3}">
+            <xacro:property name="rot" value="${pi_2*5}"/>
+        </xacro:if>
+        <!-- Link -->
+        <link name="${element}_${num}">
+        <visual>
+            <origin xyz="0 0 0" rpy="0 ${rot} 0"/>
+            <geometry>
+            <mesh filename="package://orion_description/meshes/b18650.stl"
+                scale="0.001 0.001 0.001"/>
+            </geometry>
+            <material name="DriverRed"/>
+        </visual>
+        <collision>
+            <origin xyz="0 0 0" rpy="0 ${rot} 0"/>
+            <geometry>
+            <mesh filename="package://orion_description/meshes/b18650.stl"
+                scale="0.001 0.001 0.001"/>
+            </geometry>
+        </collision>
+        <inertial>
+            <origin xyz="0 0 0"/>
+            <mass value="0.0053"/>
+            <inertia ixx="0.001" ixy="0.0" ixz="0.0"
+                    iyy="0.001" iyz="0.0"
+                    izz="0.001"/>
+        </inertial>
+        </link>
+        <joint name="${element}_${num}_joint" type="fixed">
+            <parent link="${parent}"/>
+            <child link="${element}_${num}"/>
+            <origin xyz="${x*inv} ${y} ${z}" rpy="0 0 0"/>
+        </joint>
+    </xacro:macro>
+    <xacro:macro name="bat_hold" params=" parent element num x y z">
+        <!-- Link -->
+        <link name="${element}_${num}">
+        <visual>
+            <origin xyz="0 0 0" rpy="0 0 ${pi_2}"/>
+            <geometry>
+            <mesh filename="package://orion_description/meshes/batteryholderx3.stl"
+                scale="0.001 0.001 0.001"/>
+            </geometry>
+            <material name="SoftBlack"/>
+        </visual>
+        <collision>
+            <origin xyz="0 0 0" rpy="0 0 ${pi_2}"/>
+            <geometry>
+            <mesh filename="package://orion_description/meshes/batteryholderx3.stl"
+                scale="0.001 0.001 0.001"/>
+            </geometry>
+        </collision>
+        <inertial>
+            <origin xyz="0 0 0"/>
+            <mass value="0.0053"/>
+            <inertia ixx="0.001" ixy="0.0" ixz="0.0"
+                    iyy="0.001" iyz="0.0"
+                    izz="0.001"/>
+        </inertial>
+        </link>
+        <joint name="${element}_${num}_joint" type="fixed">
+            <parent link="${parent}"/>
+            <child link="${element}_${num}"/>
+            <origin xyz="${x} ${y} ${z}" rpy="0 0 0"/>
+        </joint>
+    </xacro:macro>
+    <xacro:macro name="stack_bat" params="parent num x y z">
+        <xacro:property name="serie" value="0.009"/>
+        <xacro:bat_hold parent="${parent}" element="bathold" num="${num}"
+            x="${x}" y="${y}" z="${z}"/>
+        <xacro:b18650 parent="bathold_${num}" element="b18650_${num}" num="1"
+            x="${-0.065/2}" y="${serie}" z="0.01"/>
+        <xacro:b18650 parent="bathold_${num}" element="b18650_${num}" num="2"
+            x="${-0.065/2}" y="${-serie}" z="0.01"/>
+        <xacro:b18650 parent="bathold_${num}" element="b18650_${num}" num="3"
+            x="${-0.065/2}" y="${-serie*3}" z="0.01"/>
+    </xacro:macro>
+    <!-- //////////////////// SERVOS MACROS ///////////////////////////////-->
+    <xacro:macro name="servo_mounted" params="parent side x y z">
+        <!-- Link -->
+        <xacro:property name="inv" value="1"/>
+        <xacro:property name="flex" value="0"/>
+        <xacro:if value="${side == 2}">
+            <xacro:property name="inv" value="-1"/>
+            <xacro:property name="flex" value="${pi}"/>
+        </xacro:if>
+        <link name="servo_support_${side}">
+        <visual>
+            <origin xyz="0 0 0" rpy="${-pi_2} 0 ${flex}"/>
+            <geometry>
+            <mesh filename="package://orion_description/meshes/servo_sup.stl"
+                scale="0.001 0.001 0.001"/>
+            </geometry>
+            <material name="SoftBlack"/>
+        </visual>
+        <collision>
+            <origin xyz="0 0 0" rpy="${-pi_2} 0 ${flex}"/>
+            <geometry>
+            <mesh filename="package://orion_description/meshes/servo_sup.stl"
+                scale="0.001 0.001 0.001"/>
+            </geometry>
+        </collision>
+        <inertial>
+            <origin xyz="0 0 0"/>
+            <mass value="0.0053"/>
+            <inertia ixx="0.001" ixy="0.0" ixz="0.0"
+                    iyy="0.001" iyz="0.0"
+                    izz="0.001"/>
+        </inertial>
+        </link>
+        <joint name="servo_support_${side}_joint" type="fixed">
+            <parent link="${parent}"/>
+            <child link="servo_support_${side}"/>
+            <origin xyz="${x} ${y*inv} ${z}" rpy="0 0 0"/>
         </joint>
     </xacro:macro>
