Commit message: Description: Added raspberry, speakers, servos and spacers

File: orion_description/urdf/orion_base.urdf.xacro (robot description, xacro)
@@ -251,3 +251,106 @@
         <origin xyz="0.002 0 -0.01" rpy="0 0 0"/>
     </joint>
+    <xacro:x3xspacer_m3x10 id="hs3x10" element="lidar" parent="base_l1_s1"
+        offset_x="0.0234" offset_y="${0.03132/2}" x="-0.0575" y="0" z="0.0025"/>
+    <!-- Link LD19 -->
+    <link name="ld19">
+    <visual>
+        <origin xyz="0 0 0" rpy="0 0 ${pi}"/>
+        <geometry>
+        <mesh filename="package://orion_description/meshes/ld19.stl"
+            scale="0.001 0.001 0.001"/>
+        </geometry>
+        <material name="SoftBlack"/>
+    </visual>
+    <collision>
+        <origin xyz="0 0 0" rpy="0 0 ${pi}"/>
+        <geometry>
+        <mesh filename="package://orion_description/meshes/ld19.stl"
+            scale="0.001 0.001 0.001"/>
+        </geometry>
+    </collision>
+    <inertial>
+        <origin xyz="0 0 0" rpy="0 0 0"/>
+        <mass value="0.1"/>
+        <inertia ixx="0.001" ixy="0.0" ixz="0.0"
+                iyy="0.001" iyz="0.0"
+                izz="0.001"/>
+    </inertial>
+    </link>
+    <!-- Joint LD19 -->
+    <joint name="ld19_joint" type="fixed">
+        <parent link="base_l1_s1"/>
+        <child link="ld19"/>
+        <origin xyz="${-0.0575} -0.0035 0.0125" rpy="0 0 0"/>
+    </joint>
+    <!-- Link Lidar Serial -->
+    <link name="lidar_serial">
+    <visual>
+        <origin xyz="0 0 0" rpy="0 0 ${pi}"/>
+        <geometry>
+        <mesh filename="package://orion_description/meshes/serial_ld.stl"
+            scale="0.001 0.001 0.001"/>
+        </geometry>
+        <material name="ArduinoBlue"/>
+    </visual>
+    <collision>
+        <origin xyz="0 0 0" rpy="0 0 ${pi}"/>
+        <geometry>
+        <mesh filename="package://orion_description/meshes/serial_ld.stl"
+            scale="0.001 0.001 0.001"/>
+        </geometry>
+    </collision>
+    <inertial>
+        <origin xyz="0 0 0" rpy="0 0 ${pi}"/>
+        <mass value="0.1"/>
+        <inertia ixx="0.001" ixy="0.0" ixz="0.0"
+                iyy="0.001" iyz="0.0"
+                izz="0.001"/>
+    </inertial>
+    </link>
+    <!-- Joint Lidar Serial -->
+    <joint name="lidar_serial_joint" type="fixed">
+        <parent link="base_l1_s2"/>
+        <child link="lidar_serial"/>
+        <origin xyz="-0.03 0.025 0.0025" rpy="0 0 0"/>
+    </joint>
+    <!-- ////////////////// THIRD FLOOR COMPONENTES ////////////////////// -->
+    <xacro:speakers_mount parent="base_l2_s2" front="2" side="1" x="-0.0025"
+        y="0.0685" z= "0.0025"/>
+    <xacro:speakers_mount parent="base_l2_s2" front="2" side="2" x="-0.0025"
+        y="0.0685" z= "0.0025"/>
+    <!-- ////////////////// FOURTH FLOOR COMPONENTES ////////////////////// -->
+    <xacro:x4xspacer_m3x10 id="hm3x10" element="rpi5" parent="base_l3_s2"
+        offset_x="${0.049/2}" offset_y="${0.058/2}" x="0" y="0.0435" z="0.0025"/>
+    <!-- Link Lidar Serial -->
+    <link name="rpi5">
+    <visual>
+        <origin xyz="0 0 0" rpy="0 0 ${-pi_2}"/>
+        <geometry>
+        <mesh filename="package://orion_description/meshes/rpi5.stl"
+            scale="0.001 0.001 0.001"/>
+        </geometry>
+        <material name="RaspberryGreen"/>
+    </visual>
+    <collision>
+        <origin xyz="0 0 0" rpy="0 0 ${-pi_2}"/>
+        <geometry>
+        <mesh filename="package://orion_description/meshes/rpi5.stl"
+            scale="0.001 0.001 0.001"/>
+        </geometry>
+    </collision>
+    <inertial>
+        <origin xyz="0 0 0" rpy="0 0 ${-pi_2}"/>
+        <mass value="0.1"/>
+        <inertia ixx="0.001" ixy="0.0" ixz="0.0"
+                iyy="0.001" iyz="0.0"
+                izz="0.001"/>
+    </inertial>
+    </link>
+    <!-- Joint Lidar Serial -->
+    <joint name="rpi5_joint" type="fixed">
+        <parent link="base_l3_s2"/>
+        <child link="rpi5"/>
+        <origin xyz="0 0.0335 0.0125" rpy="0 0 0"/>
+    </joint>
 </robot>

File: orion_description/urdf/orion_macros.urdf.xacro (robot description, xacro)
@@ -587,5 +587,5 @@
     <!-- //////////////////// SERVOS MACROS ///////////////////////////////-->
     <xacro:macro name="servo_mounted" params="parent side x y z">
-        <!-- Link -->
+        <!-- Servo Mount Link -->
         <xacro:property name="inv" value="1"/>
         <xacro:property name="flex" value="0"/>
@@ -618,8 +618,149 @@
         </inertial>
         </link>
+        <!-- Servo Mount Joint -->
         <joint name="servo_support_${side}_joint" type="fixed">
             <parent link="${parent}"/>
             <child link="servo_support_${side}"/>
             <origin xyz="${x} ${y*inv} ${z}" rpy="0 0 0"/>
+        </joint>
+        <!-- Servo Link -->
+        <link name="servo_${side}">
+        <visual>
+            <origin xyz="0 0 0" rpy="${-pi_2*inv} 0 0"/>
+            <geometry>
+            <mesh filename="package://orion_description/meshes/mg996r.stl"
+                scale="0.001 0.001 0.001"/>
+            </geometry>
+            <material name="SoftBlack"/>
+        </visual>
+        <collision>
+            <origin xyz="0 0 0" rpy="${-pi_2*inv} 0 0"/>
+            <geometry>
+            <mesh filename="package://orion_description/meshes/mg996r.stl"
+                scale="0.001 0.001 0.001"/>
+            </geometry>
+        </collision>
+        <inertial>
+            <origin xyz="0 0 0"/>
+            <mass value="0.0053"/>
+            <inertia ixx="0.001" ixy="0.0" ixz="0.0"
+                    iyy="0.001" iyz="0.0"
+                    izz="0.001"/>
+        </inertial>
+        </link>
+        <!-- Servo Joint -->
+        <joint name="servo_${side}_joint" type="fixed">
+            <parent link="servo_support_${side}"/>
+            <child link="servo_${side}"/>
+            <origin xyz="0 ${-0.0216*inv} -0.01375" rpy="0 0 0"/>
+        </joint>
+        <!-- Servo Link -->
+        <link name="servo_conn_${side}">
+        <visual>
+            <origin xyz="0 0 0" rpy="0 0 0"/>
+            <geometry>
+            <mesh filename="package://orion_description/meshes/servo_conn.stl"
+                scale="0.001 0.001 0.001"/>
+            </geometry>
+            <material name="MetalGray"/>
+        </visual>
+        <collision>
+            <origin xyz="0 0 0" rpy="0 0 0"/>
+            <geometry>
+            <mesh filename="package://orion_description/meshes/servo_conn.stl"
+                scale="0.001 0.001 0.001"/>
+            </geometry>
+        </collision>
+        <inertial>
+            <origin xyz="0 0 0"/>
+            <mass value="0.0053"/>
+            <inertia ixx="0.001" ixy="0.0" ixz="0.0"
+                    iyy="0.001" iyz="0.0"
+                    izz="0.001"/>
+        </inertial>
+        </link>
+        <!-- Servo Joint -->
+        <joint name="servo_conn${side}_joint" type="continuous">
+            <axis xyz="0.0 0.0 1.0"/>
+            <parent link="servo_${side}"/>
+            <child link="servo_conn_${side}"/>
+            <origin xyz="0.0115 ${0.0431*inv} 0" rpy="${-pi_2*inv} 0 0"/>
+        </joint>
+    </xacro:macro>
+    <!--///////////////////// SPEAKERS MACROS ///////////////////////-->
+    <!-- Speakers Macro -->
+    <xacro:macro name="speakers_mount" params="parent front side x y z">
+        <!--  Properties -->
+        <xacro:property name="mulf" value="1"/>
+        <xacro:property name="muls" value="1"/>
+        <xacro:property name="inv" value="${pi}"/>
+        <xacro:if value="${front == 2}">
+            <xacro:property name="mulf" value="-1"/>
+        </xacro:if>
+        <xacro:if value="${side == 2}">
+            <xacro:property name="muls" value="-1"/>
+            <xacro:property name="inv" value="0"/>
+        </xacro:if>
+        <!-- Link speaker -->
+        <link name="speaker_sup_${front}${side}">
+        <visual>
+            <origin xyz="0 0 0" rpy="0 0 ${inv}"/>
+            <geometry>
+            <mesh filename="package://orion_description/meshes/speaker_sup.stl"
+                scale="0.001 0.001 0.001"/>
+            </geometry>
+            <material name="SoftBlack"/>
+        </visual>
+        <collision>
+            <origin xyz="0 0 0" rpy="0 0 ${inv}"/>
+            <geometry>
+            <mesh filename="package://orion_description/meshes/speaker_sup.stl"
+                scale="0.001 0.001 0.001"/>
+            </geometry>
+        </collision>
+        <inertial>
+            <origin xyz="0 0 0"/>
+            <mass value="0.0053"/>
+            <inertia ixx="0.001" ixy="0.0" ixz="0.0"
+                    iyy="0.001" iyz="0.0"
+                    izz="0.001"/>
+        </inertial>
+        </link>
+        <!-- Joint speaker support -->
+        <joint name="speaker_sup_${front}${side}_joint" type="fixed">
+            <parent link="${parent}"/>
+            <child link="speaker_sup_${front}${side}"/>
+            <origin xyz="${x*mulf} ${y*muls} ${z}" rpy="0 0 0"/>
+        </joint>
+        <!-- Link speaker support -->
+        <link name="speaker_${front}${side}">
+        <visual>
+            <origin xyz="0 0 0" rpy="0 0 ${inv}"/>
+            <geometry>
+            <mesh filename="package://orion_description/meshes/speaker.stl"
+                scale="0.001 0.001 0.001"/>
+            </geometry>
+            <material name="SoftBlack"/>
+        </visual>
+        <collision>
+            <origin xyz="0 0 0" rpy="0 0 ${inv}"/>
+            <geometry>
+            <mesh filename="package://orion_description/meshes/speaker.stl"
+                scale="0.001 0.001 0.001"/>
+            </geometry>
+        </collision>
+        <inertial>
+            <origin xyz="0 0 0"/>
+            <mass value="0.0053"/>
+            <inertia ixx="0.001" ixy="0.0" ixz="0.0"
+                    iyy="0.001" iyz="0.0"
+                    izz="0.001"/>
+        </inertial>
+        </link>
+        <!-- Joint speaker support -->
+        <joint name="speaker_${front}${side}_joint" type="fixed">
+            <parent link="speaker_sup_${front}${side}"/>
+            <child link="speaker_${front}${side}"/>
+            <origin xyz="0 ${0.0285*muls/2} 0" rpy="0 0 0"/>
         </joint>
     </xacro:macro>
@@ -661,9 +802,19 @@
     <!-- 2 symetric hex spacers by considering y axis -->
     <xacro:macro name="x2xspacer_m3x10"
-                params="name element parent offset_y x y z">
-        <xacro:spacer_m3x10 name="${name}" parent="${parent}" element="${element}"
+                params="id element parent offset_y x y z">
+        <xacro:spacer_m3x10 id="${id}" parent="${parent}" element="${element}"
             front="" side="r" x="${x}" y="${y - offset_y}" z="${z}"/>
-        <xacro:spacer_m3x10 name="${name}" parent="${parent}" element="${element}"
+        <xacro:spacer_m3x10 id="${id}" parent="${parent}" element="${element}"
             front="" side="l" x="${x}" y="${y + offset_y}" z="${z}"/>
+    </xacro:macro>
+    <!-- 3  hex spacers by considering triangle -->
+    <xacro:macro name="x3xspacer_m3x10"
+                params="id element parent offset_x offset_y x y z">
+        <xacro:spacer_m3x10 id="${id}" parent="${parent}" element="${element}"
+            front="f" side="l" x="${x + offset_x}" y="${y - offset_y}" z="${z}"/>
+        <xacro:spacer_m3x10 id="${id}" parent="${parent}" element="${element}"
+            front="r" side="l" x="${x - offset_x}" y="${y - offset_y}" z="${z}"/>
+        <xacro:spacer_m3x10 id="${id}" parent="${parent}" element="${element}"
+            front="" side="r" x="${x}" y="${y + offset_y}" z="${z}"/>
     </xacro:macro>
     <!-- 4 symetric hex spacers by considering x/y axis -->

Commit message: Description: Added maixsense, fixed minor macros errors and started design of wall

File: orion_description/urdf/orion_base.urdf.xacro (robot description, xacro)
@@ -188,4 +188,14 @@
             z="-0.026"/>
     </xacro:if>
+    <xacro:complete_lateral_wall id="servo" parent="base_l0_s1" side="1"
+        x="${-0.115/2}" y="${0.21/2 + 0.0005}" z="${0.082/2 + 0.0025/2}"
+        level="0"/>
+    <xacro:complete_lateral_wall id="servo" parent="base_l0_s1" side="2"
+        x="${-0.115/2}" y="${0.21/2 + 0.0005}" z="${0.082/2 + 0.0025/2}"
+        level="0"/>
+    <xacro:complete_front_wall id="batteries" parent="base_l0_s1" front="1"
+        x="${0.115/2}" z="${0.082/2 + 0.0025/2}" level="0"/>
+    <xacro:complete_front_wall id="batteries" parent="base_l0_s2" front="2"
+        x="${0.115/2}" z="${0.082/2 + 0.0025/2}" level="0"/>
     <!-- ///////////////// SECOND FLOOR COMPONENTS /////////////////////// -->
     <xacro:x4xspacer_m3x10 id="hm3x10" element="espadapter" parent="base_l1_s1"
@@ -317,4 +327,14 @@
         <origin xyz="-0.03 0.025 0.0025" rpy="0 0 0"/>
     </joint>
+    <xacro:complete_lateral_wall id="servo" parent="base_l1_s1" side="1"
+        x="${-0.115/2}" y="${0.21/2 + 0.0005}" z="${0.082/2 + 0.0025/2}"
+        level="1"/>
+    <xacro:complete_lateral_wall id="servo" parent="base_l1_s1" side="2"
+        x="${-0.115/2}" y="${0.21/2 + 0.0005}" z="${0.082/2 + 0.0025/2}"
+        level="1"/>
+    <xacro:complete_front_wall id="batteries" parent="base_l1_s1" front="1"
+        x="${0.115/2}" z="${0.082/2 + 0.0025/2}" level="1"/>
+    <xacro:complete_front_wall id="batteries" parent="base_l1_s2" front="2"
+        x="${0.115/2}" z="${0.082/2 + 0.0025/2}" level="1"/>
     <!-- ////////////////// THIRD FLOOR COMPONENTES ////////////////////// -->
     <xacro:speakers_mount parent="base_l2_s2" front="2" side="1" x="-0.0025"
@@ -322,4 +342,12 @@
     <xacro:speakers_mount parent="base_l2_s2" front="2" side="2" x="-0.0025"
         y="0.0685" z= "0.0025"/>
+    <xacro:complete_lateral_wall id="servo" parent="base_l2_s1" side="1"
+        x="${-0.115/2}" y="${0.21/2 + 0.0005}" z="${0.082/2 + 0.0025/2}"
+        level="2"/>
+    <xacro:complete_lateral_wall id="servo" parent="base_l2_s1" side="2"
+        x="${-0.115/2}" y="${0.21/2 + 0.0005}" z="${0.082/2 + 0.0025/2}"
+        level="2"/>
+    <xacro:complete_front_wall id="batteries" parent="base_l2_s2" front="2"
+        x="${0.115/2}" z="${0.082/2 + 0.0025/2}" level="2"/>
     <!-- ////////////////// FOURTH FLOOR COMPONENTES ////////////////////// -->
     <xacro:x4xspacer_m3x10 id="hm3x10" element="rpi5" parent="base_l3_s2"
@@ -356,3 +384,5 @@
         <origin xyz="0 0.0335 0.0125" rpy="0 0 0"/>
     </joint>
+    <xacro:complete_front_wall id="batteries" parent="base_l3_s2" front="2"
+        x="${0.115/2}" z="${0.082/2 + 0.0025/2}" level="3"/>
 </robot>

File: orion_description/urdf/orion_cameras.urdf.xacro (robot description, xacro)
@@ -98,9 +98,71 @@
             <parent link="os30a_sup"/>
             <child link="os30a"/>
-            <origin xyz="0.025 0 0.015" rpy="0 0 0"/>
+            <origin xyz="0.025 0 0.0145" rpy="0 0 0"/>
         </joint>
     </xacro:if>
     <!--  //////////////////////// A010 CAM ///////////////////////////// -->
     <xacro:if value="${camera == 'a010'}">
+        <!-- Link OS30A Support -->
+        <link name="maixsense_sup">
+        <visual>
+            <origin xyz="0 0 0" rpy="0 0 ${pi_2}"/>
+            <geometry>
+            <mesh filename="package://orion_description/meshes/maixsense_sup.stl"
+                scale="0.001 0.001 0.001"/>
+            </geometry>
+            <material name="SoftBlack"/>
+        </visual>
+        <collision>
+            <origin xyz="0 0 0" rpy="0 0 ${pi_2}"/>
+            <geometry>
+            <mesh filename="package://orion_description/meshes/maixsense_sup.stl"
+                scale="0.001 0.001 0.001"/>
+            </geometry>
+        </collision>
+        <inertial>
+            <origin xyz="0 0 0" rpy="0 0 ${pi_2}"/>
+            <mass value="0.1"/>
+            <inertia ixx="0.001" ixy="0.0" ixz="0.0"
+                    iyy="0.001" iyz="0.0"
+                    izz="0.001"/>
+        </inertial>
+        </link>
+        <!-- Joint OS30A Support -->
+        <joint name="maixsense_sup_joint" type="fixed">
+            <parent link="${level_cam}"/>
+            <child link="maixsense_sup"/>
+            <origin xyz="0.038945 -0.030451 0.0125" rpy="0 0 0"/>
+        </joint>
+        <!-- Link OS30A Support -->
+        <link name="maixsense">
+        <visual>
+            <origin xyz="0 0 0" rpy="${pi_2} 0 ${pi_2}"/>
+            <geometry>
+            <mesh filename="package://orion_description/meshes/maixsense.stl"
+                scale="0.001 0.001 0.001"/>
+            </geometry>
+            <material name="SoftBlack"/>
+        </visual>
+        <collision>
+            <origin xyz="0 0 0" rpy="${pi_2} 0 ${pi_2}"/>
+            <geometry>
+            <mesh filename="package://orion_description/meshes/maixsense.stl"
+                scale="0.001 0.001 0.001"/>
+            </geometry>
+        </collision>
+        <inertial>
+            <origin xyz="0 0 0" rpy="${pi_2} 0 ${pi_2}"/>
+            <mass value="0.1"/>
+            <inertia ixx="0.001" ixy="0.0" ixz="0.0"
+                    iyy="0.001" iyz="0.0"
+                    izz="0.001"/>
+        </inertial>
+        </link>
+        <!-- Joint OS30A Support -->
+        <joint name="maixsense_joint" type="fixed">
+            <parent link="maixsense_sup"/>
+            <child link="maixsense"/>
+            <origin xyz="0 0 0.0205" rpy="0 0 0"/>
+        </joint>
     </xacro:if>
 </robot>

File: orion_description/urdf/orion_macros.urdf.xacro (robot description, xacro)
@@ -681,9 +681,11 @@
         </link>
         <!-- Servo Joint -->
-        <joint name="servo_conn${side}_joint" type="continuous">
+        <joint name="servo_conn${side}_joint" type="revolute">
             <axis xyz="0.0 0.0 1.0"/>
             <parent link="servo_${side}"/>
             <child link="servo_conn_${side}"/>
             <origin xyz="0.0115 ${0.0431*inv} 0" rpy="${-pi_2*inv} 0 0"/>
+            <limit lower="${-pi_2}" upper="${pi_2}" effort="1.0" velocity="1.0"/>
+            <dynamics damping="0.1" friction="0.01"/>
         </joint>
     </xacro:macro>
@@ -901,3 +903,82 @@
             front="r" side="l" x="${x - offset_x}" y="${y - offset_y}" z="${z}"/>
     </xacro:macro>
+    <!-- ///////////////////////////// WALL MACROS //////////////////////// -->
+    <xacro:macro name="complete_lateral_wall"
+            params="id parent side level x y z">
+        <xacro:property name="muls" value="1"/>
+        <xacro:property name="orx" value="${pi}"/>
+        <xacro:if value="${side == 2}">
+            <xacro:property name="muls" value="-1"/>
+            <xacro:property name="orx" value="0"/>
+        </xacro:if>
+        <!-- Link -->
+        <link name="wall${id}_${level}_${side}">
+        <visual>
+            <origin xyz="0 0 0" rpy="${orx} ${pi} 0"/>
+            <geometry>
+            <mesh filename="package://orion_description/meshes/wall_${id}.stl"
+                scale="0.001 0.001 0.001"/>
+            </geometry>
+            <material name="TransparentBlack"/>
+        </visual>
+        <collision>
+            <origin xyz="0 0 0" rpy="${orx} ${pi} 0"/>
+            <geometry>
+            <mesh filename="package://orion_description/meshes/wall_${id}.stl"
+                scale="0.001 0.001 0.001"/>
+            </geometry>
+        </collision>
+        <inertial>
+            <origin xyz="0 0 0"/>
+            <mass value="0.0053"/>
+            <inertia ixx="0.001" ixy="0.0" ixz="0.0"
+                    iyy="0.001" iyz="0.0"
+                    izz="0.001"/>
+        </inertial>
+        </link>
+        <joint name="wall${id}_${level}_${side}_joint" type="fixed">
+        <parent link="${parent}"/>
+        <child link="wall${id}_${level}_${side}"/>
+        <origin xyz="${x} ${y*muls} ${z}" rpy="0 0 0"/>
+        </joint>
+    </xacro:macro>
+    <xacro:macro name="complete_front_wall"
+            params="id parent front level x z">
+        <xacro:property name="mulf" value="1"/>
+        <xacro:property name="orz" value="0"/>
+        <xacro:if value="${front == 2}">
+            <xacro:property name="mulf" value="-1"/>
+            <xacro:property name="orz" value="${pi}"/>
+        </xacro:if>
+        <!-- Link -->
+        <link name="wall${id}_${level}_${front}">
+        <visual>
+            <origin xyz="0 0 0" rpy="0 0 ${pi_2 + orz}"/>
+            <geometry>
+            <mesh filename="package://orion_description/meshes/wall_${id}.stl"
+                scale="0.001 0.001 0.001"/>
+            </geometry>
+            <material name="TransparentBlack"/>
+        </visual>
+        <collision>
+            <origin xyz="0 0 0" rpy="0 0 ${pi_2 + orz}"/>
+            <geometry>
+            <mesh filename="package://orion_description/meshes/wall_${id}.stl"
+                scale="0.001 0.001 0.001"/>
+            </geometry>
+        </collision>
+        <inertial>
+            <origin xyz="0 0 0"/>
+            <mass value="0.0053"/>
+            <inertia ixx="0.001" ixy="0.0" ixz="0.0"
+                    iyy="0.001" iyz="0.0"
+                    izz="0.001"/>
+        </inertial>
+        </link>
+        <joint name="wall${id}_${level}_${front}_joint" type="fixed">
+        <parent link="${parent}"/>
+        <child link="wall${id}_${level}_${front}"/>
+        <origin xyz="${x*mulf} 0 ${z}" rpy="0 0 0"/>
+        </joint>
+    </xacro:macro>
 </robot>

File: orion_description/urdf/orion_materials.urdf.xacro (robot description, xacro)
@@ -30,3 +30,7 @@
         <color rgba="0.5 0.5 0.5 1.0"/>
     </material>
+    <!-- Equivalent to RGB(39, 39, 39) -->
+    <material name="TransparentBlack">
+        <color rgba="0.3 0.3 0.3 0.8"/>
+    </material>
 </robot>
