Commit message: Description: Adding some walls, improving xacro | Assets: Added switches and modified half platform

File: orion_description/urdf/orion_base.urdf.xacro (robot description, xacro)
@@ -196,5 +196,5 @@
     <xacro:complete_front_wall id="batteries" parent="base_l0_s1" front="1"
         x="${0.115/2}" z="${0.082/2 + 0.0025/2}" level="0"/>
-    <xacro:complete_front_wall id="batteries" parent="base_l0_s2" front="2"
+    <xacro:complete_front_wall id="fdefault" parent="base_l0_s2" front="2"
         x="${0.115/2}" z="${0.082/2 + 0.0025/2}" level="0"/>
     <!-- ///////////////// SECOND FLOOR COMPONENTS /////////////////////// -->
@@ -327,13 +327,13 @@
         <origin xyz="-0.03 0.025 0.0025" rpy="0 0 0"/>
     </joint>
-    <xacro:complete_lateral_wall id="servo" parent="base_l1_s1" side="1"
+    <xacro:complete_lateral_wall id="llidar" parent="base_l1_s1" side="1"
         x="${-0.115/2}" y="${0.21/2 + 0.0005}" z="${0.082/2 + 0.0025/2}"
         level="1"/>
-    <xacro:complete_lateral_wall id="servo" parent="base_l1_s1" side="2"
+    <xacro:complete_lateral_wall id="llidar" parent="base_l1_s1" side="2"
         x="${-0.115/2}" y="${0.21/2 + 0.0005}" z="${0.082/2 + 0.0025/2}"
         level="1"/>
-    <xacro:complete_front_wall id="batteries" parent="base_l1_s1" front="1"
+    <xacro:complete_front_wall id="flidar" parent="base_l1_s1" front="1"
         x="${0.115/2}" z="${0.082/2 + 0.0025/2}" level="1"/>
-    <xacro:complete_front_wall id="batteries" parent="base_l1_s2" front="2"
+    <xacro:complete_front_wall id="flidar" parent="base_l1_s2" front="2"
         x="${0.115/2}" z="${0.082/2 + 0.0025/2}" level="1"/>
     <!-- ////////////////// THIRD FLOOR COMPONENTES ////////////////////// -->
@@ -342,11 +342,11 @@
     <xacro:speakers_mount parent="base_l2_s2" front="2" side="2" x="-0.0025"
         y="0.0685" z= "0.0025"/>
-    <xacro:complete_lateral_wall id="servo" parent="base_l2_s1" side="1"
+    <xacro:complete_lateral_wall id="speaker1" parent="base_l2_s1" side="1"
         x="${-0.115/2}" y="${0.21/2 + 0.0005}" z="${0.082/2 + 0.0025/2}"
         level="2"/>
-    <xacro:complete_lateral_wall id="servo" parent="base_l2_s1" side="2"
+    <xacro:complete_lateral_wall id="speaker2" parent="base_l2_s1" side="2"
         x="${-0.115/2}" y="${0.21/2 + 0.0005}" z="${0.082/2 + 0.0025/2}"
         level="2"/>
-    <xacro:complete_front_wall id="batteries" parent="base_l2_s2" front="2"
+    <xacro:complete_front_wall id="fdefault" parent="base_l2_s2" front="2"
         x="${0.115/2}" z="${0.082/2 + 0.0025/2}" level="2"/>
     <!-- ////////////////// FOURTH FLOOR COMPONENTES ////////////////////// -->
@@ -384,5 +384,5 @@
         <origin xyz="0 0.0335 0.0125" rpy="0 0 0"/>
     </joint>
-    <xacro:complete_front_wall id="batteries" parent="base_l3_s2" front="2"
+    <xacro:complete_front_wall id="rpi" parent="base_l3_s2" front="2"
         x="${0.115/2}" z="${0.082/2 + 0.0025/2}" level="3"/>
 </robot>

File: orion_description/urdf/orion_cameras.urdf.xacro (robot description, xacro)
@@ -67,5 +67,5 @@
             <parent link="${level_cam}"/>
             <child link="os30a_sup"/>
-            <origin xyz="0.0555 0 0.0025" rpy="0 0 0"/>
+            <origin xyz="${0.0555 - 0.0285} 0 0.0025" rpy="0 0 0"/>
         </joint>
         <!-- Link OS30A Support -->
@@ -103,5 +103,5 @@
     <!--  //////////////////////// A010 CAM ///////////////////////////// -->
     <xacro:if value="${camera == 'a010'}">
-        <!-- Link OS30A Support -->
+        <!-- Link Maixsense Support -->
         <link name="maixsense_sup">
         <visual>
@@ -128,5 +128,5 @@
         </inertial>
         </link>
-        <!-- Joint OS30A Support -->
+        <!-- Joint Maixsense Support -->
         <joint name="maixsense_sup_joint" type="fixed">
             <parent link="${level_cam}"/>
@@ -134,5 +134,5 @@
             <origin xyz="0.038945 -0.030451 0.0125" rpy="0 0 0"/>
         </joint>
-        <!-- Link OS30A Support -->
+        <!-- Link Maixsense -->
         <link name="maixsense">
         <visual>
@@ -159,5 +159,5 @@
         </inertial>
         </link>
-        <!-- Joint OS30A Support -->
+        <!-- Joint Maixsense -->
         <joint name="maixsense_joint" type="fixed">
             <parent link="maixsense_sup"/>

Commit message: Description: Changed macros for metric spacer in order to reduce code

File: orion_description/urdf/orion_base.urdf.xacro (robot description, xacro)
@@ -27,5 +27,5 @@
     <xacro:double_spacer_10x80 front="2" level="1" x="${0.15/2 - 0.0275}"
             y="${0.21/2 - 0.010}" z="0"/>
-    <xacro:double_spacer_10x80 front="1" level="2" x="${0.15/2 - 0.0275}"
+    <xacro:double_spacer_10x80 front="1" level="2" x="${-0.15/2 + 0.0275 + 0.006}"
             y="${0.21/2 - 0.010}" z="0"/>
     <xacro:double_spacer_10x80 front="2" level="2" x="${0.15/2 - 0.0275}"
@@ -41,5 +41,5 @@
         z="-0.0225"/>
     <!-- /////////////////////// CASTER WHEEL //////////////////////////-->
-    <xacro:x4xspacer_m4x17 id="hm4x17" element="caster" parent="base_l0_s2"
+    <xacro:x4xmetric_spacer id="m4x17" element="caster" parent="base_l0_s2"
         offset_x="0.012" offset_y="0.015" x="-0.022" y="0"
         z="${-0.001 - 0.017}"/>
@@ -48,6 +48,7 @@
     <!-- //////////////// FIRST FLOOR COMPONENTS ///////////////////// -->
     <!-- Hex spacers for Battery Support -->
-    <xacro:x6xspacer_m3x10 id="hm3x10" element="bathol" parent="base_l0_s1"
-        offset_x="${0.0855/2}" offset_y="${0.127/2}" x="0.005" y="0" z="0.0025"/>
+    <xacro:x6xmetric_spacer id="m3x10" element="bathol" parent="base_l0_s1"
+        offset_x="${0.0855/2}" offset_y="${0.127/2}" x="0.005" y="0"
+        z="0.0025"/>
     <!-- Link Battery Support-->
     <link name="bat_platform">
@@ -86,5 +87,5 @@
         z="0"/>
     <!-- Hex spacers for Motor Driver-->
-    <xacro:x4xspacer_m3x10 id="hm3x10" element="driver" parent="base_l0_s2"
+    <xacro:x4xmetric_spacer id="m3x10" element="driver" parent="base_l0_s2"
         offset_x="${0.03702/2}" offset_y="${-0.0368/2}" x="-0.023453"
         y="0.031351" z="0.0025"/>
@@ -199,5 +200,5 @@
         x="${0.115/2}" z="${0.082/2 + 0.0025/2}" level="0"/>
     <!-- ///////////////// SECOND FLOOR COMPONENTS /////////////////////// -->
-    <xacro:x4xspacer_m3x10 id="hm3x10" element="espadapter" parent="base_l1_s1"
+    <xacro:x4xmetric_spacer id="m3x10" element="esp_adapter" parent="base_l1_s1"
         offset_x="${0.0577/2}" offset_y="${0.0607/2}" x="0" y="0" z="-0.01"/>
     <!-- Link Esp32 Adapter -->
@@ -263,5 +264,5 @@
         <origin xyz="0.002 0 -0.01" rpy="0 0 0"/>
     </joint>
-    <xacro:x3xspacer_m3x10 id="hs3x10" element="lidar" parent="base_l1_s1"
+    <xacro:x3xmetric_spacer id="m3x10" element="lidar" parent="base_l1_s1"
         offset_x="0.0234" offset_y="${0.03132/2}" x="-0.0575" y="0" z="0.0025"/>
     <!-- Link LD19 -->
@@ -353,5 +354,5 @@
     </xacro:if>
     <!-- ////////////////// FOURTH FLOOR COMPONENTES ////////////////////// -->
-    <xacro:x4xspacer_m3x10 id="hm3x10" element="rpi5" parent="base_l3_s2"
+    <xacro:x4xmetric_spacer id="m3x10" element="rpi5" parent="base_l3_s2"
         offset_x="${0.049/2}" offset_y="${0.058/2}" x="0" y="0.0435" z="0.0025"/>
     <!-- Link Rasberry Pi -->

File: orion_description/urdf/orion_macros.urdf.xacro (robot description, xacro)
@@ -767,140 +767,4 @@
         </joint>
     </xacro:macro>
-    <!--///////////////////// M3 x 10 SPACERS MACROS ///////////////////////-->
-    <!-- Hex spacer M3 x 10 macro -->
-    <xacro:macro name="spacer_m3x10"
-            params="id parent element front side x y z">
-        <!-- Link -->
-        <link name="${id}_${element}_${front}${side}">
-        <visual>
-            <origin xyz="0 0 0" rpy="0 0 0"/>
-            <geometry>
-            <mesh filename="package://orion_description/meshes/spacer_m3x10.stl"
-                scale="0.001 0.001 0.001"/>
-            </geometry>
-            <material name="Brass"/>
-        </visual>
-        <collision>
-            <origin xyz="0 0 0" rpy="0 0 0"/>
-            <geometry>
-            <mesh filename="package://orion_description/meshes/spacer_m3x10.stl"
-                scale="0.001 0.001 0.001"/>
-            </geometry>
-        </collision>
-        <inertial>
-            <origin xyz="0 0 0"/>
-            <mass value="0.0053"/>
-            <inertia ixx="0.001" ixy="0.0" ixz="0.0"
-                    iyy="0.001" iyz="0.0"
-                    izz="0.001"/>
-        </inertial>
-        </link>
-        <joint name="${id}_${element}_${front}${side}_joint" type="fixed">
-            <parent link="${parent}"/>
-            <child link="${id}_${element}_${front}${side}"/>
-            <origin xyz="${x} ${y} ${z}" rpy="0 0 0"/>
-        </joint>
-    </xacro:macro>
-    <!-- 2 symetric hex spacers by considering y axis -->
-    <xacro:macro name="x2xspacer_m3x10"
-                params="id element parent offset_y x y z">
-        <xacro:spacer_m3x10 id="${id}" parent="${parent}" element="${element}"
-            front="" side="r" x="${x}" y="${y - offset_y}" z="${z}"/>
-        <xacro:spacer_m3x10 id="${id}" parent="${parent}" element="${element}"
-            front="" side="l" x="${x}" y="${y + offset_y}" z="${z}"/>
-    </xacro:macro>
-    <!-- 3  hex spacers by considering triangle -->
-    <xacro:macro name="x3xspacer_m3x10"
-                params="id element parent offset_x offset_y x y z">
-        <xacro:spacer_m3x10 id="${id}" parent="${parent}" element="${element}"
-            front="f" side="l" x="${x + offset_x}" y="${y - offset_y}" z="${z}"/>
-        <xacro:spacer_m3x10 id="${id}" parent="${parent}" element="${element}"
-            front="r" side="l" x="${x - offset_x}" y="${y - offset_y}" z="${z}"/>
-        <xacro:spacer_m3x10 id="${id}" parent="${parent}" element="${element}"
-            front="" side="r" x="${x}" y="${y + offset_y}" z="${z}"/>
-    </xacro:macro>
-    <!-- 4 symetric hex spacers by considering x/y axis -->
-    <xacro:macro name="x4xspacer_m3x10"
-                params="id element parent offset_x offset_y x y z">
-        <xacro:spacer_m3x10 id="${id}" parent="${parent}" element="${element}"
-            front="f" side="r" x="${x + offset_x}" y="${y - offset_y}" z="${z}"/>
-        <xacro:spacer_m3x10 id="${id}" parent="${parent}" element="${element}"
-            front="f" side="l" x="${x + offset_x}" y="${y + offset_y}" z="${z}"/>
-        <xacro:spacer_m3x10 id="${id}" parent="${parent}" element="${element}"
-            front="r" side="r" x="${x - offset_x}" y="${y + offset_y}" z="${z}"/>
-        <xacro:spacer_m3x10 id="${id}" parent="${parent}" element="${element}"
-            front="r" side="l" x="${x - offset_x}" y="${y - offset_y}" z="${z}"/>
-    </xacro:macro>
-    <!-- 6 symetric hex spacers by considering x/y axis -->
-    <xacro:macro name="x6xspacer_m3x10"
-                params="id element parent offset_x offset_y x y z">
-        <xacro:spacer_m3x10 id="${id}" parent="${parent}" element="${element}"
-            front="f" side="r" x="${x + offset_x}" y="${y - offset_y}" z="${z}"/>
-        <xacro:spacer_m3x10 id="${id}" parent="${parent}" element="${element}"
-            front="f" side="l" x="${x + offset_x}" y="${y + offset_y}" z="${z}"/>
-        <xacro:spacer_m3x10 id="${id}" parent="${parent}" element="${element}"
-            front="r" side="r" x="${x - offset_x}" y="${y + offset_y}" z="${z}"/>
-        <xacro:spacer_m3x10 id="${id}" parent="${parent}" element="${element}"
-            front="r" side="l" x="${x - offset_x}" y="${y - offset_y}" z="${z}"/>
-        <xacro:spacer_m3x10 id="${id}" parent="${parent}" element="${element}"
-            front="f" side="" x="${x + offset_x}" y="0" z="${z}"/>
-        <xacro:spacer_m3x10 id="${id}" parent="${parent}" element="${element}"
-            front="r" side="" x="${x - offset_x}" y="0" z="${z}"/>
-    </xacro:macro>
-    <!--///////////////////// M4 x 17 SPACERS MACROS ///////////////////////-->
-    <!-- Hex spacer M4 x 17 macro -->
-    <xacro:macro name="spacer_m4x17"
-            params="id parent element front side x y z">
-        <!-- Link -->
-        <link name="${id}_${element}_${front}${side}">
-        <visual>
-            <origin xyz="0 0 0" rpy="0 0 0"/>
-            <geometry>
-            <mesh filename="package://orion_description/meshes/spacer_m4x17.stl"
-                scale="0.001 0.001 0.001"/>
-            </geometry>
-            <material name="Brass"/>
-        </visual>
-        <collision>
-            <origin xyz="0 0 0" rpy="0 0 0"/>
-            <geometry>
-            <mesh filename="package://orion_description/meshes/spacer_m4x17.stl"
-                scale="0.001 0.001 0.001"/>
-            </geometry>
-        </collision>
-        <inertial>
-            <origin xyz="0 0 0"/>
-            <mass value="0.0053"/>
-            <inertia ixx="0.001" ixy="0.0" ixz="0.0"
-                    iyy="0.001" iyz="0.0"
-                    izz="0.001"/>
-        </inertial>
-        </link>
-        <joint name="${id}_${element}_${front}${side}_joint" type="fixed">
-        <parent link="${parent}"/>
-        <child link="${id}_${element}_${front}${side}"/>
-        <origin xyz="${x} ${y} ${z}" rpy="0 0 0"/>
-        </joint>
-    </xacro:macro>
-    <!-- 2 symetric hex spacers by considering y axis -->
-    <xacro:macro name="x2xspacer_m4x17"
-                params="id element parent offset_y x y z">
-        <xacro:spacer_m4x17 id="${id}" parent="${parent}" element="${element}"
-            front="" side="r" x="${x}" y="${y - offset_y}" z="${z}"/>
-        <xacro:spacer_m4x17 id="${id}" parent="${parent}" element="${element}"
-            front="" side="l" x="${x}" y="${y + offset_y}" z="${z}"/>
-    </xacro:macro>
-    <!-- 4 symetric hex spacers by considering x/y axis -->
-    <xacro:macro name="x4xspacer_m4x17"
-                params="id element parent offset_x offset_y x y z">
-        <xacro:spacer_m4x17 id="${id}" parent="${parent}" element="${element}"
-            front="f" side="r" x="${x + offset_x}" y="${y - offset_y}" z="${z}"/>
-        <xacro:spacer_m4x17 id="${id}" parent="${parent}" element="${element}"
-            front="f" side="l" x="${x + offset_x}" y="${y + offset_y}" z="${z}"/>
-        <xacro:spacer_m4x17 id="${id}" parent="${parent}" element="${element}"
-            front="r" side="r" x="${x - offset_x}" y="${y + offset_y}" z="${z}"/>
-        <xacro:spacer_m4x17 id="${id}" parent="${parent}" element="${element}"
-            front="r" side="l" x="${x - offset_x}" y="${y - offset_y}" z="${z}"/>
-    </xacro:macro>
     <!-- ///////////////////////////// WALL MACROS //////////////////////// -->
     <xacro:macro name="complete_lateral_wall"
@@ -982,3 +846,92 @@
         </joint>
     </xacro:macro>
+    <!-- /////////////////////////// Generic Metric Spacer /////////////////-->
+    <xacro:macro name="metric_spacer"
+            params="id parent element front side x y z">
+        <!-- Link Spacer -->
+        <link name="${id}_${element}_${front}${side}">
+        <visual>
+            <origin xyz="0 0 0" rpy="0 0 0"/>
+            <geometry>
+            <mesh filename="package://orion_description/meshes/spacer_${id}.stl"
+                scale="0.001 0.001 0.001"/>
+            </geometry>
+            <material name="Brass"/>
+        </visual>
+        <collision>
+            <origin xyz="0 0 0" rpy="0 0 0"/>
+            <geometry>
+            <mesh filename="package://orion_description/meshes/spacer_${id}.stl"
+                scale="0.001 0.001 0.001"/>
+            </geometry>
+        </collision>
+        <inertial>
+            <origin xyz="0 0 0 " rpy="0 0 0"/>
+            <xacro:if value="${id == 'm4x17'}">
+                <mass value="0.0024"/>
+                <inertia ixx="8.5251996963501e-08" ixy="0" ixz="0"
+                        iyy="8.648216387229408e-08" iyz="0"
+                        izz="1.333016690879308e-08"/>
+            </xacro:if>
+            <xacro:if value="${id == 'm3x10'}">
+                <mass value="0.0012"/>
+                <inertia ixx="1.2825999244689955e-08" ixy="0" ixz="0"
+                        iyy="1.3441082699086494e-08" iyz="0"
+                        izz="6.66508345439654e-09"/>
+            </xacro:if>
+        </inertial>
+        </link>
+        <!-- Joint Spacer -->
+        <joint name="${id}_${element}_${front}${side}_joint" type="fixed">
+            <parent link="${parent}"/>
+            <child link="${id}_${element}_${front}${side}"/>
+            <origin xyz="${x} ${y} ${z}" rpy="0 0 0"/>
+        </joint>
+    </xacro:macro>
+    <!-- 2 symetric hex spacers by considering offset -->
+    <xacro:macro name="x2xmetric_spacer"
+                params="id element parent offset_y x y z">
+        <xacro:metric_spacer id="${id}" parent="${parent}" element="${element}"
+            front="" side="r" x="${x}" y="${y - offset_y}" z="${z}"/>
+        <xacro:metric_spacer id="${id}" parent="${parent}" element="${element}"
+            front="" side="l" x="${x}" y="${y + offset_y}" z="${z}"/>
+    </xacro:macro>
+    <!-- 3  hex spacers by considering triangle -->
+    <xacro:macro name="x3xmetric_spacer"
+                params="id element parent offset_x offset_y x y z">
+        <xacro:metric_spacer id="${id}" parent="${parent}" element="${element}"
+            front="f" side="l" x="${x + offset_x}" y="${y - offset_y}" z="${z}"/>
+        <xacro:metric_spacer id="${id}" parent="${parent}" element="${element}"
+            front="r" side="l" x="${x - offset_x}" y="${y - offset_y}" z="${z}"/>
+        <xacro:metric_spacer id="${id}" parent="${parent}" element="${element}"
+            front="" side="r" x="${x}" y="${y + offset_y}" z="${z}"/>
+    </xacro:macro>
+    <!-- 4  hex spacers by considering mirror offset -->
+    <xacro:macro name="x4xmetric_spacer"
+                params="id element parent offset_x offset_y x y z">
+        <xacro:metric_spacer id="${id}" parent="${parent}" element="${element}"
+            front="f" side="r" x="${x + offset_x}" y="${y - offset_y}" z="${z}"/>
+        <xacro:metric_spacer id="${id}" parent="${parent}" element="${element}"
+            front="f" side="l" x="${x + offset_x}" y="${y + offset_y}" z="${z}"/>
+        <xacro:metric_spacer id="${id}" parent="${parent}" element="${element}"
+            front="r" side="r" x="${x - offset_x}" y="${y + offset_y}" z="${z}"/>
+        <xacro:metric_spacer id="${id}" parent="${parent}" element="${element}"
+            front="r" side="l" x="${x - offset_x}" y="${y - offset_y}" z="${z}"/>
+    </xacro:macro>
+    <!-- 6  hex spacers by considering mirror offset and middles-->
+    <xacro:macro name="x6xmetric_spacer"
+                params="id element parent offset_x offset_y x y z">
+        <xacro:metric_spacer id="${id}" parent="${parent}" element="${element}"
+            front="f" side="r" x="${x + offset_x}" y="${y - offset_y}" z="${z}"/>
+        <xacro:metric_spacer id="${id}" parent="${parent}" element="${element}"
+            front="f" side="l" x="${x + offset_x}" y="${y + offset_y}" z="${z}"/>
+        <xacro:metric_spacer id="${id}" parent="${parent}" element="${element}"
+            front="r" side="r" x="${x - offset_x}" y="${y + offset_y}" z="${z}"/>
+        <xacro:metric_spacer id="${id}" parent="${parent}" element="${element}"
+            front="r" side="l" x="${x - offset_x}" y="${y - offset_y}" z="${z}"/>
+        <xacro:metric_spacer id="${id}" parent="${parent}" element="${element}"
+            front="f" side="" x="${x + offset_x}" y="0" z="${z}"/>
+        <xacro:metric_spacer id="${id}" parent="${parent}" element="${element}"
+            front="r" side="" x="${x - offset_x}" y="0" z="${z}"/>
+    </xacro:macro>
 </robot>
