Commit message: Description: Changed wall macro and indicate changes between rpis | Assets: Added new walls

File: orion_description/urdf/orion_base.urdf.xacro (robot description, xacro)
@@ -183,10 +183,35 @@
         <origin xyz="-0.0025 0 ${0.06/2}" rpy="0 0 0"/>
     </joint>
-    <xacro:if value="${servo}">
-        <xacro:servo_mounted parent="base_l1_s2" side="1" x="0.00275" y="0.0765"
-            z="-0.026"/>
-        <xacro:servo_mounted parent="base_l1_s2" side="2" x="0.00275" y="0.0765"
-            z="-0.026"/>
-    </xacro:if>
+    <!-- Link Switch -->
+    <link name="switch">
+    <visual>
+        <origin xyz="0 0 0" rpy="${pi/2} 0 ${pi/2}"/>
+        <geometry>
+        <mesh filename="package://orion_description/meshes/switch_3s_15a.stl"
+            scale="0.001 0.001 0.001"/>
+        </geometry>
+        <material name="ArduinoBlue"/>
+    </visual>
+    <collision>
+        <origin xyz="0 0 0" rpy="${pi/2} 0 ${pi/2}"/>
+        <geometry>
+        <mesh filename="package://orion_description/meshes/switch_3s_15a.stl"
+            scale="0.001 0.001 0.001"/>
+        </geometry>
+    </collision>
+    <inertial>
+        <origin xyz="0 0 0" rpy="${pi/2} 0 ${pi/2}"/>
+        <mass value="0.1"/>
+        <inertia ixx="0.001" ixy="0.0" ixz="0.0"
+                iyy="0.001" iyz="0.0"
+                izz="0.001"/>
+    </inertial>
+    </link>
+    <!-- Joint Switch -->
+    <joint name="switch_joint" type="fixed">
+        <parent link="base_l1_s1"/>
+        <child link="switch"/>
+        <origin xyz="0.025 0.074 -0.015" rpy="0 0 0"/>
+    </joint>
     <xacro:complete_lateral_wall id="servo" parent="base_l0_s1" side="1"
         x="${-0.115/2}" y="${0.21/2 + 0.0005}" z="${0.082/2 + 0.0025/2}"
@@ -328,4 +353,10 @@
         <origin xyz="-0.03 0.025 0.0025" rpy="0 0 0"/>
     </joint>
+    <xacro:if value="${servo}">
+        <xacro:servo_mounted parent="base_l1_s2" side="1" x="0.00275" y="0.0765"
+            z="-0.026"/>
+        <xacro:servo_mounted parent="base_l1_s2" side="2" x="0.00275" y="0.0765"
+            z="-0.026"/>
+    </xacro:if>
     <xacro:complete_lateral_wall id="llidar" parent="base_l1_s1" side="1"
         x="${-0.115/2}" y="${0.21/2 + 0.0005}" z="${0.082/2 + 0.0025/2}"
@@ -344,8 +375,18 @@
         <xacro:speakers_mount parent="base_l2_s2" front="2" side="2" x="-0.0025"
             y="0.0685" z= "0.0025"/>
-        <xacro:complete_lateral_wall id="speaker1" parent="base_l2_s1" side="1"
+        <xacro:complete_lateral_wall id="curve_speaker" parent="base_l2_s1" side="1"
             x="${-0.115/2}" y="${0.21/2 + 0.0005}" z="${0.082/2 + 0.0025/2}"
             level="2"/>
-        <xacro:complete_lateral_wall id="speaker2" parent="base_l2_s1" side="2"
+        <xacro:complete_lateral_wall id="curve_speaker" parent="base_l2_s1" side="2"
+            x="${-0.115/2}" y="${0.21/2 + 0.0005}" z="${0.082/2 + 0.0025/2}"
+            level="2"/>
+        <xacro:complete_front_wall id="fdefault" parent="base_l2_s2" front="2"
+            x="${0.115/2}" z="${0.082/2 + 0.0025/2}" level="2"/>
+    </xacro:if>
+    <xacro:if value="${rasp == 'rpi5'}">
+        <xacro:complete_lateral_wall id="curve" parent="base_l2_s1" side="1"
+            x="${-0.115/2}" y="${0.21/2 + 0.0005}" z="${0.082/2 + 0.0025/2}"
+            level="2"/>
+        <xacro:complete_lateral_wall id="curve" parent="base_l2_s1" side="2"
             x="${-0.115/2}" y="${0.21/2 + 0.0005}" z="${0.082/2 + 0.0025/2}"
             level="2"/>

File: orion_description/urdf/orion_macros.urdf.xacro (robot description, xacro)
@@ -771,13 +771,11 @@
             params="id parent side level x y z">
         <xacro:property name="muls" value="1"/>
-        <xacro:property name="orx" value="${pi}"/>
         <xacro:if value="${side == 2}">
             <xacro:property name="muls" value="-1"/>
-            <xacro:property name="orx" value="0"/>
         </xacro:if>
         <!-- Link -->
         <link name="wall${id}_${level}_${side}">
         <visual>
-            <origin xyz="0 0 0" rpy="${orx} ${pi} 0"/>
+            <origin xyz="0 0 0" rpy="0 0 ${pi}"/>
             <geometry>
             <mesh filename="package://orion_description/meshes/wall_${id}.stl"
@@ -787,5 +785,5 @@
         </visual>
         <collision>
-            <origin xyz="0 0 0" rpy="${orx} ${pi} 0"/>
+            <origin xyz="0 0 0" rpy="0 0 ${pi}"/>
             <geometry>
             <mesh filename="package://orion_description/meshes/wall_${id}.stl"
@@ -804,5 +802,5 @@
         <parent link="${parent}"/>
         <child link="wall${id}_${level}_${side}"/>
-        <origin xyz="${x} ${y*muls} ${z}" rpy="0 0 0"/>
+        <origin xyz="${x} ${(y+0.00075)*muls} ${z}" rpy="0 0 0"/>
         </joint>
     </xacro:macro>
@@ -843,5 +841,5 @@
         <parent link="${parent}"/>
         <child link="wall${id}_${level}_${front}"/>
-        <origin xyz="${x*mulf} 0 ${z}" rpy="0 0 0"/>
+        <origin xyz="${(x+0.00075)*mulf} 0 ${z}" rpy="0 0 0"/>
         </joint>
     </xacro:macro>

Commit message: Description: Added screen, screen support and new speaker | Assets: Designed pending walls, screen support and new speaker

File: orion_description/urdf/orion_base.urdf.xacro (robot description, xacro)
@@ -385,4 +385,35 @@
     </xacro:if>
     <xacro:if value="${rasp == 'rpi5'}">
+        <!-- Link Stereo Speaker  -->
+        <link name="stereo">
+        <visual>
+            <origin xyz="0 0 0" rpy="0 0 ${-pi_2}"/>
+            <geometry>
+            <mesh filename="package://orion_description/meshes/speaker_stereo.stl"
+                scale="0.001 0.001 0.001"/>
+            </geometry>
+            <material name="SoftBlack"/>
+        </visual>
+        <collision>
+            <origin xyz="0 0 0" rpy="0 0 ${-pi_2}"/>
+            <geometry>
+            <mesh filename="package://orion_description/meshes/speaker_stereo.stl"
+                scale="0.001 0.001 0.001"/>
+            </geometry>
+        </collision>
+        <inertial>
+            <origin xyz="0 0 0" rpy="0 0 ${-pi_2}"/>
+            <mass value="0.1"/>
+            <inertia ixx="0.001" ixy="0.0" ixz="0.0"
+                    iyy="0.001" iyz="0.0"
+                    izz="0.001"/>
+        </inertial>
+        </link>
+        <!-- Joint Stereo Speaker -->
+        <joint name="stereo_joint" type="fixed">
+            <parent link="base_l2_s2"/>
+            <child link="stereo"/>
+            <origin xyz="-0.02 0 0.025" rpy="0 0 0"/>
+        </joint>
         <xacro:complete_lateral_wall id="curve" parent="base_l2_s1" side="1"
             x="${-0.115/2}" y="${0.21/2 + 0.0005}" z="${0.082/2 + 0.0025/2}"
@@ -391,5 +422,5 @@
             x="${-0.115/2}" y="${0.21/2 + 0.0005}" z="${0.082/2 + 0.0025/2}"
             level="2"/>
-        <xacro:complete_front_wall id="fdefault" parent="base_l2_s2" front="2"
+        <xacro:complete_front_wall id="stereo" parent="base_l2_s2" front="2"
             x="${0.115/2}" z="${0.082/2 + 0.0025/2}" level="2"/>
     </xacro:if>
@@ -428,5 +459,73 @@
         <origin xyz="0 0.0335 0.0125" rpy="0 0 0"/>
     </joint>
+    <xacro:complete_lateral_wall id="screen" parent="base_l3_s1" side="1"
+            x="${-0.115/2 + 0.005}" y="${0.21/2 + 0.0005}" z="${0.082/2 + 0.0025/2}"
+            level="2"/>
+    <xacro:complete_lateral_wall id="screen" parent="base_l3_s1" side="2"
+            x="${-0.115/2 + 0.005}" y="${0.21/2 + 0.0005}" z="${0.082/2 + 0.0025/2}"
+            level="2"/>
     <xacro:complete_front_wall id="rpi" parent="base_l3_s2" front="2"
         x="${0.115/2}" z="${0.082/2 + 0.0025/2}" level="3"/>
+    <!-- Link Screen Sup  -->
+    <link name="screen_sup">
+    <visual>
+        <origin xyz="0 0 0" rpy="0 0 ${pi_2}"/>
+        <geometry>
+        <mesh filename="package://orion_description/meshes/screen_sup.stl"
+            scale="0.001 0.001 0.001"/>
+        </geometry>
+        <material name="TransparentBlack"/>
+    </visual>
+    <collision>
+        <origin xyz="0 0 0" rpy="0 0 ${pi_2}"/>
+        <geometry>
+        <mesh filename="package://orion_description/meshes/screen_sup.stl"
+            scale="0.001 0.001 0.001"/>
+        </geometry>
+    </collision>
+    <inertial>
+        <origin xyz="0 0 0" rpy="0 0 ${pi_2}"/>
+        <mass value="0.1"/>
+        <inertia ixx="0.001" ixy="0.0" ixz="0.0"
+                iyy="0.001" iyz="0.0"
+                izz="0.001"/>
+    </inertial>
+    </link>
+    <!-- Joint Screen Sup -->
+    <joint name="screen_sup_joint" type="fixed">
+        <parent link="base_l3_s1"/>
+        <child link="screen_sup"/>
+        <origin xyz="0 0 0" rpy="0 0 0"/>
+    </joint>
+    <!-- Link Screen Sup  -->
+    <link name="screen">
+    <visual>
+        <origin xyz="0 0 0" rpy="${pi_4} 0 ${pi_2}"/>
+        <geometry>
+        <mesh filename="package://orion_description/meshes/screen_il9225.stl"
+            scale="0.001 0.001 0.001"/>
+        </geometry>
+        <material name="DriverRed"/>
+    </visual>
+    <collision>
+        <origin xyz="0 0 0" rpy="${pi_4} 0 ${pi_2}"/>
+        <geometry>
+        <mesh filename="package://orion_description/meshes/screen_il9225.stl"
+            scale="0.001 0.001 0.001"/>
+        </geometry>
+    </collision>
+    <inertial>
+        <origin xyz="0 0 0" rpy="${pi_4} 0 ${pi_2}"/>
+        <mass value="0.1"/>
+        <inertia ixx="0.001" ixy="0.0" ixz="0.0"
+                iyy="0.001" iyz="0.0"
+                izz="0.001"/>
+    </inertial>
+    </link>
+    <!-- Joint Screen Sup -->
+    <joint name="screen_joint" type="fixed">
+        <parent link="screen_sup"/>
+        <child link="screen"/>
+        <origin xyz="0.0275 0 0.0525" rpy="0 0 0"/>
+    </joint>
 </robot>

File: orion_description/urdf/orion_macros.urdf.xacro (robot description, xacro)
@@ -775,5 +775,5 @@
         </xacro:if>
         <!-- Link -->
-        <link name="wall${id}_${level}_${side}">
+        <link name="wall_${id}_${level}_${side}">
         <visual>
             <origin xyz="0 0 0" rpy="0 0 ${pi}"/>
@@ -799,7 +799,7 @@
         </inertial>
         </link>
-        <joint name="wall${id}_${level}_${side}_joint" type="fixed">
+        <joint name="wall_${id}_${level}_${side}_joint" type="fixed">
         <parent link="${parent}"/>
-        <child link="wall${id}_${level}_${side}"/>
+        <child link="wall_${id}_${level}_${side}"/>
         <origin xyz="${x} ${(y+0.00075)*muls} ${z}" rpy="0 0 0"/>
         </joint>
@@ -814,5 +814,5 @@
         </xacro:if>
         <!-- Link -->
-        <link name="wall${id}_${level}_${front}">
+        <link name="wall_${id}_${level}_${front}">
         <visual>
             <origin xyz="0 0 0" rpy="0 0 ${pi_2 + orz}"/>
@@ -838,7 +838,7 @@
         </inertial>
         </link>
-        <joint name="wall${id}_${level}_${front}_joint" type="fixed">
+        <joint name="wall_${id}_${level}_${front}_joint" type="fixed">
         <parent link="${parent}"/>
-        <child link="wall${id}_${level}_${front}"/>
+        <child link="wall_${id}_${level}_${front}"/>
         <origin xyz="${(x+0.00075)*mulf} 0 ${z}" rpy="0 0 0"/>
         </joint>

File: orion_description/urdf/orion_materials.urdf.xacro (robot description, xacro)
@@ -32,5 +32,5 @@
     <!-- Equivalent to RGB(39, 39, 39) -->
     <material name="TransparentBlack">
-        <color rgba="0.3 0.3 0.3 0.8"/>
+        <color rgba="0.3 0.3 0.3 1.0"/>
     </material>
     <!-- Equivalent to RGB(141, 141, 141) -->

Commit message: Description: Added physicks (mass and inertia) to all links

File: orion_description/urdf/orion_base.urdf.xacro (robot description, xacro)
@@ -70,8 +70,8 @@
     <inertial>
         <origin xyz="0 0 0" rpy="0 0 ${pi_2}"/>
-        <mass value="0.1"/>
-        <inertia ixx="0.001" ixy="0.0" ixz="0.0"
-                iyy="0.001" iyz="0.0"
-                izz="0.001"/>
+        <mass value="0.018"/>
+        <inertia ixx="1.2564374999999998e-05" ixy="0.0" ixz="0.0"
+                iyy="2.6539499999999996e-05" iyz="0.0"
+                izz="3.9091874999999996e-05"/>
     </inertial>
     </link>
@@ -91,5 +91,5 @@
         y="0.031351" z="0.0025"/>
     <!-- Link Motor Driver-->
-    <link name="driver_platform">
+    <link name="driver">
     <visual>
         <origin xyz="0 0 0" rpy="0 0 0"/>
@@ -109,14 +109,14 @@
     <inertial>
         <origin xyz="0 0 0" rpy="0 0 0"/>
-        <mass value="0.1"/>
-        <inertia ixx="0.001" ixy="0.0" ixz="0.0"
-                iyy="0.001" iyz="0.0"
-                izz="0.001"/>
+        <mass value="0.026"/>
+        <inertia ixx="5.575206798350021e-06" ixy="0.0" ixz="0.0"
+                iyy="5.588291024131272e-06" iyz="0.0"
+                izz="8.062726989147962e-06"/>
     </inertial>
     </link>
     <!-- Joint Motor Driver -->
-    <joint name="driver_platform" type="fixed">
+    <joint name="driver" type="fixed">
         <parent link="base_l0_s2"/>
-        <child link="driver_platform"/>
+        <child link="driver"/>
         <origin xyz="-0.023453 0.031351 0.0125" rpy="0 0 0"/>
     </joint>
@@ -140,8 +140,8 @@
     <inertial>
         <origin xyz="0 0 0" rpy="0 0 ${-pi_2}"/>
-        <mass value="0.1"/>
-        <inertia ixx="0.001" ixy="0.0" ixz="0.0"
-                iyy="0.001" iyz="0.0"
-                izz="0.001"/>
+        <mass value="0.010"/>
+        <inertia ixx="2.0760416666666664e-06" ixy="0.0" ixz="0.0"
+                iyy="5.797708333333332e-06" iyz="0.0"
+                izz="3.872083333333333e-06"/>
     </inertial>
     </link>
@@ -171,8 +171,8 @@
     <inertial>
         <origin xyz="0 0 0" rpy="${pi_2} 0 ${-pi_2}"/>
-        <mass value="0.1"/>
-        <inertia ixx="0.001" ixy="0.0" ixz="0.0"
-                iyy="0.001" iyz="0.0"
-                izz="0.001"/>
+        <mass value="0.025"/>
+        <inertia ixx="3.4813802083333333e-06" ixy="0.0" ixz="0.0"
+                iyy="9.114713541666667e-06" iyz="0.0"
+                izz="1.1970833333333332e-05"/>
     </inertial>
     </link>
@@ -186,5 +186,5 @@
     <link name="switch">
     <visual>
-        <origin xyz="0 0 0" rpy="${pi/2} 0 ${pi/2}"/>
+        <origin xyz="0 0 0" rpy="${pi_2} 0 ${pi_2}"/>
         <geometry>
         <mesh filename="package://orion_description/meshes/switch_3s_15a.stl"
@@ -194,5 +194,5 @@
     </visual>
     <collision>
-        <origin xyz="0 0 0" rpy="${pi/2} 0 ${pi/2}"/>
+        <origin xyz="0 0 0" rpy="${pi_2} 0 ${pi_2}"/>
         <geometry>
         <mesh filename="package://orion_description/meshes/switch_3s_15a.stl"
@@ -201,9 +201,9 @@
     </collision>
     <inertial>
-        <origin xyz="0 0 0" rpy="${pi/2} 0 ${pi/2}"/>
-        <mass value="0.1"/>
-        <inertia ixx="0.001" ixy="0.0" ixz="0.0"
-                iyy="0.001" iyz="0.0"
-                izz="0.001"/>
+        <origin xyz="0 0 0" rpy="${pi_2} 0 ${pi_2}"/>
+        <mass value="0.0586"/>
+        <inertia ixx="2.0657530893410246e-05" ixy="0.0" ixz="0.0"
+                iyy="1.8508864831011573e-05" iyz="0.0"
+                izz="6.875354057755155e-06"/>
     </inertial>
     </link>
@@ -246,8 +246,8 @@
     <inertial>
         <origin xyz="0 0 0" rpy="${pi} 0 0"/>
-        <mass value="0.1"/>
-        <inertia ixx="0.001" ixy="0.0" ixz="0.0"
-                iyy="0.001" iyz="0.0"
-                izz="0.001"/>
+        <mass value="0.030"/>
+        <inertia ixx="1.1184306270694732e-05" ixy="0.0" ixz="0.0"
+                iyy="1.021680627069473e-05" iyz="0.0"
+                izz="2.0812499999999994e-05"/>
     </inertial>
     </link>
@@ -277,8 +277,8 @@
     <inertial>
         <origin xyz="0 0 0" rpy="${pi} 0 ${-pi_2}"/>
-        <mass value="0.1"/>
-        <inertia ixx="0.001" ixy="0.0" ixz="0.0"
-                iyy="0.001" iyz="0.0"
-                izz="0.001"/>
+        <mass value="0.0201"/>
+        <inertia ixx="4.904162034278915e-06" ixy="0.0" ixz="0.0"
+                iyy="1.5830928543782435e-06" iyz="0.0"
+                izz="6.0040505352397235e-06"/>
     </inertial>
     </link>
@@ -309,9 +309,9 @@
     </collision>
     <inertial>
-        <origin xyz="0 0 0" rpy="0 0 0"/>
-        <mass value="0.1"/>
-        <inertia ixx="0.001" ixy="0.0" ixz="0.0"
-                iyy="0.001" iyz="0.0"
-                izz="0.001"/>
+        <origin xyz="0 0 0" rpy="0 0 ${pi}"/>
+        <mass value="0.047"/>
+        <inertia ixx="1.3696192839509037e-05" ixy="0.0" ixz="0.0"
+                iyy="1.6724159273229613e-05" iyz="0.0"
+                izz="1.981213921926534e-05"/>
     </inertial>
     </link>
@@ -341,8 +341,8 @@
     <inertial>
         <origin xyz="0 0 0" rpy="0 0 ${pi}"/>
-        <mass value="0.1"/>
-        <inertia ixx="0.001" ixy="0.0" ixz="0.0"
-                iyy="0.001" iyz="0.0"
-                izz="0.001"/>
+        <mass value="0.01"/>
+        <inertia ixx="1.4388020833333332e-06" ixy="0.0" ixz="0.0"
+                iyy="3.713020833333333e-07" iyz="0.0"
+                izz="1.7341666666666667e-06"/>
     </inertial>
     </link>
@@ -404,8 +404,8 @@
         <inertial>
             <origin xyz="0 0 0" rpy="0 0 ${-pi_2}"/>
-            <mass value="0.1"/>
-            <inertia ixx="0.001" ixy="0.0" ixz="0.0"
-                    iyy="0.001" iyz="0.0"
-                    izz="0.001"/>
+            <mass value="0.0891"/>
+            <inertia ixx="2.2075679430880743e-05" ixy="0.0" ixz="0.0"
+                    iyy="6.239156111823016e-05" iyz="0.0"
+                    izz="5.4111982712956106e-05"/>
         </inertial>
         </link>
@@ -447,8 +447,8 @@
     <inertial>
         <origin xyz="0 0 0" rpy="0 0 ${-pi_2}"/>
-        <mass value="0.1"/>
-        <inertia ixx="0.001" ixy="0.0" ixz="0.0"
-                iyy="0.001" iyz="0.0"
-                izz="0.001"/>
+        <mass value="0.046"/>
+        <inertia ixx="1.3894925828259282e-05" ixy="0.0" ixz="0.0"
+                iyy="3.130518601304774e-05" iyz="0.0"
+                izz="4.278463267464035e-05"/>
     </inertial>
     </link>
@@ -486,8 +486,8 @@
     <inertial>
         <origin xyz="0 0 0" rpy="0 0 ${pi_2}"/>
-        <mass value="0.1"/>
-        <inertia ixx="0.001" ixy="0.0" ixz="0.0"
-                iyy="0.001" iyz="0.0"
-                izz="0.001"/>
+        <mass value="0.064"/>
+        <inertia ixx="0.00010683527996134758" ixy="0.0" ixz="0.0"
+                iyy="0.0002715" iyz="0.0"
+                izz="0.0003057352799613475"/>
     </inertial>
     </link>
@@ -517,8 +517,8 @@
     <inertial>
         <origin xyz="0 0 0" rpy="${pi_4} 0 ${pi_2}"/>
-        <mass value="0.1"/>
-        <inertia ixx="0.001" ixy="0.0" ixz="0.0"
-                iyy="0.001" iyz="0.0"
-                izz="0.001"/>
+        <mass value="0.0549"/>
+        <inertia ixx="7.3348232666702275e-06" ixy="0.0" ixz="0.0"
+                iyy="1.847275287121583e-05" iyz="0.0"
+                izz="2.4489976137886056e-05"/>
     </inertial>
     </link>

File: orion_description/urdf/orion_cameras.urdf.xacro (robot description, xacro)
@@ -23,8 +23,8 @@
         <inertial>
             <origin xyz="0 0 0" rpy="0 0 ${pi_2}"/>
-            <mass value="0.1"/>
-            <inertia ixx="0.001" ixy="0.0" ixz="0.0"
-                    iyy="0.001" iyz="0.0"
-                    izz="0.001"/>
+            <mass value="0.310"/>
+            <inertia ixx="0.0001453125" ixy="0.0" ixz="0.0"
+                    iyy="0.0007542674781328592" iyz="0.0"
+                    izz="0.0007949549781328593"/>
         </inertial>
         </link>
@@ -57,8 +57,8 @@
         <inertial>
             <origin xyz="0 0 0" rpy="0 0 ${pi_2}"/>
-            <mass value="0.1"/>
-            <inertia ixx="0.001" ixy="0.0" ixz="0.0"
-                    iyy="0.001" iyz="0.0"
-                    izz="0.001"/>
+            <mass value="0.006"/>
+            <inertia ixx="5.791913396592736e-07" ixy="0.0" ixz="0.0"
+                    iyy="1.992091044590605e-06" iyz="0.0"
+                    izz="1.6121002950686689e-06"/>
         </inertial>
         </link>
@@ -88,8 +88,8 @@
         <inertial>
             <origin xyz="0 0 0" rpy="0 0 ${pi_2}"/>
-            <mass value="0.1"/>
-            <inertia ixx="0.001" ixy="0.0" ixz="0.0"
-                    iyy="0.001" iyz="0.0"
-                    izz="0.001"/>
+            <mass value="0.096"/>
+            <inertia ixx="9.999999999999999e-06" ixy="0.0" ixz="0.0"
+                    iyy="6.979999999999999e-05" iyz="0.0"
+                    izz="6.979999999999999e-05"/>
         </inertial>
         </link>
@@ -122,8 +122,8 @@
         <inertial>
             <origin xyz="0 0 0" rpy="0 0 ${pi_2}"/>
-            <mass value="0.1"/>
-            <inertia ixx="0.001" ixy="0.0" ixz="0.0"
-                    iyy="0.001" iyz="0.0"
-                    izz="0.001"/>
+            <mass value="0.002"/>
+            <inertia ixx="6.15e-08" ixy="0.0" ixz="0.0"
+                    iyy="1.4166666666666665e-07" iyz="0.0"
+                    izz="1.2816666666666664e-07"/>
         </inertial>
         </link>
@@ -153,8 +153,8 @@
         <inertial>
             <origin xyz="0 0 0" rpy="${pi_2} 0 ${pi_2}"/>
-            <mass value="0.1"/>
-            <inertia ixx="0.001" ixy="0.0" ixz="0.0"
-                    iyy="0.001" iyz="0.0"
-                    izz="0.001"/>
+            <mass value="0.01"/>
+            <inertia ixx="1.4708639141126087e-06" ixy="0.0" ixz="0.0"
+                    iyy="7.106770833333332e-07" iyz="0.0"
+                    izz="1.997790997445942e-06"/>
         </inertial>
         </link>
