Commit message: Description: Added physicks (mass and inertia) to all links

File: orion_description/urdf/orion_macros.urdf.xacro (robot description, xacro)
@@ -1,94 +1,4 @@
 <?xml version="1.0"?>
 <robot xmlns:xacro="http://www.ros.org/wiki/xacro">
-    <!-- Macro for adding two symmetrical spacers -->
-    <xacro:macro name="symmetrical_spacers"
-                params="name parent base_position offset_from_position mesh_file
-                        scale:=1.0 rpy:='0 0 0'">
-        <!-- Left Spacer -->
-        <link name="${name}_left">
-        <visual>
-            <geometry>
-            <mesh filename="${mesh_file}" scale="${scale} ${scale} ${scale}"/>
-            </geometry>
-        </visual>
-        </link>
-        <joint name="${name}_left_joint" type="fixed">
-        <parent link="${parent}"/>
-        <child link="${name}_left"/>
-        <origin xyz="${base_position[0] - offset_from_position} ${base_position[1]} ${base_position[2]}"
-                rpy="${rpy}"/>
-        </joint>
-        <!-- Right Spacer -->
-        <link name="${name}_right">
-        <visual>
-            <geometry>
-            <mesh filename="${mesh_file}" scale="${scale} ${scale} ${scale}"/>
-            </geometry>
-        </visual>
-        </link>
-        <joint name="${name}_right_joint" type="fixed">
-        <parent link="${parent}"/>
-        <child link="${name}_right"/>
-        <origin xyz="${base_position[0] + offset_from_position} ${base_position[1]} ${base_position[2]}"
-                rpy="${rpy}"/>
-        </joint>
-    </xacro:macro>
-    <!-- Macro for adding four symmetrical spacers -->
-    <xacro:macro name="four_symmetrical_spacers"
-                params="name parent origin offset_x offset_y mesh_file
-                        scale:=1.0 rpy:='0 0 0'">
-        <!-- Front-Left Spacer -->
-        <link name="${name}_front_left">
-        <visual>
-            <geometry>
-            <mesh filename="${mesh_file}" scale="${scale} ${scale} ${scale}"/>
-            </geometry>
-        </visual>
-        </link>
-        <joint name="${name}_front_left_joint" type="fixed">
-        <parent link="${parent}"/>
-        <child link="${name}_front_left"/>
-        <origin xyz="${origin[0] - offset_x} ${origin[1] + offset_y} ${origin[2]}" rpy="${rpy}"/>
-        </joint>
-        <!-- Front-Right Spacer -->
-        <link name="${name}_front_right">
-        <visual>
-            <geometry>
-            <mesh filename="${mesh_file}" scale="${scale} ${scale} ${scale}"/>
-            </geometry>
-        </visual>
-        </link>
-        <joint name="${name}_front_right_joint" type="fixed">
-        <parent link="${parent}"/>
-        <child link="${name}_front_right"/>
-        <origin xyz="${origin[0] + offset_x} ${origin[1] + offset_y} ${origin[2]}" rpy="${rpy}"/>
-        </joint>
-        <!-- Back-Left Spacer -->
-        <link name="${name}_back_left">
-        <visual>
-            <geometry>
-            <mesh filename="${mesh_file}" scale="${scale} ${scale} ${scale}"/>
-            </geometry>
-        </visual>
-        </link>
-        <joint name="${name}_back_left_joint" type="fixed">
-        <parent link="${parent}"/>
-        <child link="${name}_back_left"/>
-        <origin xyz="${origin[0] - offset_x} ${origin[1] - offset_y} ${origin[2]}" rpy="${rpy}"/>
-        </joint>
-        <!-- Back-Right Spacer -->
-        <link name="${name}_back_right">
-        <visual>
-            <geometry>
-            <mesh filename="${mesh_file}" scale="${scale} ${scale} ${scale}"/>
-            </geometry>
-        </visual>
-        </link>
-        <joint name="${name}_back_right_joint" type="fixed">
-        <parent link="${parent}"/>
-        <child link="${name}_back_right"/>
-        <origin xyz="${origin[0] + offset_x} ${origin[1] - offset_y} ${origin[2]}" rpy="${rpy}"/>
-        </joint>
-    </xacro:macro>
     <!--//////////////////// MATH AND NUMS MACROS ///////////////////////-->
     <xacro:property name="pi_2" value="${pi / 2}"/>
@@ -136,9 +46,9 @@
         </collision>
         <inertial>
-            <origin xyz="0 0 0"/>
-            <mass value="0.0053"/>
-            <inertia ixx="0.001" ixy="0.0" ixz="0.0"
-                    iyy="0.001" iyz="0.0"
-                    izz="0.001"/>
+            <origin xyz="0 0 0" rpy="0 0 ${gyro}"/>
+            <mass value="0.012"/>
+            <inertia ixx="6.799999999999999e-06" ixy="0.0" ixz="0.0"
+                    iyy="6.799999999999999e-06" iyz="0.0"
+                    izz="8e-07"/>
         </inertial>
         </link>
@@ -181,8 +91,8 @@
         <inertial>
             <origin xyz="0 0 0" rpy="0 0 ${mul*pi_2}"/>
-            <mass value="0.1"/>
-            <inertia ixx="0.001" ixy="0.0" ixz="0.0"
-                    iyy="0.001" iyz="0.0"
-                    izz="0.001"/>
+            <mass value="0.053"/>
+            <inertia ixx="5.843802083333332e-05" ixy="0.0" ixz="0.0"
+                    iyy="0.00019480260416666664" iyz="0.0"
+                    izz="0.0002531854166666666"/>
         </inertial>
         </link>
@@ -199,34 +109,4 @@
         <xacro:half_base level="${level}" side="2" parent="base_link" x="${x}"
             y="${y}" z="${z}"/>
-    </xacro:macro>
-    <xacro:macro name="generic_sphere" params="name parent x y z">
-    <!-- Link -->
-        <link name="${name}">
-        <visual>
-            <origin xyz="0 0 0" rpy="0 0 0"/>
-            <geometry>
-                <sphere radius="0.005"/>
-            </geometry>
-        </visual>
-        <collision>
-            <origin xyz="0 0 0" rpy="0 0 0"/>
-            <geometry>
-                <sphere radius="0.005"/>
-            </geometry>
-        </collision>
-        <inertial>
-            <origin xyz="${x} ${y} ${z}"/>
-            <mass value="0.1"/>
-            <inertia ixx="0.001" ixy="0.0" ixz="0.0"
-                    iyy="0.001" iyz="0.0"
-                    izz="0.001"/>
-        </inertial>
-        </link>
-        <!-- Fixed Joint -->
-        <joint name="${name}_joint" type="fixed">
-        <parent link="${parent}"/>
-        <child link="${name}"/>
-        <origin xyz="${x} ${y} ${z}" rpy="0 0 0"/>
-        </joint>
     </xacro:macro>
     <!--  /////////////////// MOTOR DC MACROS ///////////////////////////////-->
@@ -262,9 +142,9 @@
         </collision>
         <inertial>
-            <origin xyz="0 0 0"/>
-            <mass value="0.0053"/>
-            <inertia ixx="0.001" ixy="0.0" ixz="0.0"
-                    iyy="0.001" iyz="0.0"
-                    izz="0.001"/>
+            <origin xyz="0 0 0" rpy="${pi} 0 ${orin}"/>
+            <mass value="0.011753"/>
+            <inertia ixx="2.1329054208642935e-06" ixy="0.0" ixz="0.0"
+                    iyy="1.7437733457263675e-06" iyz="0.0"
+                    izz="1.7440374248620737e-06"/>
         </inertial>
         </link>
@@ -293,9 +173,9 @@
         </collision>
         <inertial>
-            <origin xyz="0 0 0"/>
-            <mass value="0.0053"/>
-            <inertia ixx="0.001" ixy="0.0" ixz="0.0"
-                    iyy="0.001" iyz="0.0"
-                    izz="0.001"/>
+            <origin xyz="0 0 0" rpy="${-pi_2*muls} 0 0"/>
+            <mass value="0.099"/>
+            <inertia ixx="5.612122306673401e-05" ixy="0.0" ixz="0.0"
+                    iyy="5.6124427915649726e-05" iyz="0.0"
+                    izz="1.0309295151084287e-05"/>
         </inertial>
         </link>
@@ -324,9 +204,9 @@
         </collision>
         <inertial>
-            <origin xyz="0 0 0"/>
-            <mass value="0.0053"/>
-            <inertia ixx="0.001" ixy="0.0" ixz="0.0"
-                    iyy="0.001" iyz="0.0"
-                    izz="0.001"/>
+            <origin xyz="0 0 0" rpy="${orin} 0 ${pi_6*muls}"/>
+            <mass value="0.0152"/>
+            <inertia ixx="6.244666666666666e-07" ixy="0.0" ixz="0.0"
+                    iyy="6.958222391764178e-07" iyz="0.0"
+                    izz="4.994889058430845e-07"/>
         </inertial>
         </link>
@@ -356,9 +236,9 @@
         </collision>
         <inertial>
-            <origin xyz="0 0 0"/>
-            <mass value="0.0053"/>
-            <inertia ixx="0.001" ixy="0.0" ixz="0.0"
-                    iyy="0.001" iyz="0.0"
-                    izz="0.001"/>
+            <origin xyz="0 0 0" rpy="0 ${-pi_2*muls} 0"/>
+            <mass value="0.0109"/>
+            <inertia ixx="4.816756860757923e-06" ixy="0.0" ixz="0.0"
+                    iyy="2.9882463541666663e-06" iyz="0.0"
+                    izz="2.9867490482579234e-06"/>
         </inertial>
         </link>
@@ -387,9 +267,9 @@
         </collision>
         <inertial>
-            <origin xyz="0 0 0"/>
-            <mass value="0.0053"/>
-            <inertia ixx="0.001" ixy="0.0" ixz="0.0"
-                    iyy="0.001" iyz="0.0"
-                    izz="0.001"/>
+            <origin xyz="0 0 0" rpy="0 ${pi_2*muls} 0"/>
+            <mass value="0.0399"/>
+            <inertia ixx="3.15394093727487e-05" ixy="0.0" ixz="0.0"
+                    iyy="1.7872841935074492e-05" iyz="0.0"
+                    izz="1.7872841935074492e-05"/>
         </inertial>
         </link>
@@ -421,9 +301,9 @@
         </collision>
         <inertial>
-            <origin xyz="0 0 0"/>
-            <mass value="0.0053"/>
-            <inertia ixx="0.001" ixy="0.0" ixz="0.0"
-                    iyy="0.001" iyz="0.0"
-                    izz="0.001"/>
+            <origin xyz="0 0 0" rpy="${pi} 0 ${pi_2}"/>
+            <mass value="0.01085"/>
+            <inertia ixx="9.360136765056053e-07" ixy="0.0" ixz="0.0"
+                    iyy="1.315763414372338e-06" iyz="0.0"
+                    izz="2.2314830712000656e-06"/>
         </inertial>
         </link>
@@ -452,9 +332,9 @@
         </collision>
         <inertial>
-            <origin xyz="0 0 0"/>
-            <mass value="0.0053"/>
-            <inertia ixx="0.001" ixy="0.0" ixz="0.0"
-                    iyy="0.001" iyz="0.0"
-                    izz="0.001"/>
+            <origin xyz="0 0 0" rpy="0 0 ${-pi_2}"/>
+            <mass value="0.01633"/>
+            <inertia ixx="1.6321007868011535e-06" ixy="0.0" ixz="0.0"
+                    iyy="1.3901075509910613e-06" iyz="0.0"
+                    izz="1.644364587792215e-06"/>
         </inertial>
         </link>
@@ -484,9 +364,9 @@
         </collision>
         <inertial>
-            <origin xyz="0 0 0"/>
-            <mass value="0.0053"/>
-            <inertia ixx="0.001" ixy="0.0" ixz="0.0"
-                    iyy="0.001" iyz="0.0"
-                    izz="0.001"/>
+            <origin xyz="0 0 0" rpy="${pi_2} 0 0"/>
+            <mass value="0.00794"/>
+            <inertia ixx="5.723473258925721e-07" ixy="0.0" ixz="0.0"
+                    iyy="8.268436933141506e-07" iyz="0.0"
+                    izz="5.724272007549117e-07"/>
         </inertial>
         </link>
@@ -530,8 +410,8 @@
         <inertial>
             <origin xyz="0 0 0"/>
-            <mass value="0.0053"/>
-            <inertia ixx="0.001" ixy="0.0" ixz="0.0"
-                    iyy="0.001" iyz="0.0"
-                    izz="0.001"/>
+            <mass value="0.048"/>
+            <inertia ixx="1.9520194552672923e-06" ixy="0.0" ixz="0.0"
+                    iyy="1.9520999999999995e-06" iyz="0.0"
+                    izz="2.5911945526729246e-07"/>
         </inertial>
         </link>
@@ -561,9 +441,9 @@
         </collision>
         <inertial>
-            <origin xyz="0 0 0"/>
-            <mass value="0.0053"/>
-            <inertia ixx="0.001" ixy="0.0" ixz="0.0"
-                    iyy="0.001" iyz="0.0"
-                    izz="0.001"/>
+            <origin xyz="0 0 0" rpy="0 0 ${pi_2}"/>
+            <mass value="0.02012"/>
+            <inertia ixx="1.4044179166666666e-06" ixy="0.0" ixz="0.0"
+                    iyy="2.9665263333333333e-06" iyz="0.0"
+                    izz="4.369602916666666e-06"/>
         </inertial>
         </link>
@@ -611,9 +491,9 @@
         </collision>
         <inertial>
-            <origin xyz="0 0 0"/>
-            <mass value="0.0053"/>
-            <inertia ixx="0.001" ixy="0.0" ixz="0.0"
-                    iyy="0.001" iyz="0.0"
-                    izz="0.001"/>
+            <origin xyz="0 0 0" rpy="${-pi_2} 0 ${flex}"/>
+            <mass value="0.012"/>
+            <inertia ixx="3.1172499999999997e-06" ixy="0.0" ixz="0.0"
+                    iyy="4.2049999999999996e-06" iyz="0.0"
+                    izz="6.60025e-06"/>
         </inertial>
         </link>
@@ -642,9 +522,9 @@
         </collision>
         <inertial>
-            <origin xyz="0 0 0"/>
-            <mass value="0.0053"/>
-            <inertia ixx="0.001" ixy="0.0" ixz="0.0"
-                    iyy="0.001" iyz="0.0"
-                    izz="0.001"/>
+            <origin xyz="0 0 0" rpy="${-pi_2*inv} 0 0"/>
+            <mass value="0.055"/>
+            <inertia ixx="1.1155878535842904e-05" ixy="0.0" ixz="0.0"
+                    iyy="2.1057527828089415e-05" iyz="0.0"
+                    izz="1.3568315958913178e-05"/>
         </inertial>
         </link>
@@ -673,9 +553,9 @@
         </collision>
         <inertial>
-            <origin xyz="0 0 0"/>
-            <mass value="0.0053"/>
-            <inertia ixx="0.001" ixy="0.0" ixz="0.0"
-                    iyy="0.001" iyz="0.0"
-                    izz="0.001"/>
+            <origin xyz="0 0 0" rpy="0 0 0"/>
+            <mass value="0.005"/>
+            <inertia ixx="1.750719658194081e-07" ixy="0.0" ixz="0.0"
+                    iyy="1.750397680831338e-07" iyz="0.0"
+                    izz="3.332367339025419e-07"/>
         </inertial>
         </link>
@@ -722,9 +602,9 @@
         </collision>
         <inertial>
-            <origin xyz="0 0 0"/>
-            <mass value="0.0053"/>
-            <inertia ixx="0.001" ixy="0.0" ixz="0.0"
-                    iyy="0.001" iyz="0.0"
-                    izz="0.001"/>
+            <origin xyz="0 0 0" rpy="0 0 ${inv}"/>
+            <mass value="0.007"/>
+            <inertia ixx="1.402333333333333e-06" ixy="0.0" ixz="0.0"
+                    iyy="2.578333333333333e-06" iyz="0.0"
+                    izz="1.2926666666666665e-06"/>
         </inertial>
         </link>
@@ -735,5 +615,5 @@
             <origin xyz="${x*mulf} ${y*muls} ${z}" rpy="0 0 0"/>
         </joint>
-        <!-- Link speaker support -->
+        <!-- Link speaker -->
         <link name="speaker_${front}${side}">
         <visual>
@@ -753,12 +633,12 @@
         </collision>
         <inertial>
-            <origin xyz="0 0 0"/>
-            <mass value="0.0053"/>
-            <inertia ixx="0.001" ixy="0.0" ixz="0.0"
-                    iyy="0.001" iyz="0.0"
-                    izz="0.001"/>
-        </inertial>
-        </link>
-        <!-- Joint speaker support -->
+            <origin xyz="0 0 0" rpy="0 0 ${inv}"/>
+            <mass value="0.0456"/>
+            <inertia ixx="1.102e-05" ixy="0.0" ixz="0.0"
+                    iyy="1.6081600000000002e-05" iyz="0.0"
+                    izz="1.102e-05"/>
+        </inertial>
+        </link>
+        <!-- Joint speaker -->
         <joint name="speaker_${front}${side}_joint" type="fixed">
             <parent link="speaker_sup_${front}${side}"/>
@@ -792,9 +672,9 @@
         </collision>
         <inertial>
-            <origin xyz="0 0 0"/>
-            <mass value="0.0053"/>
-            <inertia ixx="0.001" ixy="0.0" ixz="0.0"
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
File: orion_description/urdf/orion_materials.urdf.xacro (robot description, xacro)
@@ -32,5 +32,5 @@
     <!-- Equivalent to RGB(39, 39, 39) -->
     <material name="TransparentBlack">
-        <color rgba="0.3 0.3 0.3 1.0"/>
+        <color rgba="0.3 0.3 0.3 0.8"/>
     </material>
     <!-- Equivalent to RGB(141, 141, 141) -->

Commit message: Description: New rsp launch file and minor fixed in URDF

File: orion_description/urdf/orion_base.urdf.xacro (robot description, xacro)
@@ -116,5 +116,5 @@
     </link>
     <!-- Joint Motor Driver -->
-    <joint name="driver" type="fixed">
+    <joint name="driver_joint" type="fixed">
         <parent link="base_l0_s2"/>
         <child link="driver"/>
