Commit message: Description: Changed management of gazebo references

File: orion_description/urdf/orion_base.urdf.xacro (robot description, xacro)
@@ -47,9 +47,9 @@
         z="${-0.002 - 0.017}"/>
     <!-- //////////////// FIRST FLOOR COMPONENTS ///////////////////// -->
-    <!-- Hex spacers for Battery Support -->
+    <!-- .................. Hex spacers for stack .................... -->
     <xacro:x6xmetric_spacer id="m3x10" element="bathol" parent="base_l0_s1"
         offset_x="${0.0855/2}" offset_y="${0.127/2}" x="0.005" y="0"
         z="0.0025"/>
-    <!-- Link Battery Support-->
+    <!-- ..................... Battery Platform ....................... -->
     <link name="bat_platform">
     <visual>
@@ -76,5 +76,4 @@
     </inertial>
     </link>
-    <!-- Joint Battery Support -->
     <joint name="bat_platform_joint" type="fixed">
         <parent link="base_l0_s1"/>
@@ -82,13 +81,19 @@
         <origin xyz="0.005 0 0.0125" rpy="0 0 0"/>
     </joint>
-    <!-- Battery Stacks -->
+    <xacro:if value="${gazebo}">
+        <gazebo reference="bat_platform">
+            <mu1>1.0</mu1>
+            <mu2>1.0</mu2>
+        </gazebo>
+    </xacro:if>
+    <!-- ....................... Battery Stacks ........................ -->
     <xacro:stack_bat parent="bat_platform" num="1" x="0" y="-0.023" z="0"/>
     <xacro:stack_bat parent="bat_platform" num="2" x="0" y="${0.023+0.02}"
         z="0"/>
-    <!-- Hex spacers for Motor Driver-->
+    <!-- ............... Hex spacers for Motor Driver................... -->
     <xacro:x4xmetric_spacer id="m3x10" element="driver" parent="base_l0_s2"
         offset_x="${0.03702/2}" offset_y="${-0.0368/2}" x="-0.023453"
         y="0.031351" z="0.0025"/>
-    <!-- Link Motor Driver-->
+    <!-- ......................... Motor Driver ........................ -->
     <link name="driver">
     <visual>
@@ -115,5 +120,4 @@
     </inertial>
     </link>
-    <!-- Joint Motor Driver -->
     <joint name="driver_joint" type="fixed">
         <parent link="base_l0_s2"/>
@@ -121,5 +125,11 @@
         <origin xyz="-0.023453 0.031351 0.0125" rpy="0 0 0"/>
     </joint>
-    <!-- Link Regulator Support-->
+    <xacro:if value="${gazebo}">
+        <gazebo reference="driver">
+            <mu1>1.0</mu1>
+            <mu2>1.0</mu2>
+        </gazebo>
+    </xacro:if>
+    <!-- ........................ Regulator Support ......................... -->
     <link name="reg_support">
     <visual>
@@ -146,5 +156,4 @@
     </inertial>
     </link>
-    <!-- Joint Regulator Support -->
     <joint name="reg_support_joint" type="fixed">
         <parent link="base_l0_s2"/>
@@ -152,5 +161,11 @@
         <origin xyz="-0.036 -0.0275 0.0025" rpy="0 0 0"/>
     </joint>
-    <!-- Link Regulator Support-->
+    <xacro:if value="${gazebo}">
+        <gazebo reference="reg_support">
+            <mu1>1.0</mu1>
+            <mu2>1.0</mu2>
+        </gazebo>
+    </xacro:if>
+    <!-- ....................... Regulator ............................... -->
     <link name="regulator">
     <visual>
@@ -177,5 +192,4 @@
     </inertial>
     </link>
-    <!-- Joint Regulator -->
     <joint name="reg_joint" type="fixed">
         <parent link="reg_support"/>
@@ -183,5 +197,11 @@
         <origin xyz="-0.0025 0 ${0.06/2}" rpy="0 0 0"/>
     </joint>
-    <!-- Link Switch -->
+    <xacro:if value="${gazebo}">
+        <gazebo reference="regulator">
+            <mu1>1.0</mu1>
+            <mu2>1.0</mu2>
+        </gazebo>
+    </xacro:if>
+    <!-- ......................... Switch ........................... -->
     <link name="switch">
     <visual>
@@ -208,5 +228,4 @@
     </inertial>
     </link>
-    <!-- Joint Switch -->
     <joint name="switch_joint" type="fixed">
         <parent link="base_l1_s1"/>
@@ -214,4 +233,11 @@
         <origin xyz="0.025 0.074 -0.015" rpy="0 0 0"/>
     </joint>
+    <xacro:if value="${gazebo}">
+        <gazebo reference="switch">
+            <mu1>1.0</mu1>
+            <mu2>1.0</mu2>
+        </gazebo>
+    </xacro:if>
+    <!-- ......................... Walls definitions ...................... -->
     <xacro:complete_lateral_wall id="servo" parent="base_l0_s1" side="1"
         x="${-0.115/2}" y="${0.21/2 + 0.0005}" z="${0.082/2 + 0.0025/2}"
@@ -225,7 +251,8 @@
         x="${0.115/2}" z="${0.082/2 + 0.0025/2}" level="0"/>
     <!-- ///////////////// SECOND FLOOR COMPONENTS /////////////////////// -->
+    <!-- ..................... Spacers for esp32 adp ..................... -->
     <xacro:x4xmetric_spacer id="m3x10" element="esp_adapter" parent="base_l1_s1"
         offset_x="${0.0577/2}" offset_y="${0.0607/2}" x="0" y="0" z="-0.01"/>
-    <!-- Link Esp32 Adapter -->
+    <!-- .......................... Esp32 Adapter ....................... -->
     <link name="esp32_adapter">
     <visual>
@@ -252,5 +279,4 @@
     </inertial>
     </link>
-    <!-- Joint Esp32 Adapter -->
     <joint name="esp32_adapter_joint" type="fixed">
         <parent link="base_l1_s1"/>
@@ -258,5 +284,11 @@
         <origin xyz="0 0 -0.01" rpy="0 0 0"/>
     </joint>
-    <!-- Link Esp32 -->
+    <xacro:if value="${gazebo}">
+        <gazebo reference="esp32_adapter">
+            <mu1>1.0</mu1>
+            <mu2>1.0</mu2>
+        </gazebo>
+    </xacro:if>
+    <!-- ....................... ESP32 ....................................... -->
     <link name="esp32">
     <visual>
@@ -283,5 +315,4 @@
     </inertial>
     </link>
-    <!-- Joint Esp32 -->
     <joint name="esp32_joint" type="fixed">
         <parent link="esp32_adapter"/>
@@ -289,7 +320,14 @@
         <origin xyz="0.002 0 -0.01" rpy="0 0 0"/>
     </joint>
+    <xacro:if value="${gazebo}">
+        <gazebo reference="esp32">
+            <mu1>1.0</mu1>
+            <mu2>1.0</mu2>
+        </gazebo>
+    </xacro:if>
+    <!-- .......................... LIDAR spacers .......................... -->
     <xacro:x3xmetric_spacer id="m3x10" element="lidar" parent="base_l1_s1"
         offset_x="0.0234" offset_y="${0.03132/2}" x="-0.0575" y="0" z="0.0025"/>
-    <!-- Link LD19 -->
+    <!-- ............................ LD19 ................................. -->
     <link name="ld19">
     <visual>
@@ -316,5 +354,4 @@
     </inertial>
     </link>
-    <!-- Joint LD19 -->
     <joint name="ld19_joint" type="fixed">
         <parent link="base_l1_s1"/>
@@ -322,5 +359,11 @@
         <origin xyz="${-0.0575} -0.0035 0.0125" rpy="0 0 0"/>
     </joint>
-    <!-- Link Lidar Serial -->
+    <xacro:if value="${gazebo}">
+        <gazebo reference="ld19">
+            <mu1>1.0</mu1>
+            <mu2>1.0</mu2>
+        </gazebo>
+    </xacro:if>
+    <!-- ......................... LIDAR serial .......................... -->
     <link name="lidar_serial">
     <visual>
@@ -347,5 +390,4 @@
     </inertial>
     </link>
-    <!-- Joint Lidar Serial -->
     <joint name="lidar_serial_joint" type="fixed">
         <parent link="base_l1_s2"/>
@@ -353,4 +395,11 @@
         <origin xyz="-0.03 0.025 0.0025" rpy="0 0 0"/>
     </joint>
+    <xacro:if value="${gazebo}">
+        <gazebo reference="lidar_serial">
+            <mu1>1.0</mu1>
+            <mu2>1.0</mu2>
+        </gazebo>
+    </xacro:if>
+    <!-- ....................... Servo Definitions ........................ -->
     <xacro:if value="${servo}">
         <xacro:servo_mounted parent="base_l1_s2" side="1" x="0.00275" y="0.0765"
@@ -359,4 +408,5 @@
             z="-0.026"/>
     </xacro:if>
+    <!-- ......................... Wall definitions ........................ -->
     <xacro:complete_lateral_wall id="llidar" parent="base_l1_s1" side="1"
         x="${-0.115/2}" y="${0.21/2 + 0.0005}" z="${0.082/2 + 0.0025/2}"
@@ -385,30 +435,29 @@
     </xacro:if>
     <xacro:if value="${rasp == 'rpi5'}">
-        <!-- Link Stereo Speaker  -->
+        <!-- ....................... Stereo Speaker ............................. -->
         <link name="stereo">
-        <visual>
-            <origin xyz="0 0 0" rpy="0 0 ${-pi_2}"/>
-            <geometry>
-            <mesh filename="package://orion_description/meshes/speaker_stereo.stl"
-                scale="0.001 0.001 0.001"/>
-            </geometry>
-            <material name="SoftBlack"/>
-        </visual>
-        <collision>
-            <origin xyz="0 0 0" rpy="0 0 ${-pi_2}"/>
-            <geometry>
-            <mesh filename="package://orion_description/meshes/speaker_stereo.stl"
-                scale="0.001 0.001 0.001"/>
-            </geometry>
-        </collision>
-        <inertial>
-            <origin xyz="0 0 0" rpy="0 0 ${-pi_2}"/>
-            <mass value="0.0891"/>
-            <inertia ixx="2.2075679430880743e-05" ixy="0.0" ixz="0.0"
-                    iyy="6.239156111823016e-05" iyz="0.0"
-                    izz="5.4111982712956106e-05"/>
-        </inertial>
+            <visual>
+                <origin xyz="0 0 0" rpy="0 0 ${-pi_2}"/>
+                <geometry>
+                <mesh filename="package://orion_description/meshes/speaker_stereo.stl"
+                    scale="0.001 0.001 0.001"/>
+                </geometry>
+                <material name="SoftBlack"/>
+            </visual>
+            <collision>
+                <origin xyz="0 0 0" rpy="0 0 ${-pi_2}"/>
+                <geometry>
+                <mesh filename="package://orion_description/meshes/speaker_stereo.stl"
+                    scale="0.001 0.001 0.001"/>
+                </geometry>
+            </collision>
+            <inertial>
+                <origin xyz="0 0 0" rpy="0 0 ${-pi_2}"/>
+                <mass value="0.0891"/>
+                <inertia ixx="2.2075679430880743e-05" ixy="0.0" ixz="0.0"
+                        iyy="6.239156111823016e-05" iyz="0.0"
+                        izz="5.4111982712956106e-05"/>
+            </inertial>
         </link>
-        <!-- Joint Stereo Speaker -->
         <joint name="stereo_joint" type="fixed">
             <parent link="base_l2_s2"/>
@@ -416,4 +465,11 @@
             <origin xyz="-0.02 0 0.025" rpy="0 0 0"/>
         </joint>
+        <xacro:if value="${gazebo}">
+            <gazebo reference="stereo">
+                <mu1>1.0</mu1>
+                <mu2>1.0</mu2>
+            </gazebo>
+        </xacro:if>
+        <!-- ........................ Wall definitions ...................... -->
         <xacro:complete_lateral_wall id="curve" parent="base_l2_s1" side="1"
             x="${-0.115/2}" y="${0.21/2 + 0.0005}" z="${0.082/2 + 0.0025/2}"
@@ -453,5 +509,4 @@
     </inertial>
     </link>
-    <!-- Joint Rasberry Pi-->
     <joint name="${rasp}_joint" type="fixed">
         <parent link="base_l3_s2"/>
@@ -459,4 +514,11 @@
         <origin xyz="0 0.0335 0.0125" rpy="0 0 0"/>
     </joint>
+    <xacro:if value="${gazebo}">
+        <gazebo reference="${rasp}">
+            <mu1>1.0</mu1>
+            <mu2>1.0</mu2>
+        </gazebo>
+    </xacro:if>
+    <!-- ......................... Walls definitions ............................ -->
     <xacro:complete_lateral_wall id="screen" parent="base_l3_s1" side="1"
             x="${-0.115/2 + 0.005}" y="${0.21/2 + 0.0005}" z="${0.082/2 + 0.0025/2}"
@@ -467,5 +529,5 @@
     <xacro:complete_front_wall id="rpi" parent="base_l3_s2" front="2"
         x="${0.115/2}" z="${0.082/2 + 0.0025/2}" level="3"/>
-    <!-- Link Screen Sup  -->
+    <!-- .......................... Screen Sup ................................ -->
     <link name="screen_sup">
     <visual>
@@ -492,5 +554,4 @@
     </inertial>
     </link>
-    <!-- Joint Screen Sup -->
     <joint name="screen_sup_joint" type="fixed">
         <parent link="base_l3_s1"/>
@@ -498,5 +559,11 @@
         <origin xyz="0 0 0" rpy="0 0 0"/>
     </joint>
-    <!-- Link Screen Sup  -->
+    <xacro:if value="${gazebo}">
+        <gazebo reference="screen_sup">
+            <mu1>1.0</mu1>
+            <mu2>1.0</mu2>
+        </gazebo>
+    </xacro:if>
+    <!-- ...................... Screen Sup ................................. -->
     <link name="screen">
     <visual>
@@ -523,5 +590,4 @@
     </inertial>
     </link>
-    <!-- Joint Screen Sup -->
     <joint name="screen_joint" type="fixed">
         <parent link="screen_sup"/>
@@ -529,3 +595,9 @@
         <origin xyz="0.0275 0 0.0525" rpy="0 0 0"/>
     </joint>
+    <xacro:if value="${gazebo}">
+        <gazebo reference="screen">
+            <mu1>1.0</mu1>
+            <mu2>1.0</mu2>
+        </gazebo>
+    </xacro:if>
 </robot>

File: orion_description/urdf/orion_gz.urdf.xacro (robot description, xacro)
@@ -1,488 +1,4 @@
 <?xml version="1.0"?>
 <robot xmlns:xacro="http://www.ros.org/wiki/xacro">
-    <gazebo reference="accel">
-        <mu1>1.0</mu1>
-        <mu2>1.0</mu2>
-    </gazebo>
-    <gazebo reference="accel_base">
-        <mu1>1.0</mu1>
-        <mu2>1.0</mu2>
-    </gazebo>
-    <gazebo reference="b18650_1_1">
-        <mu1>1.0</mu1>
-        <mu2>1.0</mu2>
-    </gazebo>
-    <gazebo reference="b18650_1_2">
-        <mu1>1.0</mu1>
-        <mu2>1.0</mu2>
-    </gazebo>
-    <gazebo reference="b18650_1_3">
-        <mu1>1.0</mu1>
-        <mu2>1.0</mu2>
-    </gazebo>
-    <gazebo reference="b18650_2_1">
-        <mu1>1.0</mu1>
-        <mu2>1.0</mu2>
-    </gazebo>
-    <gazebo reference="b18650_2_2">
-        <mu1>1.0</mu1>
-        <mu2>1.0</mu2>
-    </gazebo>
-    <gazebo reference="b18650_2_3">
-        <mu1>1.0</mu1>
-        <mu2>1.0</mu2>
-    </gazebo>
-    <gazebo reference="base_l0_s1">
-        <mu1>1.0</mu1>
-        <mu2>1.0</mu2>
-    </gazebo>
-    <gazebo reference="base_l0_s2">
-        <mu1>1.0</mu1>
-        <mu2>1.0</mu2>
-    </gazebo>
-    <gazebo reference="base_l1_s1">
-        <mu1>1.0</mu1>
-        <mu2>1.0</mu2>
-    </gazebo>
-    <gazebo reference="base_l1_s2">
-        <mu1>1.0</mu1>
-        <mu2>1.0</mu2>
-    </gazebo>
-    <gazebo reference="base_l2_s1">
-        <mu1>1.0</mu1>
-        <mu2>1.0</mu2>
-    </gazebo>
-    <gazebo reference="base_l2_s2">
-        <mu1>1.0</mu1>
-        <mu2>1.0</mu2>
-    </gazebo>
-    <gazebo reference="base_l3_s1">
-        <mu1>1.0</mu1>
-        <mu2>1.0</mu2>
-    </gazebo>
-    <gazebo reference="base_l3_s2">
-        <mu1>1.0</mu1>
-        <mu2>1.0</mu2>
-    </gazebo>
-    <gazebo reference="base_l4_s2">
-        <mu1>1.0</mu1>
-        <mu2>1.0</mu2>
-    </gazebo>
-    <gazebo reference="base_link">
-        <mu1>1.0</mu1>
-        <mu2>1.0</mu2>
-    </gazebo>
-    <gazebo reference="bat_platform">
-        <mu1>1.0</mu1>
-        <mu2>1.0</mu2>
-    </gazebo>
-    <gazebo reference="bathold_1">
-        <mu1>1.0</mu1>
-        <mu2>1.0</mu2>
-    </gazebo>
-    <gazebo reference="bathold_2">
-        <mu1>1.0</mu1>
-        <mu2>1.0</mu2>
-    </gazebo>
-    <gazebo reference="caster_base_2">
-        <mu1>1.0</mu1>
-        <mu2>1.0</mu2>
-    </gazebo>
-    <gazebo reference="caster_middle_2">
-        <mu1>1.0</mu1>
-        <mu2>1.0</mu2>
-    </gazebo>
-    <gazebo reference="caster_wheel_2">
-        <mu1>1.0</mu1>
-        <mu2>1.0</mu2>
-    </gazebo>
-    <gazebo reference="coupling_11">
-        <mu1>1.0</mu1>
-        <mu2>1.0</mu2>
-    </gazebo>
-    <gazebo reference="coupling_12">
-        <mu1>1.0</mu1>
-        <mu2>1.0</mu2>
-    </gazebo>
-    <gazebo reference="driver">
-        <mu1>1.0</mu1>
-        <mu2>1.0</mu2>
-    </gazebo>
-    <gazebo reference="esp32">
-        <mu1>1.0</mu1>
-        <mu2>1.0</mu2>
-    </gazebo>
-    <gazebo reference="esp32_adapter">
-        <mu1>1.0</mu1>
-        <mu2>1.0</mu2>
-    </gazebo>
-    <gazebo reference="ld19">
-        <mu1>1.0</mu1>
-        <mu2>1.0</mu2>
-    </gazebo>
-    <gazebo reference="lidar_serial">
-        <mu1>1.0</mu1>
-        <mu2>1.0</mu2>
-    </gazebo>
-    <gazebo reference="m3x10_accel_base_fl">
-        <mu1>1.0</mu1>
-        <mu2>1.0</mu2>
-    </gazebo>
-    <gazebo reference="m3x10_accel_base_fr">
-        <mu1>1.0</mu1>
-        <mu2>1.0</mu2>
-    </gazebo>
-    <gazebo reference="m3x10_accel_base_rl">
-        <mu1>1.0</mu1>
-        <mu2>1.0</mu2>
-    </gazebo>
-    <gazebo reference="m3x10_accel_base_rr">
-        <mu1>1.0</mu1>
-        <mu2>1.0</mu2>
-    </gazebo>
-    <gazebo reference="m3x10_accel_l2_s1_fl">
-        <mu1>1.0</mu1>
-        <mu2>1.0</mu2>
-    </gazebo>
-    <gazebo reference="m3x10_accel_l2_s1_fr">
-        <mu1>1.0</mu1>
-        <mu2>1.0</mu2>
-    </gazebo>
-    <gazebo reference="m3x10_accel_l2_s1_rl">
-        <mu1>1.0</mu1>
-        <mu2>1.0</mu2>
-    </gazebo>
-    <gazebo reference="m3x10_accel_l2_s1_rr">
-        <mu1>1.0</mu1>
-        <mu2>1.0</mu2>
-    </gazebo>
-    <gazebo reference="m3x10_bathol_f">
-        <mu1>1.0</mu1>
-        <mu2>1.0</mu2>
-    </gazebo>
-    <gazebo reference="m3x10_bathol_fl">
-        <mu1>1.0</mu1>
-        <mu2>1.0</mu2>
-    </gazebo>
-    <gazebo reference="m3x10_bathol_fr">
-        <mu1>1.0</mu1>
-        <mu2>1.0</mu2>
-    </gazebo>
-    <gazebo reference="m3x10_bathol_r">
-        <mu1>1.0</mu1>
-        <mu2>1.0</mu2>
-    </gazebo>
-    <gazebo reference="m3x10_bathol_rl">
-        <mu1>1.0</mu1>
-        <mu2>1.0</mu2>
-    </gazebo>
-    <gazebo reference="m3x10_bathol_rr">
-        <mu1>1.0</mu1>
-        <mu2>1.0</mu2>
-    </gazebo>
-    <gazebo reference="m3x10_driver_fl">
-        <mu1>1.0</mu1>
-        <mu2>1.0</mu2>
-    </gazebo>
-    <gazebo reference="m3x10_driver_fr">
-        <mu1>1.0</mu1>
-        <mu2>1.0</mu2>
-    </gazebo>
-    <gazebo reference="m3x10_driver_rl">
-        <mu1>1.0</mu1>
-        <mu2>1.0</mu2>
-    </gazebo>
-    <gazebo reference="m3x10_driver_rr">
-        <mu1>1.0</mu1>
-        <mu2>1.0</mu2>
-    </gazebo>
-    <gazebo reference="m3x10_esp_adapter_fl">
-        <mu1>1.0</mu1>
-        <mu2>1.0</mu2>
-    </gazebo>
-    <gazebo reference="m3x10_esp_adapter_fr">
-        <mu1>1.0</mu1>
-        <mu2>1.0</mu2>
-    </gazebo>
-    <gazebo reference="m3x10_esp_adapter_rl">
-        <mu1>1.0</mu1>
-        <mu2>1.0</mu2>
-    </gazebo>
-    <gazebo reference="m3x10_esp_adapter_rr">
-        <mu1>1.0</mu1>
-        <mu2>1.0</mu2>
-    </gazebo>
-    <gazebo reference="m3x10_lidar_fl">
-        <mu1>1.0</mu1>
-        <mu2>1.0</mu2>
-    </gazebo>
-    <gazebo reference="m3x10_lidar_r">
-        <mu1>1.0</mu1>
-        <mu2>1.0</mu2>
-    </gazebo>
-    <gazebo reference="m3x10_lidar_rl">
-        <mu1>1.0</mu1>
-        <mu2>1.0</mu2>
-    </gazebo>
-    <gazebo reference="m3x10_rpi5_fl">
-        <mu1>1.0</mu1>
-        <mu2>1.0</mu2>
-    </gazebo>
-    <gazebo reference="m3x10_rpi5_fr">
-        <mu1>1.0</mu1>
-        <mu2>1.0</mu2>
-    </gazebo>
-    <gazebo reference="m3x10_rpi5_rl">
-        <mu1>1.0</mu1>
-        <mu2>1.0</mu2>
-    </gazebo>
-    <gazebo reference="m3x10_rpi5_rr">
-        <mu1>1.0</mu1>
-        <mu2>1.0</mu2>
-    </gazebo>
-    <gazebo reference="m4x17_caster_fl">
-        <mu1>1.0</mu1>
-        <mu2>1.0</mu2>
-    </gazebo>
-    <gazebo reference="m4x17_caster_fr">
-        <mu1>1.0</mu1>
-        <mu2>1.0</mu2>
-    </gazebo>
-    <gazebo reference="m4x17_caster_rl">
-        <mu1>1.0</mu1>
-        <mu2>1.0</mu2>
-    </gazebo>
-    <gazebo reference="m4x17_caster_rr">
-        <mu1>1.0</mu1>
-        <mu2>1.0</mu2>
-    </gazebo>
-    <gazebo reference="maixsense">
-        <mu1>1.0</mu1>
-        <mu2>1.0</mu2>
-    </gazebo>
-    <gazebo reference="maixsense_sup">
-        <mu1>1.0</mu1>
-        <mu2>1.0</mu2>
-    </gazebo>
-    <gazebo reference="motor_dc_11">
-        <mu1>1.0</mu1>
-        <mu2>1.0</mu2>
-    </gazebo>
-    <gazebo reference="motor_dc_12">
-        <mu1>1.0</mu1>
-        <mu2>1.0</mu2>
-    </gazebo>
-    <gazebo reference="motor_support_11">
-        <mu1>1.0</mu1>
-        <mu2>1.0</mu2>
-    </gazebo>
-    <gazebo reference="motor_support_12">
-        <mu1>1.0</mu1>
-        <mu2>1.0</mu2>
-    </gazebo>
-    <gazebo reference="neumatic_11">
-        <mu1>1.0</mu1>
-        <mu2>1.0</mu2>
-    </gazebo>
-    <gazebo reference="neumatic_12">
-        <mu1>1.0</mu1>
-        <mu2>1.0</mu2>
-    </gazebo>
-    <gazebo reference="picam">
-        <mu1>1.0</mu1>
-        <mu2>1.0</mu2>
-    </gazebo>
-    <gazebo reference="picam_sup">
-        <mu1>1.0</mu1>
-        <mu2>1.0</mu2>
-    </gazebo>
-    <gazebo reference="reg_support">
-        <mu1>1.0</mu1>
-        <mu2>1.0</mu2>
-    </gazebo>
-    <gazebo reference="regulator">
-        <mu1>1.0</mu1>
-        <mu2>1.0</mu2>
-    </gazebo>
-    <gazebo reference="ring_11">
-        <mu1>1.0</mu1>
-        <mu2>1.0</mu2>
-    </gazebo>
-    <gazebo reference="ring_12">
-        <mu1>1.0</mu1>
-        <mu2>1.0</mu2>
-    </gazebo>
-    <gazebo reference="rpi5">
-        <mu1>1.0</mu1>
-        <mu2>1.0</mu2>
-    </gazebo>
-    <gazebo reference="screen">
-        <mu1>1.0</mu1>
-        <mu2>1.0</mu2>
-    </gazebo>
-    <gazebo reference="screen_sup">
-        <mu1>1.0</mu1>
-        <mu2>1.0</mu2>
-    </gazebo>
-    <gazebo reference="servo">
-        <mu1>1.0</mu1>
-        <mu2>1.0</mu2>
-    </gazebo>
-    <gazebo reference="servo_1">
-        <mu1>1.0</mu1>
-        <mu2>1.0</mu2>
-    </gazebo>
-    <gazebo reference="servo_2">
-        <mu1>1.0</mu1>
-        <mu2>1.0</mu2>
-    </gazebo>
-    <gazebo reference="servo_conn">
-        <mu1>1.0</mu1>
-        <mu2>1.0</mu2>
-    </gazebo>
-    <gazebo reference="servo_conn_1">
-        <mu1>1.0</mu1>
-        <mu2>1.0</mu2>
-    </gazebo>
-    <gazebo reference="servo_conn_2">
-        <mu1>1.0</mu1>
-        <mu2>1.0</mu2>
-    </gazebo>
-    <gazebo reference="servo_support_1">
-        <mu1>1.0</mu1>
-        <mu2>1.0</mu2>
-    </gazebo>
-    <gazebo reference="servo_support_2">
-        <mu1>1.0</mu1>
-        <mu2>1.0</mu2>
-    </gazebo>
-    <gazebo reference="spacer_l0_11">
-        <mu1>1.0</mu1>
-        <mu2>1.0</mu2>
-    </gazebo>
-    <gazebo reference="spacer_l0_12">
-        <mu1>1.0</mu1>
-        <mu2>1.0</mu2>
-    </gazebo>
-    <gazebo reference="spacer_l0_21">
-        <mu1>1.0</mu1>
-        <mu2>1.0</mu2>
-    </gazebo>
-    <gazebo reference="spacer_l0_22">
-        <mu1>1.0</mu1>
-        <mu2>1.0</mu2>
-    </gazebo>
-    <gazebo reference="spacer_l1_11">
-        <mu1>1.0</mu1>
-        <mu2>1.0</mu2>
-    </gazebo>
-    <gazebo reference="spacer_l1_12">
-        <mu1>1.0</mu1>
-        <mu2>1.0</mu2>
-    </gazebo>
-    <gazebo reference="spacer_l1_21">
-        <mu1>1.0</mu1>
-        <mu2>1.0</mu2>
-    </gazebo>
-    <gazebo reference="spacer_l1_22">
-        <mu1>1.0</mu1>
-        <mu2>1.0</mu2>
-    </gazebo>
-    <gazebo reference="spacer_l2_11">
-        <mu1>1.0</mu1>
-        <mu2>1.0</mu2>
-    </gazebo>
-    <gazebo reference="spacer_l2_12">
-        <mu1>1.0</mu1>
-        <mu2>1.0</mu2>
-    </gazebo>
-    <gazebo reference="spacer_l2_21">
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