Commit message: Description: Changed management of gazebo references

File: orion_description/urdf/orion_macros.urdf.xacro (robot description, xacro)
@@ -7,5 +7,5 @@
     <xacro:property name="pi_8" value="${pi / 8}"/>
     <!--///////////////////// 10 x 80 SPACERS MACROS ///////////////////////-->
-    <!-- single custom spacer 10 x 80 mm -->
+    <!-- ......................... Single custom spacer ................... -->
     <xacro:macro name="spacer_10x80" params="front side level x y z">
         <!-- Orientation properties -->
@@ -53,5 +53,4 @@
         </inertial>
         </link>
-        <!-- Joint definition -->
         <joint name="spacer_l${level}_${front}${side}_joint" type="fixed">
             <parent link="base_l${level}_s${front}"/>
@@ -59,5 +58,12 @@
             <origin xyz="${x*mulf} ${y*muls} ${z+0.0025}" rpy="0 0 0"/>
         </joint>
-    </xacro:macro>
+        <xacro:if value="${gazebo}">
+        <gazebo reference="spacer_l${level}_${front}${side}">
+            <mu1>1.0</mu1>
+            <mu2>1.0</mu2>
+        </gazebo>
+    </xacro:if>
+    </xacro:macro>
+    <!-- ....................... Double 10x80 Spacer .................... -->
     <xacro:macro name="double_spacer_10x80" params="front level x y z">
         <xacro:spacer_10x80 front="${front}" side="1" level="${level}" x="${x}"
@@ -67,4 +73,5 @@
     </xacro:macro>
     <!--//////////////////// BASES AND LEVELS MACROS ///////////////////////-->
+    <!-- ................... Half base macro .............................. -->
     <xacro:macro name="half_base" params="level side parent x y z">
         <xacro:property name="mul" value="1"/>
@@ -72,5 +79,4 @@
             <xacro:property name="mul" value="-1"/>
         </xacro:if>
-        <!-- Link -->
         <link name="base_l${level}_s${side}">
         <visual>
@@ -97,5 +103,4 @@
         </inertial>
         </link>
-        <!-- Fixed Joint -->
         <joint name="base_l${level}_s${side}_joint" type="fixed">
             <parent link="${parent}"/>
@@ -103,5 +108,10 @@
             <origin xyz="${x + (mul*0.115/2)} ${y} ${z}" rpy="0 0 0"/>
         </joint>
-    </xacro:macro>
+        <gazebo reference="base_l${level}_s${side}">
+            <mu1>1.0</mu1>
+            <mu2>1.0</mu2>
+        </gazebo>
+    </xacro:macro>
+    <!-- ...................... Complete base ............................ -->
     <xacro:macro name="com_base" params="level parent x y z">
         <xacro:half_base level="${level}" side="1" parent="base_link" x="${x}"
@@ -111,5 +121,5 @@
     </xacro:macro>
     <!--  /////////////////// MOTOR DC MACROS ///////////////////////////////-->
-    <!--  Motor DC Component Kit -->
+    <!-- ....................... Motor DC Kit .............................. -->
     <xacro:macro name="motor_dc" params="front side x y z">
         <!-- Properties -->
@@ -124,5 +134,5 @@
             <xacro:property name="orin" value="${pi}"/>
         </xacro:if>
-        <!-- Link motor mount definition-->
+        <!-- Motor mount definition-->
         <link name="motor_support_${front}${side}">
         <visual>
@@ -149,5 +159,4 @@
         </inertial>
         </link>
-        <!-- Joint motor mount definition-->
         <joint name="motor_support_${front}${side}_joint" type="fixed">
             <parent link="base_l0_s${front}"/>
@@ -155,4 +164,8 @@
             <origin xyz="${x*mulf} ${y*muls} ${z+0.0025}" rpy="0 0 0"/>
         </joint>
+        <gazebo reference="motor_support_${front}${side}">
+            <mu1>1.0</mu1>
+            <mu2>1.0</mu2>
+        </gazebo>
         <!-- Link motor dc definition-->
         <link name="motor_dc_${front}${side}">
@@ -180,5 +193,4 @@
         </inertial>
         </link>
-        <!-- Joint motor dc definition-->
         <joint name="motor_dc_${front}${side}_joint" type="fixed">
             <parent link="motor_support_${front}${side}"/>
@@ -186,5 +198,9 @@
             <origin xyz="0 ${-0.05625*muls} 0" rpy="0 0 0"/>
         </joint>
-        <!-- Link coupling definition-->
+        <gazebo reference="motor_dc_${front}${side}">
+            <mu1>1.0</mu1>
+            <mu2>1.0</mu2>
+        </gazebo>
+        <!-- Coupling definition-->
         <link name="coupling_${front}${side}">
         <visual>
@@ -211,5 +227,4 @@
         </inertial>
         </link>
-        <!-- Joint coupling definition-->
         <joint name="coupling_${front}${side}_joint" type="continuous">
             <axis xyz="0.0 0.0 1.0"/>
@@ -218,5 +233,9 @@
             <origin xyz="0 ${(0.01120 + 0.000325)*muls} 0" rpy="${-pi_2*muls+orin} 0 0"/>
         </joint>
-        <!-- LInk Ring  definition-->
+        <gazebo reference="coupling_${front}${side}">
+            <mu1>1.0</mu1>
+            <mu2>1.0</mu2>
+        </gazebo>
+        <!-- Ring definition -->
         <link name="ring_${front}${side}">
         <visual>
@@ -243,5 +262,4 @@
         </inertial>
         </link>
-        <!-- Joint ring definition-->
         <joint name="ring_${front}${side}_joint" type="fixed">
             <parent link="coupling_${front}${side}"/>
@@ -249,5 +267,9 @@
             <origin xyz="0 0 ${0.0068*muls}" rpy="0 0 0"/>
         </joint>
-        <!-- Link neumatic definition-->
+        <gazebo reference="ring_${front}${side}">
+            <mu1>1.0</mu1>
+            <mu2>1.0</mu2>
+        </gazebo>
+        <!-- Neumatic definition-->
         <link name="neumatic_${front}${side}">
         <visual>
@@ -274,5 +296,4 @@
         </inertial>
         </link>
-        <!-- Joint neumatic definition-->
         <joint name="neumatic_${front}${side}_joint" type="fixed">
             <parent link="ring_${front}${side}"/>
@@ -280,8 +301,13 @@
             <origin xyz="0 0 0" rpy="0 0 0"/>
         </joint>
+        <gazebo reference="neumatic_${front}${side}">
+            <mu1>1.0</mu1>
+            <mu2>1.0</mu2>
+        </gazebo>
     </xacro:macro>
     <!--////////////////////////// CASTER WHEEL ////////////////////////////-->
+    <!-- ......................... Macro for caster ....................... -->
     <xacro:macro name="caster_wheel" params="parent front x y z">
-        <!-- Link caster base definition-->
+        <!-- Caster base definition-->
         <link name="caster_base_${front}">
         <visual>
@@ -308,5 +334,4 @@
         </inertial>
         </link>
-        <!-- Joint caster base definition-->
         <joint name="caster_base_${front}_joint" type="fixed">
             <parent link="${parent}"/>
@@ -314,5 +339,9 @@
             <origin xyz="${x} ${y} ${z}" rpy="0 0 0"/>
         </joint>
-        <!-- Link caster middle definition-->
+        <gazebo reference="caster_base_${front}">
+            <mu1>1.0</mu1>
+            <mu2>1.0</mu2>
+        </gazebo>
+        <!-- Caster middle definition-->
         <link name="caster_middle_${front}">
         <visual>
@@ -339,5 +368,4 @@
         </inertial>
         </link>
-        <!-- Joint caster middle definition-->
         <joint name="caster_middle_${front}_joint" type="continuous">
             <axis xyz="0.0 0.0 1.0"/>
@@ -346,5 +374,9 @@
             <origin xyz="0 0 -0.002" rpy="${pi} 0 0"/>
         </joint>
-        <!-- Link caster wheel definition-->
+        <gazebo reference="caster_middle_${front}">
+            <mu1>1.0</mu1>
+            <mu2>1.0</mu2>
+        </gazebo>
+        <!-- Caster wheel definition-->
         <link name="caster_wheel_${front}">
         <visual>
@@ -371,14 +403,17 @@
         </inertial>
         </link>
-        <!-- Joint caster wheel definition-->
         <joint name="caster_wheel_${front}_joint" type="continuous">
             <axis xyz="0.0 0.0 1.0"/>
             <parent link="caster_middle_${front}"/>
             <child link="caster_wheel_${front}"/>
-            <origin xyz="-0.0108 0 0.0185" rpy="${pi/2} 0 0"/>
-        </joint>
+            <origin xyz="-0.0108 0 0.0185" rpy="${pi_2} 0 0"/>
+        </joint>
+        <gazebo reference="caster_wheel_${front}">
+            <mu1>1.0</mu1>
+            <mu2>1.0</mu2>
+        </gazebo>
     </xacro:macro>
     <!-- ///////////////////// BATTERIES MACROS ////////////////////////////-->
-    <!-- B18650 Macro-->
+    <!-- ...................... B18650 Macro .............................. -->
     <xacro:macro name="b18650" params="parent element num x y z">
         <xacro:property name="inv" value="1"/>
@@ -421,5 +456,10 @@
             <origin xyz="${x*inv} ${y} ${z}" rpy="0 0 0"/>
         </joint>
-    </xacro:macro>
+        <gazebo reference="${element}_${num}">
+            <mu1>1.0</mu1>
+            <mu2>1.0</mu2>
+        </gazebo>
+    </xacro:macro>
+    <!-- ........................ Battery holder macro ........................ -->
     <xacro:macro name="bat_hold" params=" parent element num x y z">
         <!-- Link -->
@@ -453,4 +493,8 @@
             <origin xyz="${x} ${y} ${z}" rpy="0 0 0"/>
         </joint>
+        <gazebo reference="${element}_${num}">
+            <mu1>1.0</mu1>
+            <mu2>1.0</mu2>
+        </gazebo>
     </xacro:macro>
     <xacro:macro name="stack_bat" params="parent num x y z">
@@ -498,5 +542,4 @@
         </inertial>
         </link>
-        <!-- Servo Mount Joint -->
         <joint name="servo_support_${side}_joint" type="fixed">
             <parent link="${parent}"/>
@@ -504,4 +547,8 @@
             <origin xyz="${x} ${y*inv} ${z}" rpy="0 0 0"/>
         </joint>
+        <gazebo reference="servo_support_${side}">
+            <mu1>1.0</mu1>
+            <mu2>1.0</mu2>
+        </gazebo>
         <!-- Servo Link -->
         <link name="servo_${side}">
@@ -529,5 +576,4 @@
         </inertial>
         </link>
-        <!-- Servo Joint -->
         <joint name="servo_${side}_joint" type="fixed">
             <parent link="servo_support_${side}"/>
@@ -535,5 +581,9 @@
             <origin xyz="0 ${-0.0216*inv} -0.01375" rpy="0 0 0"/>
         </joint>
-        <!-- Servo Link -->
+        <gazebo reference="servo_${side}">
+            <mu1>1.0</mu1>
+            <mu2>1.0</mu2>
+        </gazebo>
+        <!-- Servo Conn -->
         <link name="servo_conn_${side}">
         <visual>
@@ -560,5 +610,4 @@
         </inertial>
         </link>
-        <!-- Servo Joint -->
         <joint name="servo_conn${side}_joint" type="revolute">
             <axis xyz="0.0 0.0 1.0"/>
@@ -569,4 +618,8 @@
             <dynamics damping="0.1" friction="0.01"/>
         </joint>
+        <gazebo reference="servo_conn_${side}">
+            <mu1>1.0</mu1>
+            <mu2>1.0</mu2>
+        </gazebo>
     </xacro:macro>
     <!--///////////////////// SPEAKERS MACROS ///////////////////////-->
@@ -584,5 +637,5 @@
             <xacro:property name="inv" value="0"/>
         </xacro:if>
-        <!-- Link speaker -->
+        <!-- Speaker support -->
         <link name="speaker_sup_${front}${side}">
         <visual>
@@ -609,5 +662,4 @@
         </inertial>
         </link>
-        <!-- Joint speaker support -->
         <joint name="speaker_sup_${front}${side}_joint" type="fixed">
             <parent link="${parent}"/>
@@ -615,5 +667,9 @@
             <origin xyz="${x*mulf} ${y*muls} ${z}" rpy="0 0 0"/>
         </joint>
-        <!-- Link speaker -->
+        <gazebo reference="speaker_sup_${front}${side}">
+            <mu1>1.0</mu1>
+            <mu2>1.0</mu2>
+        </gazebo>
+        <!-- Speaker -->
         <link name="speaker_${front}${side}">
         <visual>
@@ -640,5 +696,4 @@
         </inertial>
         </link>
-        <!-- Joint speaker -->
         <joint name="speaker_${front}${side}_joint" type="fixed">
             <parent link="speaker_sup_${front}${side}"/>
@@ -646,4 +701,8 @@
             <origin xyz="0 ${0.0285*muls/2} 0" rpy="0 0 0"/>
         </joint>
+        <gazebo reference="speaker_${front}${side}">
+            <mu1>1.0</mu1>
+            <mu2>1.0</mu2>
+        </gazebo>
     </xacro:macro>
     <!-- ///////////////////////////// WALL MACROS //////////////////////// -->
@@ -654,5 +713,4 @@
             <xacro:property name="muls" value="-1"/>
         </xacro:if>
-        <!-- Link -->
         <link name="wall_${id}_${level}_${side}">
         <visual>
@@ -684,4 +742,8 @@
         <origin xyz="${x} ${(y+0.00075)*muls} ${z}" rpy="0 0 0"/>
         </joint>
+        <gazebo reference="wall_${id}_${level}_${side}">
+            <mu1>1.0</mu1>
+            <mu2>1.0</mu2>
+        </gazebo>
     </xacro:macro>
     <xacro:macro name="complete_front_wall"
@@ -723,4 +785,8 @@
         <origin xyz="${(x+0.00075)*mulf} 0 ${z}" rpy="0 0 0"/>
         </joint>
+        <gazebo reference="wall_${id}_${level}_${front}">
+            <mu1>1.0</mu1>
+            <mu2>1.0</mu2>
+        </gazebo>
     </xacro:macro>
     <!-- /////////////////////////// Generic Metric Spacer /////////////////-->
@@ -766,4 +832,9 @@
             <origin xyz="${x} ${y} ${z}" rpy="0 0 0"/>
         </joint>
+        <!-- Gazebo Spacer -->
+        <gazebo reference="${id}_${element}_${front}${side}">
+            <mu1>1.0</mu1>
+            <mu2>1.0</mu2>
+        </gazebo>
     </xacro:macro>
     <!-- 2 symetric hex spacers by considering offset -->

Commit message: Description: Added diff controller and lidar sensor plugin for Gazebo

File: orion_description/urdf/orion_base.urdf.xacro (robot description, xacro)
@@ -361,8 +361,15 @@
     <xacro:if value="${gazebo}">
         <gazebo reference="ld19">
-            <mu1>1.0</mu1>
-            <mu2>1.0</mu2>
-        </gazebo>
-    </xacro:if>
+            <selfCollide>false</selfCollide>
+            <mu1 value="0.05" />
+            <mu2 value="0.05" />
+        </gazebo>
+    </xacro:if>
+    <link name="laser_scan"/>
+    <joint name="laser_joint" type="fixed">
+        <parent link="ld19"/>
+        <child link="laser_scan"/>
+        <origin xyz="0 0 0.03" rpy="0 0 0"/>
+    </joint>
     <!-- ......................... LIDAR serial .......................... -->
     <link name="lidar_serial">

File: orion_description/urdf/orion_gz.urdf.xacro (robot description, xacro)
@@ -2,7 +2,12 @@
 <robot xmlns:xacro="http://www.ros.org/wiki/xacro">
     <gazebo>
+        <plugin
+			filename="gz-sim-sensors-system"
+			name="gz::sim::systems::Sensors">
+			<render_engine>ogre2</render_engine>
+        </plugin>
         <plugin filename="gz-sim-diff-drive-system" name="gz::sim::systems::DiffDrive">
-            <right_joint>coupling_11_joint</right_joint>
-            <left_joint>coupling_12_joint</left_joint>
+            <right_joint>coupling_12_joint</right_joint>
+            <left_joint>coupling_11_joint</left_joint>
             <wheel_separation>0.21</wheel_separation>
             <wheel_radius>0.03</wheel_radius>
@@ -18,3 +23,31 @@
         </plugin>
     </gazebo>
+    <gazebo reference="laser_scan">
+		<sensor name='gpu_lidar' type='gpu_lidar'>
+          <topic>lidar</topic>
+          <update_rate>10</update_rate>
+          <lidar>
+            <scan>
+              <horizontal>
+                <samples>640</samples>
+                <resolution>1</resolution>
+                <min_angle>-1.396263</min_angle>
+                <max_angle>1.396263</max_angle>
+              </horizontal>
+              <vertical>
+                <samples>16</samples>
+                <resolution>1</resolution>
+                <min_angle>-0.261799</min_angle>
+                <max_angle>0.261799</max_angle>
+              </vertical>
+            </scan>
+            <range>
+              <min>0.08</min>
+              <max>10.0</max>
+              <resolution>0.01</resolution>
+            </range>
+          </lidar>
+          <visualize>true</visualize>
+        </sensor>
+    </gazebo>
 </robot>

File: orion_description/urdf/orion_macros.urdf.xacro (robot description, xacro)
@@ -307,4 +307,6 @@
     </xacro:macro>
     <!--////////////////////////// CASTER WHEEL ////////////////////////////-->
+    <!--xacro:property name="caster_type" value="continuous"/-->
+    <xacro:property name="caster_type" value="fixed"/>
     <!-- ......................... Macro for caster ....................... -->
     <xacro:macro name="caster_wheel" params="parent front x y z">
@@ -368,5 +370,5 @@
         </inertial>
         </link>
-        <joint name="caster_middle_${front}_joint" type="continuous">
+        <joint name="caster_middle_${front}_joint" type="${caster_type}">
             <axis xyz="0.0 0.0 1.0"/>
             <parent link="caster_base_${front}"/>
@@ -403,5 +405,5 @@
         </inertial>
         </link>
-        <joint name="caster_wheel_${front}_joint" type="continuous">
+        <joint name="caster_wheel_${front}_joint" type="${caster_type}">
             <axis xyz="0.0 0.0 1.0"/>
             <parent link="caster_middle_${front}"/>
@@ -410,6 +412,6 @@
         </joint>
         <gazebo reference="caster_wheel_${front}">
-            <mu1>1.0</mu1>
-            <mu2>1.0</mu2>
+            <mu1>0.001</mu1>
+            <mu2>0.001</mu2>
         </gazebo>
     </xacro:macro>
