Commit message: Description: Added RGBD, depth and normal cameras, fixed lidar params, epxlored usage of servos but still missing

File: orion_description/urdf/orion_base.urdf.xacro (robot description, xacro)
@@ -370,5 +370,5 @@
         <parent link="ld19"/>
         <child link="laser_scan"/>
-        <origin xyz="0 0 0.03" rpy="0 0 0"/>
+        <origin xyz="0 -0.0025 0.0285" rpy="0 0 0"/>
     </joint>
     <!-- ......................... LIDAR serial .......................... -->

File: orion_description/urdf/orion_gz.urdf.xacro (robot description, xacro)
@@ -1,4 +1,8 @@
 <?xml version="1.0"?>
 <robot xmlns:xacro="http://www.ros.org/wiki/xacro">
+    <!-- ////////////////////// PROPERTIES ////////////////////////////// -->
+    <xacro:property name="noise_and_dist" value="true"/>
+    <!-- ////////////////////// GENERAL PLUGINS ///////////////////////// -->
+    <!-- ...................... Required for sensors systems ............ -->
     <gazebo>
         <plugin
@@ -7,5 +11,10 @@
 			<render_engine>ogre2</render_engine>
         </plugin>
-        <plugin filename="gz-sim-diff-drive-system" name="gz::sim::systems::DiffDrive">
+    </gazebo>
+    <!-- ////////////////////// JOINT PLUGINS /////////////////////////// -->
+    <gazebo>
+        <!-- ...................... Differential Controller ..............-->
+        <plugin filename="gz-sim-diff-drive-system"
+            name="gz::sim::systems::DiffDrive">
             <right_joint>coupling_12_joint</right_joint>
             <left_joint>coupling_11_joint</left_joint>
@@ -17,37 +26,202 @@
             <odom_topic>odom</odom_topic>
         </plugin>
+        <plugin
+            filename="gz-sim-joint-position-controller-system"
+            name="gz::sim::systems::JointPositionController">
+            <joint_name>servo_conn1_joint</joint_name>
+            <topic>servo_conn1</topic>
+            <p_gain>1</p_gain>
+            <i_gain>0.1</i_gain>
+            <d_gain>0.01</d_gain>
+            <i_max>1</i_max>
+            <i_min>-1</i_min>
+            <cmd_max>1000</cmd_max>
+            <cmd_min>-1000</cmd_min>
+        </plugin>
+        <plugin
+            filename="gz-sim-joint-position-controller-system"
+            name="gz::sim::systems::JointPositionController">
+            <joint_name>servo_conn2_joint</joint_name>
+            <topic>servo_conn2</topic>
+            <p_gain>1</p_gain>
+            <i_gain>0.1</i_gain>
+            <d_gain>0.01</d_gain>
+            <i_max>1</i_max>
+            <i_min>-1</i_min>
+            <cmd_max>1000</cmd_max>
+            <cmd_min>-1000</cmd_min>
+        </plugin>
+        <!-- ...................... Joint state publisher ................ -->
         <plugin filename="gz-sim-joint-state-publisher-system" name="gz::sim::systems::JointStatePublisher">
             <topic>joint_states</topic>
             <joint_name>coupling_11_joint</joint_name>
             <joint_name>coupling_12_joint</joint_name>
+            <xacro:if value="${servo}">
+                <joint_name>servo_conn1_joint</joint_name>
+                <joint_name>servo_conn2_joint</joint_name>
+            </xacro:if>
+            <xacro:if value="${camera == 'a010' and g_mov}">
+                <joint_name>g_mov_servo_conn_joint</joint_name>
+            </xacro:if>
         </plugin>
     </gazebo>
+    <!-- ////////////////////// SENSOR PLUGINS ///////////////////////// -->
+    <!-- .......................... LIDARs ............................. -->
     <gazebo reference="laser_scan">
 		<sensor name='gpu_lidar' type='gpu_lidar'>
-          <topic>lidar</topic>
-          <update_rate>10</update_rate>
-          <lidar>
-            <scan>
-              <horizontal>
-                <samples>640</samples>
-                <resolution>1</resolution>
-                <min_angle>-1.396263</min_angle>
-                <max_angle>1.396263</max_angle>
-              </horizontal>
-              <vertical>
-                <samples>16</samples>
-                <resolution>1</resolution>
-                <min_angle>-0.261799</min_angle>
-                <max_angle>0.261799</max_angle>
-              </vertical>
-            </scan>
-            <range>
-              <min>0.08</min>
-              <max>10.0</max>
-              <resolution>0.01</resolution>
-            </range>
-          </lidar>
-          <visualize>true</visualize>
+            <topic>lidar</topic>
+            <update_rate>10</update_rate>
+            <!-- Inof based on: -->
+            <!-- https://www.ldrobot.com/images/2023/05/23/LDROBOT_LD19_Datasheet_EN_v2.6_Q1JXIRVq.pdf -->
+            <ray>
+                <scan>
+                <horizontal>
+                    <samples>720</samples>
+                    <resolution>1</resolution>
+                    <min_angle>0</min_angle>
+                    <max_angle>${2*pi}</max_angle>
+                </horizontal>
+                <vertical>
+                    <samples>1</samples>
+                    <resolution>0.01</resolution>
+                    <min_angle>0</min_angle>
+                    <max_angle>0</max_angle>
+                </vertical>
+                </scan>
+                <range>
+                    <min>0.03</min>
+                    <max>12.0</max>
+                    <resolution>0.01</resolution>
+                </range>
+                <!-- Noise addition -->
+                <noise>
+                    <type>gaussian</type>
+                    <mean>0.0</mean>
+                    <stddev>0.01</stddev>
+                </noise>
+            </ray>
+            <always_on>1</always_on>
+            <visualize>true</visualize>
         </sensor>
     </gazebo>
+    <!-- .......................... Cameras ................................ -->
+    <xacro:if value="${camera== 'astra_s'}">
+        <gazebo reference="camera_link">
+            <sensor name="camera" type="rgbd_camera">
+                <!-- Data based on https://store.orbbec.com/products/astra-s -->
+                <camera>
+                    <horizontal_fov>1.1013</horizontal_fov>
+                    <image>
+                    <width>640</width>
+                    <height>480</height>
+                    </image>
+                    <clip>
+                        <near>0.4</near>
+                        <far>2</far>
+                    </clip>
+                    <xacro:if value="${noise_and_dist}">
+                        <!-- Noise addition -->
+                        <noise>
+                            <type>gaussian</type>
+                            <mean>0.003</mean>
+                            <stddev>0.01</stddev>
+                        </noise>
+                        <!-- Distorsion addition -->
+                        <distortion>
+                            <k1>0.02</k1>
+                            <k2>0.02</k2>
+                            <k3>0.01</k3>
+                            <p1>0.01</p1>
+                            <p2>0.01</p2>
+                            <center>0.5 0.5</center>
+                        </distortion>
+                    </xacro:if>
+                </camera>
+                <always_on>1</always_on>
+                <update_rate>30</update_rate>
+                <visualize>true</visualize>
+                <topic>rgbd_camera</topic>
+            </sensor>
+        </gazebo>
+    </xacro:if>
+    <xacro:if value="${camera== 'os30a'}">
+        <gazebo reference="camera_link">
+            <sensor name="camera" type="rgbd_camera">
+                <!-- Data based on : -->
+                <!-- https://www.ydlidar.com/Public/upload/files/2022-11-30/BMVM-OS30A%20Data%20Sheet%20V1.0%20(221130).pdf -->
+                <camera>
+                    <horizontal_fov>1.263618</horizontal_fov>
+                    <image>
+                    <width>1080</width>
+                    <height>920</height>
+                    </image>
+                    <clip>
+                        <near>0.2</near>
+                        <far>2.5</far>
+                    </clip>
+                    <xacro:if value="${noise_and_dist}">
+                        <!-- Noise addition -->
+                        <noise>
+                            <type>gaussian</type>
+                            <mean>0.0</mean>
+                            <stddev>0.015</stddev>
+                        </noise>
+                        <!-- Distorsion addition -->
+                        <distortion>
+                            <k1>-0.1</k1>
+                            <k2>0.02</k2>
+                            <k3>0.01</k3>
+                            <p1>0.0</p1>
+                            <p2>0.0</p2>
+                            <center>0.5 0.5</center>
+                        </distortion>
+                    </xacro:if>
+                </camera>
+                <always_on>1</always_on>
+                <update_rate>30</update_rate>
+                <visualize>true</visualize>
+                <topic>rgbd_camera</topic>
+            </sensor>
+        </gazebo>
+    </xacro:if>
+    <xacro:if value="${camera== 'a010'}">
+        <gazebo reference="camera_link">
+            <!-- Data based on: -->
+            <!-- https://pdf.direnc.net/upload/1-14-inc-lcd-ekranli-3d-tof-derinlik-sensoru-kamera-datasheet.pdf -->
+            <sensor name="camera" type="depth_camera">
+                <camera>
+                    <horizontal_fov>1.22</horizontal_fov>
+                    <image>
+                    <width>100</width>
+                    <height>100</height>
+                    </image>
+                    <clip>
+                        <near>0.15</near>
+                        <far>1.5</far>
+                    </clip>
+                    <xacro:if value="${noise_and_dist}">
+                        <!-- Noise addition -->
+                        <noise>
+                            <type>gaussian</type>
+                            <mean>0.0</mean>
+                            <stddev>0.01</stddev>
+                        </noise>
+                        <!-- Distorsion addition -->
+                        <distortion>
+                            <k1>-0.025</k1>
+                            <k2>0.005</k2>
+                            <k3>0.002</k3>
+                            <p1>0.0</p1>
+                            <p2>0.0</p2>
+                            <center>0.5 0.5</center>
+                        </distortion>
+                    </xacro:if>
+                </camera>
+                <always_on>1</always_on>
+                <update_rate>20</update_rate>
+                <visualize>true</visualize>
+                <topic>depth_camera</topic>
+            </sensor>
+        </gazebo>
+    </xacro:if>
 </robot>

Commit message: Description: Added touch sensor visual/collision, re-added diffdrive controller, fixed odometry | Assets: Created toys and touch support, added 3D print stls for toys

File: orion_description/urdf/orion_base.urdf.xacro (robot description, xacro)
@@ -486,4 +486,13 @@
             </gazebo>
         </xacro:if>
+        <!-- ........................ Touch sensors ........................ -->
+        <xacro:touch_sensor x="0.005" y="0.1075" z="0.0825" upper="0" side="1"
+            parent="base_l2_s2" prefix="2"/>
+        <xacro:touch_sensor x="0.005" y="-0.1075" z="0.0825" upper="0" side="2"
+            parent="base_l2_s2" prefix="2"/>
+        <xacro:touch_sensor x="0.0425" y="0.0335" z="0.0025" upper="1" side="1"
+            parent="base_l4_s2" prefix="4"/>
+        <xacro:touch_sensor x="0.0425" y="-0.0335" z="0.0025" upper="1" side="2"
+            parent="base_l4_s2" prefix="4"/>
         <!-- ........................ Wall definitions ...................... -->
         <xacro:complete_lateral_wall id="curve" parent="base_l2_s1" side="1"

File: orion_description/urdf/orion_gz.urdf.xacro (robot description, xacro)
@@ -12,6 +12,46 @@
         </plugin>
     </gazebo>
+    <!-- ......................... Scene Broadcaster .................... -->
+    <gazebo>
+        <plugin
+            filename="gz-sim-scene-broadcaster-system"
+            name="gz::sim::systems::SceneBroadcaster">
+        </plugin>
+    </gazebo>
     <!-- ////////////////////// JOINT PLUGINS /////////////////////////// -->
     <gazebo>
+        <!-- ...................... Diff Drive Controller ............... -->
+        <plugin
+            filename="gz-sim-diff-drive-system"
+            name="gz::sim::systems::DiffDrive">
+            <left_joint>coupling_11_joint</left_joint>
+            <right_joint>coupling_12_joint</right_joint>
+            <wheel_separation>0.1597</wheel_separation>
+            <wheel_radius>${0.0335/2}</wheel_radius>
+            <odom_publish_frequency>1</odom_publish_frequency>
+            <max_linear_acceleration>1</max_linear_acceleration>
+            <min_linear_acceleration>-1</min_linear_acceleration>
+            <max_angular_acceleration>2</max_angular_acceleration>
+            <min_angular_acceleration>-2</min_angular_acceleration>
+            <max_linear_velocity>2.791666667</max_linear_velocity>
+            <min_linear_velocity>-2.791666667</min_linear_velocity>
+            <max_angular_velocity>2.791666667</max_angular_velocity>
+            <min_angular_velocity>-2.791666667</min_angular_velocity>
+            <odom_topic>/unused/diff_drive_odometry</odom_topic>
+            <tf_topic>/unused/diff_drive_tf</tf_topic>
+            <odom_publish_frequency>1</odom_publish_frequency>
+            <frame_id>odom_diff_drive</frame_id>
+            <child_frame_id>base_link</child_frame_id>
+        <!-- ..................... Odometry Publisher ................. -->
+        <gazebo>
+            <plugin
+            filename="ignition-gazebo-odometry-publisher-system"
+            name="gz::sim::systems::OdometryPublisher">
+            <odom_publish_frequency>20</odom_publish_frequency>
+            <robot_base_frame>base_link</robot_base_frame>
+            <odom_frame>odom</odom_frame>
+            </plugin>
+        </gazebo>
+        </plugin>
         <!-- ...................... Joint state publisher ................ -->
         <plugin filename="gz-sim-joint-state-publisher-system" name="gz::sim::systems::JointStatePublisher">
@@ -19,4 +59,6 @@
             <joint_name>coupling_11_joint</joint_name>
             <joint_name>coupling_12_joint</joint_name>
+            <joint_name>caster_middle_2_joint</joint_name>
+            <joint_name>caster_wheel_2_joint</joint_name>
         <xacro:if value="${servo}">
             <joint_name>servo_conn1_joint</joint_name>
@@ -32,7 +74,6 @@
     <gazebo reference="laser_scan">
 		<sensor name='gpu_lidar' type='gpu_lidar'>
-            <topic>lidar</topic>
             <update_rate>10</update_rate>
-            <!-- Inof based on: -->
+            <!-- Info based on: -->
             <!-- https://www.ldrobot.com/images/2023/05/23/LDROBOT_LD19_Datasheet_EN_v2.6_Q1JXIRVq.pdf -->
             <ray>
@@ -103,5 +144,4 @@
                 <update_rate>30</update_rate>
                 <visualize>true</visualize>
-                <topic>rgbd_camera</topic>
             </sensor>
         </gazebo>
@@ -143,5 +183,4 @@
                 <update_rate>30</update_rate>
                 <visualize>true</visualize>
-                <topic>rgbd_camera</topic>
             </sensor>
         </gazebo>
@@ -183,5 +222,4 @@
                 <update_rate>20</update_rate>
                 <visualize>true</visualize>
-                <topic>depth_camera</topic>
             </sensor>
         </gazebo>

File: orion_description/urdf/orion_macros.urdf.xacro (robot description, xacro)
@@ -316,5 +316,5 @@
     <!--////////////////////////// CASTER WHEEL ////////////////////////////-->
     <!--xacro:property name="caster_type" value="continuous"/-->
-    <xacro:property name="caster_type" value="fixed"/>
+    <xacro:property name="caster_type" value="continuous"/>
     <!-- ......................... Macro for caster ....................... -->
     <xacro:macro name="caster_wheel" params="parent front x y z">
@@ -910,5 +910,95 @@
             front="r" side="" x="${x - offset_x}" y="0" z="${z}"/>
     </xacro:macro>
-    <!-- ///////////////////// Cameras macros ////////////////////// -->
+    <!-- ////////////////////// Touch sensors macros //////////////////////-->
+    <xacro:macro name="touch_sensor" params="x y z upper side parent prefix">
+        <xacro:property name="rotR" value="${-pi_2}"/>
+        <xacro:property name="rotP" value="${pi}"/>
+        <xacro:property name="rotY" value="0"/>
+        <xacro:if value="${side == 2}">
+            <xacro:property name="rotR" value="${pi_2}"/>
+        </xacro:if>
+        <xacro:if value="${upper}">
+            <xacro:property name="rotR" value="0"/>
+            <xacro:property name="rotP" value="0"/>
+            <xacro:property name="rotY" value="${-pi_2}"/>
+        </xacro:if>
+        <link name="touch_sensor_${prefix}${side}">
+            <visual name="">
+                <origin xyz="0.0 0.0 0.0" rpy="${rotR} ${rotP} ${rotY}"/>
+                <geometry>
+                    <mesh filename="package://orion_description/meshes/touch_sensor.stl"
+                    scale="0.001 0.001 0.001"/>
+                </geometry>
+                <material name="ArduinoBlue"/>
+            </visual>
+            <collision>
+                <origin xyz="0.0 0.0 0.0" rpy="${rotR} ${rotP} ${rotY}"/>
+                <geometry>
+                    <mesh filename="package://orion_description/meshes/touch_sensor.stl"
+                    scale="0.001 0.001 0.001"/>
+                </geometry>
+            </collision>
+            <inertial>
+                <origin xyz="0.0 0.0 0.0" rpy="${rotR} ${rotP} ${rotY}"/>
+                <mass value="0.001984467"/>
+                <inertia ixx="1.3218052332160457e-07" ixy="0.0" ixz="0.0"
+                         iyy="1.0060793220379826e-07" iyz="0.0"
+                         izz="2.2367231024415283e-07"/>
+            </inertial>
+        </link>
+        <joint name="touch_sensor_${prefix}${side}_joint" type="fixed">
+            <origin xyz="${x} ${y} ${z}" rpy="0.0 0.0 0.0"/>
+            <parent link="${parent}"/>
+            <child link="touch_sensor_${prefix}${side}"/>
+        </joint>
+        <xacro:property name="rotR" value="0"/>
+        <xacro:property name="rotP" value="0"/>
+        <xacro:property name="rotY" value="${pi}"/>
+        <xacro:property name="offsetZ" value="-0.0065"/>
+        <xacro:property name="offsetY" value="0.002"/>
+        <xacro:property name="offsetX" value="0"/>
+        <xacro:if value="${side == 2}">
+            <xacro:property name="rotY" value="0"/>
+            <xacro:property name="offsetY" value="-0.002"/>
+        </xacro:if>
+        <xacro:if value="${upper}">
+            <xacro:property name="rotR" value="${-pi_2}"/>
+            <xacro:property name="rotP" value="0"/>
+            <xacro:property name="rotY" value="${-pi_2}"/>
+            <xacro:property name="offsetZ" value="0.00175"/>
+            <xacro:property name="offsetY" value="0"/>
+            <xacro:property name="offsetX" value="-0.0065"/>
+        </xacro:if>
+        <link name="touch_sup_${prefix}${side}">
+            <visual name="">
+                <origin xyz="0 0 0" rpy="${rotR} ${rotP} ${rotY}"/>
+                <geometry>
+                    <mesh filename="package://orion_description/meshes/touch_sensor_sup.stl"
+                    scale="0.001 0.001 0.001"/>
+                </geometry>
+                <material name="PLAWhite"/>
+            </visual>
+            <collision>
+                <origin xyz="0 0 0" rpy="${rotR} ${rotP} ${rotY}"/>
+                <geometry>
+                    <mesh filename="package://orion_description/meshes/touch_sensor_sup.stl"
+                    scale="0.001 0.001 0.001"/>
+                </geometry>
+            </collision>
+            <inertial>
+                <origin xyz="0 0 0" rpy="${rotR} ${rotP} ${rotY}"/>
+                <mass value="0.004"/>
+                <inertia ixx="4.400208333333333e-07" ixy="0.0" ixz="0.0"
+                         iyy="6.019366727956135e-07" iyz="0.0"
+                         izz="2.252908394622803e-07"/>
+            </inertial>
+        </link>
+        <joint name="touch_sup_${prefix}${side}_joint" type="fixed">
+            <origin xyz="${offsetX} ${offsetY} ${offsetZ}" rpy="0 0 0"/>
+            <parent link="touch_sensor_${prefix}${side}"/>
+            <child link="touch_sup_${prefix}${side}"/>
+        </joint>
+    </xacro:macro>
+    <!-- /////////////////////// Cameras macros //////////////////////// -->
     <xacro:macro name="camera_sensor" params="x y z R P Y parent">
         <!-- ................... Camera sensors links .................. -->
