Commit message: Description: Fixed servo moves caused by interference of collisions

File: orion_description/urdf/orion_arms.urdf.xacro (robot description, xacro)
@@ -38,11 +38,11 @@
             <xacro:if value="${gazebo}">
                 <gazebo reference="simple_arm_${side}">
-                    <mu1>1.0</mu1>
-                    <mu2>1.0</mu2>
+                    <mu1>0.0005</mu1>
+                    <mu2>0.0005</mu2>
                 </gazebo>
             </xacro:if>
         </xacro:macro>
-        <xacro:simple_arm x="0" y="0" z="0.003" parent="servo_conn_1" side="1"/>
-        <xacro:simple_arm x="0" y="0" z="0.003" parent="servo_conn_2" side="2"/>
+        <xacro:simple_arm x="0" y="0" z="0.004" parent="servo_conn_1" side="1"/>
+        <xacro:simple_arm x="0" y="0" z="0.004" parent="servo_conn_2" side="2"/>
     </xacro:if>
 </robot>

File: orion_description/urdf/orion_gz.urdf.xacro (robot description, xacro)
@@ -20,6 +20,6 @@
     </gazebo>
     <!-- ////////////////////// JOINT PLUGINS /////////////////////////// -->
-    <gazebo>
-        <!-- ...................... Diff Drive Controller ............... -->
+    <!-- ...................... Diff Drive Controller ............... -->
+    <gazebo>
         <plugin
             filename="gz-sim-diff-drive-system"
@@ -39,18 +39,67 @@
             <min_angular_velocity>-2.791666667</min_angular_velocity>
         </plugin>
-        <!-- ..................... Odometry Publisher ................. -->
-        <gazebo>
-            <plugin
-                filename="gz-sim-odometry-publisher-system"
-                name="gz::sim::systems::OdometryPublisher">
-            </plugin>
-        </gazebo>
+    </gazebo>
+    <!-- ..................... Odometry Publisher ................. -->
+    <gazebo>
+        <plugin
+            filename="gz-sim-odometry-publisher-system"
+            name="gz::sim::systems::OdometryPublisher">
+            <odom_publish_frequency>20</odom_publish_frequency>
+            <robot_base_frame>base_link</robot_base_frame>
+            <odom_frame>odom</odom_frame>
+        </plugin>
+    </gazebo>
+    <!-- .................... Servo controllers ................ -->
+    <gazebo>
+        <plugin
+            filename="gz-sim-joint-position-controller-system"
+            name="gz::sim::systems::JointPositionController">
+            <joint_name>servo_conn1_joint</joint_name>
+            <p_gain>10</p_gain>
+            <i_gain>0.1</i_gain>
+            <d_gain>0.01</d_gain>
+            <i_max>1</i_max>
+            <i_min>-1</i_min>
+            <cmd_max>1000</cmd_max>
+            <cmd_min>-1000</cmd_min>
+        </plugin>
+    </gazebo>
+    <gazebo>
+        <plugin
+            filename="gz-sim-joint-position-controller-system"
+            name="gz::sim::systems::JointPositionController">
+            <joint_name>servo_conn2_joint</joint_name>
+            <p_gain>10</p_gain>
+            <i_gain>0.1</i_gain>
+            <d_gain>0.01</d_gain>
+            <i_max>1</i_max>
+            <i_min>-1</i_min>
+            <cmd_max>1000</cmd_max>
+            <cmd_min>-1000</cmd_min>
+        </plugin>
+    </gazebo>
+    <gazebo>
+        <plugin
+            filename="gz-sim-joint-position-controller-system"
+            name="gz::sim::systems::JointPositionController">
+            <joint_name>g_mov_servo_conn_joint</joint_name>
+            <p_gain>10</p_gain>
+            <i_gain>0.1</i_gain>
+            <d_gain>0.01</d_gain>
+            <i_max>1</i_max>
+            <i_min>-1</i_min>
+            <cmd_max>1000</cmd_max>
+            <cmd_min>-1000</cmd_min>
+        </plugin>
+    </gazebo>
         <!-- ...................... Joint state publisher ................ -->
-        <plugin filename="gz-sim-joint-state-publisher-system" name="gz::sim::systems::JointStatePublisher">
+    <gazebo>
+        <plugin filename="gz-sim-joint-state-publisher-system"
+            name="gz::sim::systems::JointStatePublisher">
             <joint_name>coupling_11_joint</joint_name>
             <joint_name>coupling_12_joint</joint_name>
             <joint_name>caster_middle_2_joint</joint_name>
             <joint_name>caster_wheel_2_joint</joint_name>
-        <xacro:if value="${servo}">
+            <xacro:if value="${servo}">
             <joint_name>servo_conn1_joint</joint_name>
             <joint_name>servo_conn2_joint</joint_name>
@@ -215,4 +264,128 @@
             </sensor>
         </gazebo>
+        <gazebo reference="g_mov_cam_link">
+        <sensor name="camera" type="camera">
+            <!-- Data based on : -->
+            <!-- https://static.chipdip.ru/lib/664/DOC001664108.pdf -->
+            <camera>
+                <horizontal_fov>1.361357</horizontal_fov>
+                <image>
+                <width>1080</width>
+                <height>810</height>
+                </image>
+                <clip>
+                    <near>0.2</near>
+                    <far>10.0</far>
+                </clip>
+                <xacro:if value="true">
+                    <!-- Noise addition -->
+                    <noise>
+                        <type>gaussian</type>
+                        <mean>0.0</mean>
+                        <stddev>0.015</stddev>
+                    </noise>
+                    <!-- Distorsion addition -->
+                    <distortion>
+                        <k1>-0.1</k1>
+                        <k2>0.02</k2>
+                        <k3>0.01</k3>
+                        <p1>0.0</p1>
+                        <p2>0.0</p2>
+                        <center>0.5 0.5</center>
+                    </distortion>
+                </xacro:if>
+            </camera>
+            <always_on>1</always_on>
+            <update_rate>30</update_rate>
+            <visualize>true</visualize>
+        </sensor>
+        </gazebo>
+        <xacro:if value="${g_mov}">
+            <gazebo>
+                <plugin
+                    filename="gz-sim-imu-system"
+                    name="gz::sim::systems::Imu">
+                </plugin>
+            </gazebo>
+            <gazebo reference="imu">
+                <sensor name="imu_sensor" type="imu">
+                    <always_on>1</always_on>
+                    <update_rate>50</update_rate>
+                    <imu>
+                    <enable_orientation>true</enable_orientation>
+                    <angular_velocity>
+                        <x>
+                        <noise type="gaussian">
+                            <mean>0</mean>
+                            <stddev>0.009</stddev>
+                            <bias_mean>0.00075</bias_mean>
+                            <bias_stddev>0.005</bias_stddev>
+                            <dynamic_bias_stddev>0.00002</dynamic_bias_stddev>
+                            <dynamic_bias_correlation_time>400.0</dynamic_bias_correlation_time>
+                            <precision>0.00025</precision>
+                        </noise>
+                        </x>
+                        <y>
+                        <noise type="gaussian">
+                            <mean>0</mean>
+                            <stddev>0.009</stddev>
+                            <bias_mean>0.00075</bias_mean>
+                            <bias_stddev>0.005</bias_stddev>
+                            <dynamic_bias_stddev>0.00002</dynamic_bias_stddev>
+                            <dynamic_bias_correlation_time>400.0</dynamic_bias_correlation_time>
+                            <precision>0.00025</precision>
+                        </noise>
+                        </y>
+                        <z>
+                        <noise type="gaussian">
+                            <mean>0</mean>
+                            <stddev>0.009</stddev>
+                            <bias_mean>0.00075</bias_mean>
+                            <bias_stddev>0.005</bias_stddev>
+                            <dynamic_bias_stddev>0.00002</dynamic_bias_stddev>
+                            <dynamic_bias_correlation_time>400.0</dynamic_bias_correlation_time>
+                            <precision>0.00025</precision>
+                        </noise>
+                        </z>
+                    </angular_velocity>
+                    <linear_acceleration>
+                        <x>
+                        <noise type="gaussian">
+                            <mean>0</mean>
+                            <stddev>0.021</stddev>
+                            <bias_mean>0.05</bias_mean>
+                            <bias_stddev>0.0075</bias_stddev>
+                            <dynamic_bias_stddev>0.000375</dynamic_bias_stddev>
+                            <dynamic_bias_correlation_time>175.0</dynamic_bias_correlation_time>
+                            <precision>0.005</precision>
+                        </noise>
+                        </x>
+                        <y>
+                        <noise type="gaussian">
+                            <mean>0</mean>
+                            <stddev>0.021</stddev>
+                            <bias_mean>0.05</bias_mean>
+                            <bias_stddev>0.0075</bias_stddev>
+                            <dynamic_bias_stddev>0.000375</dynamic_bias_stddev>
+                            <dynamic_bias_correlation_time>175.0</dynamic_bias_correlation_time>
+                            <precision>0.005</precision>
+                        </noise>
+                        </y>
+                        <z>
+                        <noise type="gaussian">
+                            <mean>0</mean>
+                            <stddev>0.021</stddev>
+                            <bias_mean>0.05</bias_mean>
+                            <bias_stddev>0.0075</bias_stddev>
+                            <dynamic_bias_stddev>0.000375</dynamic_bias_stddev>
+                            <dynamic_bias_correlation_time>175.0</dynamic_bias_correlation_time>
+                            <precision>0.005</precision>
+                        </noise>
+                        </z>
+                    </linear_acceleration>
+                    </imu>
+                </sensor>
+            </gazebo>
+        </xacro:if>
     </xacro:if>
 </robot>

File: orion_description/urdf/orion_macros.urdf.xacro (robot description, xacro)
@@ -592,6 +592,6 @@
         </joint>
         <gazebo reference="servo_${side}">
-            <mu1>1.0</mu1>
-            <mu2>1.0</mu2>
+            <mu1>0.05</mu1>
+            <mu2>0.05</mu2>
         </gazebo>
         <!-- Servo Conn -->
@@ -624,11 +624,11 @@
             <parent link="servo_${side}"/>
             <child link="servo_conn_${side}"/>
-            <origin xyz="0.0115 ${0.0431*inv} 0" rpy="${-pi_2*inv} 0 0"/>
-            <limit lower="${-pi_2}" upper="${pi_2}" effort="1.0" velocity="1.0"/>
-            <dynamics damping="0.1" friction="0.01"/>
+            <origin xyz="0.01 ${0.0431*inv} 0" rpy="${-pi_2*inv} 0 0"/>
+            <limit lower="${-pi_2}" upper="${pi_2}" effort="0.92" velocity="6.0"/>
+            <dynamics damping="0.05" friction="0.002"/>
         </joint>
         <gazebo reference="servo_conn_${side}">
-            <mu1>1.0</mu1>
-            <mu2>1.0</mu2>
+            <mu1>0.05</mu1>
+            <mu2>0.05</mu2>
         </gazebo>
     </xacro:macro>
@@ -761,6 +761,6 @@
         </joint>
         <gazebo reference="wall_${id}_${level}_${side}">
-            <mu1>1.0</mu1>
-            <mu2>1.0</mu2>
+            <mu1>0.05</mu1>
+            <mu2>0.05</mu2>
         </gazebo>
     </xacro:macro>

Commit message: Assets: Fixed pieces errors after first assembly and updated manufacturing files | Description: Updates according new assets

File: orion_description/urdf/orion_arms.urdf.xacro (robot description, xacro)
@@ -43,6 +43,6 @@
             </xacro:if>
         </xacro:macro>
-        <xacro:simple_arm x="0" y="0" z="0.004" parent="servo_conn_1" side="1"/>
-        <xacro:simple_arm x="0" y="0" z="0.004" parent="servo_conn_2" side="2"/>
+        <xacro:simple_arm x="0" y="0" z="0.0045" parent="servo_conn_1" side="1"/>
+        <xacro:simple_arm x="0" y="0" z="0.0045" parent="servo_conn_2" side="2"/>
     </xacro:if>
 </robot>

File: orion_description/urdf/orion_base.urdf.xacro (robot description, xacro)
@@ -36,13 +36,13 @@
             y="${0.21/2 - 0.010}" z="0"/>
     <!-- //////////////////////// MOTORS DC ////////////////////////////-->
-    <xacro:motor_dc front="1" side="1" x="-0.0025" y="${0.05718+0.036/2}"
+    <xacro:motor_dc front="1" side="1" x="-0.0025" y="${0.05418+0.036/2}"
         z="-0.0225"/>
-    <xacro:motor_dc front="1" side="2" x="-0.0025" y="${0.05718+0.036/2}"
+    <xacro:motor_dc front="1" side="2" x="-0.0025" y="${0.05418+0.036/2}"
         z="-0.0225"/>
     <!-- /////////////////////// CASTER WHEEL //////////////////////////-->
     <xacro:x4xmetric_spacer id="m4x17" element="caster" parent="base_l0_s2"
-        offset_x="0.012" offset_y="0.015" x="-0.022" y="0"
+        offset_x="0.012" offset_y="0.015" x="-0.023" y="0"
         z="${-0.001 - 0.017}"/>
-    <xacro:caster_wheel parent="base_l0_s2" front="2" x="-0.022" y="0"
+    <xacro:caster_wheel parent="base_l0_s2" front="2" x="-0.023" y="0"
         z="${-0.002 - 0.017}"/>
     <!-- //////////////// FIRST FLOOR COMPONENTS ///////////////////// -->
@@ -167,5 +167,5 @@
         <parent link="base_l0_s2"/>
         <child link="reg_support"/>
-        <origin xyz="-0.036 -0.0275 0.0025" rpy="0 0 0"/>
+        <origin xyz="-0.026 -0.0275 0.0025" rpy="0 0 0"/>
     </joint>
     <xacro:if value="${gazebo}">

File: orion_description/urdf/orion_cameras.urdf.xacro (robot description, xacro)
@@ -170,5 +170,5 @@
             <xacro:include filename="$(find g_mov_description)/urdf/g_mov_macros.urdf.xacro"/>
             <xacro:g_mov_assem parent="${level_cam}" spacer="m3x10" offset="${0.033/2}"
-                x="0.017825" y="0.035" z="0" joint_prefix="g_mov"/>
+                x="0.013825" y="0.035" z="0.0025" joint_prefix="g_mov"/>
         </xacro:if>
         <!-- ......................... Camera sensors links ............................ -->

File: orion_description/urdf/orion_macros.urdf.xacro (robot description, xacro)
@@ -624,5 +624,5 @@
             <parent link="servo_${side}"/>
             <child link="servo_conn_${side}"/>
-            <origin xyz="0.01 ${0.0431*inv} 0" rpy="${-pi_2*inv} 0 0"/>
+            <origin xyz="0.01 ${0.0406*inv} 0" rpy="${-pi_2*inv} 0 0"/>
             <limit lower="${-pi_2}" upper="${pi_2}" effort="0.92" velocity="6.0"/>
             <dynamics damping="0.05" friction="0.002"/>
@@ -709,5 +709,5 @@
             <parent link="speaker_sup_${front}${side}"/>
             <child link="speaker_${front}${side}"/>
-            <origin xyz="0 ${0.0285*muls/2} 0" rpy="0 0 0"/>
+            <origin xyz="0 ${0.0375*muls/2} 0" rpy="0 0 0"/>
         </joint>
         <gazebo reference="speaker_${front}${side}">
