Commit message: Description: Started with robot base platform

File: orion_description/urdf/orion.urdf.xacro (robot description, xacro)
@@ -2,8 +2,8 @@
 <robot xmlns:xacro="http://www.ros.org/wiki/xacro" name="orion">
     <!-- Include other files -->
-    <xacro:include filename="$(find orion_desription)/urdf/orion_materials.urdf.xacro"/>
-    <xacro:include filename="$(find orion_desription)/urdf/orion_macros.urdf.xacro"/>
-    <xacro:include filename="$(find orion_desription)/urdf/orion_base.urdf.xacro"/>
-    <xacro:include filename="$(find orion_desription)/urdf/orion_arms.urdf.xacro"/>
-    <xacro:include filename="$(find orion_desription)/urdf/orion_cameras.urdf.xacro"/>
+    <xacro:include filename="$(find orion_description)/urdf/orion_materials.urdf.xacro"/>
+    <xacro:include filename="$(find orion_description)/urdf/orion_macros.urdf.xacro"/>
+    <xacro:include filename="$(find orion_description)/urdf/orion_base.urdf.xacro"/>
+    <xacro:include filename="$(find orion_description)/urdf/orion_arms.urdf.xacro"/>
+    <xacro:include filename="$(find orion_description)/urdf/orion_cameras.urdf.xacro"/>
 </robot>

File: orion_description/urdf/orion_base.urdf.xacro (robot description, xacro)
@@ -3,3 +3,5 @@
     <!-- This xacro file aims for adding the mobile platform to the robot-->
     <!-- FOR NOW IT IS EMPTY-->
+    <link name="base_link"/>
+    <xacro:generic_base name="base1" parent="base_link" x="0" y="0" z="0"/>
 </robot>

File: orion_description/urdf/orion_macros.urdf.xacro (robot description, xacro)
@@ -91,4 +91,36 @@
         </joint>
     </xacro:macro>
+    <xacro:macro name="generic_base" params="name parent x y z">
+    <!-- Link -->
+        <link name="${name}">
+        <visual>
+            <origin xyz="0 0 0" rpy="0 0 0"/>
+            <geometry>
+            <mesh filename="package://orion_description/meshes/half_platform.stl"
+                scale="0.001 0.001 0.001"/>
+            </geometry>
+        </visual>
+        <collision>
+            <origin xyz="0 0 0" rpy="0 0 0"/>
+            <geometry>
+            <mesh filename="package://orion_description/meshes/half_platform.stl"
+                scale="0.001 0.001 0.001"/>
+            </geometry>
+        </collision>
+        <inertial>
+            <origin xyz="${x} ${y} ${z}"/>
+            <mass value="0.1"/>
+            <inertia ixx="0.001" ixy="0.0" ixz="0.0"
+                    iyy="0.001" iyz="0.0"
+                    izz="0.001"/>
+        </inertial>
+        </link>
+        <!-- Fixed Joint -->
+        <joint name="${name}_joint" type="fixed">
+        <parent link="${parent}"/>
+        <child link="${name}"/>
+        <origin xyz="${x} ${y} ${z}" rpy="0 0 0"/>
+        </joint>
+    </xacro:macro>
     <!--///////////////////// M3 x 10 SPACERS MACROS ///////////////////////-->
     <!-- Hex spacer M3 x 10 macro -->

Commit message: Description: Added modularity/change of cams for astra and os30a

File: orion_description/urdf/orion.urdf.xacro (robot description, xacro)
@@ -1,4 +1,6 @@
 <?xml version="1.0"?>
 <robot xmlns:xacro="http://www.ros.org/wiki/xacro" name="orion">
+    <xacro:property name="camera" default="$(arg camera)"/>
+    <xacro:property name="servo" default="$(arg servo)"/>
     <!-- Include other files -->
     <xacro:include filename="$(find orion_description)/urdf/orion_materials.urdf.xacro"/>

File: orion_description/urdf/orion_base.urdf.xacro (robot description, xacro)
@@ -182,8 +182,10 @@
         <origin xyz="-0.0025 0 ${0.06/2}" rpy="0 0 0"/>
     </joint>
-    <xacro:servo_mounted parent="base_l1_s2" side="1" x="0.00275" y="0.0765"
-        z="-0.026"/>
-    <xacro:servo_mounted parent="base_l1_s2" side="2" x="0.00275" y="0.0765"
-        z="-0.026"/>
+    <xacro:if value="${servo}">
+        <xacro:servo_mounted parent="base_l1_s2" side="1" x="0.00275" y="0.0765"
+            z="-0.026"/>
+        <xacro:servo_mounted parent="base_l1_s2" side="2" x="0.00275" y="0.0765"
+            z="-0.026"/>
+    </xacro:if>
     <!-- ///////////////// SECOND FLOOR COMPONENTS /////////////////////// -->
     <xacro:x4xspacer_m3x10 id="hm3x10" element="espadapter" parent="base_l1_s1"
@@ -323,5 +325,5 @@
     <xacro:x4xspacer_m3x10 id="hm3x10" element="rpi5" parent="base_l3_s2"
         offset_x="${0.049/2}" offset_y="${0.058/2}" x="0" y="0.0435" z="0.0025"/>
-    <!-- Link Lidar Serial -->
+    <!-- Link Rasberry Pi -->
     <link name="rpi5">
     <visual>
@@ -348,5 +350,5 @@
     </inertial>
     </link>
-    <!-- Joint Lidar Serial -->
+    <!-- Joint Rasberry Pi -->
     <joint name="rpi5_joint" type="fixed">
         <parent link="base_l3_s2"/>

File: orion_description/urdf/orion_cameras.urdf.xacro (robot description, xacro)
@@ -1,5 +1,106 @@
 <?xml version="1.0"?>
 <robot xmlns:xacro="http://www.ros.org/wiki/xacro">
-<!-- This xacro file aims for adding the cameras to the robot-->
-<!-- FOR NOW IT IS EMPTY-->
+    <xacro:property name="level_cam" value="base_l2_s1"/>
+    <!--  //////////////////////// ASTRA_S CAM ///////////////////////////// -->
+    <xacro:if value="${camera == 'astra_s'}">
+        <!-- Link Astra S -->
+        <link name="astra">
+        <visual>
+            <origin xyz="0 0 0" rpy="0 0 ${pi_2}"/>
+            <geometry>
+            <mesh filename="package://orion_description/meshes/astra_s.stl"
+                scale="0.001 0.001 0.001"/>
+            </geometry>
+            <material name="SoftBlack"/>
+        </visual>
+        <collision>
+            <origin xyz="0 0 0" rpy="0 0 ${pi_2}"/>
+            <geometry>
+            <mesh filename="package://orion_description/meshes/astra_s.stl"
+                scale="0.001 0.001 0.001"/>
+            </geometry>
+        </collision>
+        <inertial>
+            <origin xyz="0 0 0" rpy="0 0 ${pi_2}"/>
+            <mass value="0.1"/>
+            <inertia ixx="0.001" ixy="0.0" ixz="0.0"
+                    iyy="0.001" iyz="0.0"
+                    izz="0.001"/>
+        </inertial>
+        </link>
+        <!-- Joint Astra S -->
+        <joint name="astra_joint" type="fixed">
+            <parent link="${level_cam}"/>
+            <child link="astra"/>
+            <origin xyz="0.023 0 0.0325" rpy="0 0 0"/>
+        </joint>
+    </xacro:if>
+    <!--  //////////////////////// OS30A CAM ///////////////////////////// -->
+    <xacro:if value="${camera == 'os30a'}">
+        <!-- Link OS30A Support -->
+        <link name="os30a_sup">
+        <visual>
+            <origin xyz="0 0 0" rpy="0 0 ${pi_2}"/>
+            <geometry>
+            <mesh filename="package://orion_description/meshes/os30a_sup.stl"
+                scale="0.001 0.001 0.001"/>
+            </geometry>
+            <material name="SoftBlack"/>
+        </visual>
+        <collision>
+            <origin xyz="0 0 0" rpy="0 0 ${pi_2}"/>
+            <geometry>
+            <mesh filename="package://orion_description/meshes/os30a_sup.stl"
+                scale="0.001 0.001 0.001"/>
+            </geometry>
+        </collision>
+        <inertial>
+            <origin xyz="0 0 0" rpy="0 0 ${pi_2}"/>
+            <mass value="0.1"/>
+            <inertia ixx="0.001" ixy="0.0" ixz="0.0"
+                    iyy="0.001" iyz="0.0"
+                    izz="0.001"/>
+        </inertial>
+        </link>
+        <!-- Joint OS30A Support -->
+        <joint name="os30a_sup_joint" type="fixed">
+            <parent link="${level_cam}"/>
+            <child link="os30a_sup"/>
+            <origin xyz="0.0555 0 0.0025" rpy="0 0 0"/>
+        </joint>
+        <!-- Link OS30A Support -->
+        <link name="os30a">
+        <visual>
+            <origin xyz="0 0 0" rpy="0 0 ${pi_2}"/>
+            <geometry>
+            <mesh filename="package://orion_description/meshes/os30a.stl"
+                scale="0.001 0.001 0.001"/>
+            </geometry>
+            <material name="MetalGray"/>
+        </visual>
+        <collision>
+            <origin xyz="0 0 0" rpy="0 0 ${pi_2}"/>
+            <geometry>
+            <mesh filename="package://orion_description/meshes/os30a.stl"
+                scale="0.001 0.001 0.001"/>
+            </geometry>
+        </collision>
+        <inertial>
+            <origin xyz="0 0 0" rpy="0 0 ${pi_2}"/>
+            <mass value="0.1"/>
+            <inertia ixx="0.001" ixy="0.0" ixz="0.0"
+                    iyy="0.001" iyz="0.0"
+                    izz="0.001"/>
+        </inertial>
+        </link>
+        <!-- Joint OS30A Support -->
+        <joint name="os30a_joint" type="fixed">
+            <parent link="os30a_sup"/>
+            <child link="os30a"/>
+            <origin xyz="0.025 0 0.015" rpy="0 0 0"/>
+        </joint>
+    </xacro:if>
+    <!--  //////////////////////// A010 CAM ///////////////////////////// -->
+    <xacro:if value="${camera == 'a010'}">
+    </xacro:if>
 </robot>

Commit message: Description: Added G-Mov Module and possibility of changing rpi4/% | Assets: Added rpi4 with heatsinks

File: orion_description/urdf/orion.urdf.xacro (robot description, xacro)
@@ -3,4 +3,6 @@
     <xacro:property name="camera" default="$(arg camera)"/>
     <xacro:property name="servo" default="$(arg servo)"/>
+    <xacro:property name="g_mov" default="$(arg g_mov)"/>
+    <xacro:property name="rasp" default="$(arg rasp)"/>
     <!-- Include other files -->
     <xacro:include filename="$(find orion_description)/urdf/orion_materials.urdf.xacro"/>

File: orion_description/urdf/orion_base.urdf.xacro (robot description, xacro)
@@ -338,25 +338,27 @@
         x="${0.115/2}" z="${0.082/2 + 0.0025/2}" level="1"/>
     <!-- ////////////////// THIRD FLOOR COMPONENTES ////////////////////// -->
-    <xacro:speakers_mount parent="base_l2_s2" front="2" side="1" x="-0.0025"
-        y="0.0685" z= "0.0025"/>
-    <xacro:speakers_mount parent="base_l2_s2" front="2" side="2" x="-0.0025"
-        y="0.0685" z= "0.0025"/>
-    <xacro:complete_lateral_wall id="speaker1" parent="base_l2_s1" side="1"
-        x="${-0.115/2}" y="${0.21/2 + 0.0005}" z="${0.082/2 + 0.0025/2}"
-        level="2"/>
-    <xacro:complete_lateral_wall id="speaker2" parent="base_l2_s1" side="2"
-        x="${-0.115/2}" y="${0.21/2 + 0.0005}" z="${0.082/2 + 0.0025/2}"
-        level="2"/>
-    <xacro:complete_front_wall id="fdefault" parent="base_l2_s2" front="2"
-        x="${0.115/2}" z="${0.082/2 + 0.0025/2}" level="2"/>
+    <xacro:if value="${rasp == 'rpi4'}">
+        <xacro:speakers_mount parent="base_l2_s2" front="2" side="1" x="-0.0025"
+            y="0.0685" z= "0.0025"/>
+        <xacro:speakers_mount parent="base_l2_s2" front="2" side="2" x="-0.0025"
+            y="0.0685" z= "0.0025"/>
+        <xacro:complete_lateral_wall id="speaker1" parent="base_l2_s1" side="1"
+            x="${-0.115/2}" y="${0.21/2 + 0.0005}" z="${0.082/2 + 0.0025/2}"
+            level="2"/>
+        <xacro:complete_lateral_wall id="speaker2" parent="base_l2_s1" side="2"
+            x="${-0.115/2}" y="${0.21/2 + 0.0005}" z="${0.082/2 + 0.0025/2}"
+            level="2"/>
+        <xacro:complete_front_wall id="fdefault" parent="base_l2_s2" front="2"
+            x="${0.115/2}" z="${0.082/2 + 0.0025/2}" level="2"/>
+    </xacro:if>
     <!-- ////////////////// FOURTH FLOOR COMPONENTES ////////////////////// -->
     <xacro:x4xspacer_m3x10 id="hm3x10" element="rpi5" parent="base_l3_s2"
         offset_x="${0.049/2}" offset_y="${0.058/2}" x="0" y="0.0435" z="0.0025"/>
     <!-- Link Rasberry Pi -->
-    <link name="rpi5">
-    <visual>
-        <origin xyz="0 0 0" rpy="0 0 ${-pi_2}"/>
-        <geometry>
-        <mesh filename="package://orion_description/meshes/rpi5.stl"
+    <link name="${rasp}">
+    <visual>
+        <origin xyz="0 0 0" rpy="0 0 ${-pi_2}"/>
+        <geometry>
+        <mesh filename="package://orion_description/meshes/${rasp}.stl"
             scale="0.001 0.001 0.001"/>
         </geometry>
@@ -366,20 +368,20 @@
         <origin xyz="0 0 0" rpy="0 0 ${-pi_2}"/>
         <geometry>
-        <mesh filename="package://orion_description/meshes/rpi5.stl"
-            scale="0.001 0.001 0.001"/>
-        </geometry>
-    </collision>
-    <inertial>
-        <origin xyz="0 0 0" rpy="0 0 ${-pi_2}"/>
-        <mass value="0.1"/>
-        <inertia ixx="0.001" ixy="0.0" ixz="0.0"
-                iyy="0.001" iyz="0.0"
-                izz="0.001"/>
-    </inertial>
-    </link>
-    <!-- Joint Rasberry Pi -->
-    <joint name="rpi5_joint" type="fixed">
+        <mesh filename="package://orion_description/meshes/${rasp}.stl"
+            scale="0.001 0.001 0.001"/>
+        </geometry>
+    </collision>
+    <inertial>
+        <origin xyz="0 0 0" rpy="0 0 ${-pi_2}"/>
+        <mass value="0.1"/>
+        <inertia ixx="0.001" ixy="0.0" ixz="0.0"
+                iyy="0.001" iyz="0.0"
+                izz="0.001"/>
+    </inertial>
+    </link>
+    <!-- Joint Rasberry Pi-->
+    <joint name="${rasp}_joint" type="fixed">
         <parent link="base_l3_s2"/>
-        <child link="rpi5"/>
+        <child link="${rasp}"/>
         <origin xyz="0 0.0335 0.0125" rpy="0 0 0"/>
     </joint>

File: orion_description/urdf/orion_cameras.urdf.xacro (robot description, xacro)
@@ -165,4 +165,9 @@
             <origin xyz="0 0 0.0205" rpy="0 0 0"/>
         </joint>
+        <xacro:if value="${g_mov}">
+            <xacro:include filename="$(find g_mov_description)/urdf/g_mov_macros.urdf.xacro"/>
+            <xacro:g_mov_assem parent="${level_cam}" spacer="m3x10" offset="${0.033/2}"
+                x="0.017825" y="0.035" z="0" joint_prefix="g_mov"/>
+        </xacro:if>
     </xacro:if>
 </robot>

File: orion_description/urdf/orion_materials.urdf.xacro (robot description, xacro)
@@ -34,3 +34,7 @@
         <color rgba="0.3 0.3 0.3 0.8"/>
     </material>
+    <!-- Equivalent to RGB(141, 141, 141) -->
+    <material name="PLAGray">
+        <color rgba="0.6 0.6 0.6 1.0"/>
+    </material>
 </robot>

Commit message: Description: Start adding gazebo reference for sim package

File: orion_description/urdf/orion.urdf.xacro (robot description, xacro)
@@ -5,4 +5,5 @@
     <xacro:property name="g_mov" default="$(arg g_mov)"/>
     <xacro:property name="rasp" default="$(arg rasp)"/>
+    <xacro:property name="gazebo" default="$(arg gazebo)"/>
     <!-- Include other files -->
     <xacro:include filename="$(find orion_description)/urdf/orion_materials.urdf.xacro"/>
@@ -11,3 +12,6 @@
     <xacro:include filename="$(find orion_description)/urdf/orion_arms.urdf.xacro"/>
     <xacro:include filename="$(find orion_description)/urdf/orion_cameras.urdf.xacro"/>
+    <xacro:if value="${gazebo}">
+        <xacro:include filename="$(find orion_description)/urdf/orion_gz.urdf.xacro"/>
+    </xacro:if>
 </robot>
