Commit message: Description: Changed colors and added arms | Assets: Created arms and toys

File: orion_description/urdf/orion.urdf.xacro (robot description, xacro)
@@ -6,4 +6,6 @@
     <xacro:property name="rasp" default="$(arg rasp)"/>
     <xacro:property name="gazebo" default="$(arg gazebo)"/>
+    <!-- For colors consider mdf, transparent or pla -->
+    <xacro:property name="color" default="mdf"/>
     <!-- Include other files -->
     <xacro:include filename="$(find orion_description)/urdf/orion_materials.urdf.xacro"/>

File: orion_description/urdf/orion_arms.urdf.xacro (robot description, xacro)
@@ -2,4 +2,47 @@
 <robot xmlns:xacro="http://www.ros.org/wiki/xacro">
 <!-- This xacro file aims for adding the arms to the robot-->
-<!-- FOR NOW IT IS EMPTY-->
+    <xacro:if value="${servo}">
+        <xacro:macro name="simple_arm" params="x y z parent side">
+            <!-- Link Spacer -->
+            <link name="simple_arm_${side}">
+            <visual>
+                <origin xyz="0 0 0" rpy="${-pi_2} 0 0"/>
+                <geometry>
+                <mesh filename="package://orion_description/meshes/simple_arm.stl"
+                    scale="0.001 0.001 0.001"/>
+                </geometry>
+                <material name="PLAWhite"/>
+            </visual>
+            <collision>
+                <origin xyz="0 0 0" rpy="${-pi_2} 0 0"/>
+                <geometry>
+                <mesh filename="package://orion_description/meshes/simple_arm.stl"
+                    scale="0.001 0.001 0.001"/>
+                </geometry>
+            </collision>
+            <inertial>
+                <origin xyz="0.0 0.0 0.0" rpy="${-pi_2} 0.0 0.0"/>
+                <mass value="1"/>
+                <inertia ixx="8.550666163126637e-09" ixy="0" ixz="0"
+                        iyy="8.960721799390997e-09" iyz="0"
+                        izz="4.443388969597693e-09"/>
+            </inertial>
+            </link>
+            <!-- Joint Spacer -->
+            <joint name="simple_arm_${side}_joint" type="fixed">
+                <parent link="${parent}"/>
+                <child link="simple_arm_${side}"/>
+                <origin xyz="${x} ${y} ${z}" rpy="0 0 0"/>
+            </joint>
+            <!-- Gazebo Spacer -->
+            <xacro:if value="${gazebo}">
+                <gazebo reference="simple_arm_${side}">
+                    <mu1>1.0</mu1>
+                    <mu2>1.0</mu2>
+                </gazebo>
+            </xacro:if>
+        </xacro:macro>
+        <xacro:simple_arm x="0" y="0" z="0.003" parent="servo_conn_1" side="1"/>
+        <xacro:simple_arm x="0" y="0" z="0.003" parent="servo_conn_2" side="2"/>
+    </xacro:if>
 </robot>

File: orion_description/urdf/orion_base.urdf.xacro (robot description, xacro)
@@ -59,5 +59,13 @@
             scale="0.001 0.001 0.001"/>
         </geometry>
-        <material name="PureWhite"/>
+        <xacro:if value="${color == 'mdf'}">
+                <material name="MDF"/>
+            </xacro:if>
+            <xacro:if value="${color == 'transparent'}">
+                <material name="TransparentBlack"/>
+            </xacro:if>
+            <xacro:if value="${color == 'pla'}">
+                <material name="PLAWhite"/>
+            </xacro:if>
     </visual>
     <collision>
@@ -139,5 +147,5 @@
             scale="0.001 0.001 0.001"/>
         </geometry>
-        <material name="SoftBlack"/>
+        <material name="PLAWhite"/>
     </visual>
     <collision>
@@ -544,5 +552,13 @@
             scale="0.001 0.001 0.001"/>
         </geometry>
-        <material name="TransparentBlack"/>
+        <xacro:if value="${color == 'mdf'}">
+                <material name="MDF"/>
+            </xacro:if>
+            <xacro:if value="${color == 'transparent'}">
+                <material name="TransparentBlack"/>
+            </xacro:if>
+            <xacro:if value="${color == 'pla'}">
+                <material name="PLAWhite"/>
+            </xacro:if>
     </visual>
     <collision>
@@ -572,5 +588,5 @@
         </gazebo>
     </xacro:if>
-    <!-- ...................... Screen Sup ................................. -->
+    <!-- ...................... Screen ................................. -->
     <link name="screen">
     <visual>

File: orion_description/urdf/orion_gz.urdf.xacro (robot description, xacro)
@@ -14,42 +14,4 @@
     <!-- ////////////////////// JOINT PLUGINS /////////////////////////// -->
     <gazebo>
-        <!-- ...................... Differential Controller ..............-->
-        <plugin filename="gz-sim-diff-drive-system"
-            name="gz::sim::systems::DiffDrive">
-            <right_joint>coupling_12_joint</right_joint>
-            <left_joint>coupling_11_joint</left_joint>
-            <wheel_separation>0.21</wheel_separation>
-            <wheel_radius>0.03</wheel_radius>
-            <max_linear_acceleration>0.1</max_linear_acceleration>
-            <odom_publish_frequency>100</odom_publish_frequency>
-            <topic>cmd_vel</topic>
-            <odom_topic>odom</odom_topic>
-        </plugin>
-        <plugin
-            filename="gz-sim-joint-position-controller-system"
-            name="gz::sim::systems::JointPositionController">
-            <joint_name>servo_conn1_joint</joint_name>
-            <topic>servo_conn1</topic>
-            <p_gain>1</p_gain>
-            <i_gain>0.1</i_gain>
-            <d_gain>0.01</d_gain>
-            <i_max>1</i_max>
-            <i_min>-1</i_min>
-            <cmd_max>1000</cmd_max>
-            <cmd_min>-1000</cmd_min>
-        </plugin>
-        <plugin
-            filename="gz-sim-joint-position-controller-system"
-            name="gz::sim::systems::JointPositionController">
-            <joint_name>servo_conn2_joint</joint_name>
-            <topic>servo_conn2</topic>
-            <p_gain>1</p_gain>
-            <i_gain>0.1</i_gain>
-            <d_gain>0.01</d_gain>
-            <i_max>1</i_max>
-            <i_min>-1</i_min>
-            <cmd_max>1000</cmd_max>
-            <cmd_min>-1000</cmd_min>
-        </plugin>
         <!-- ...................... Joint state publisher ................ -->
         <plugin filename="gz-sim-joint-state-publisher-system" name="gz::sim::systems::JointStatePublisher">
@@ -57,11 +19,11 @@
             <joint_name>coupling_11_joint</joint_name>
             <joint_name>coupling_12_joint</joint_name>
-            <xacro:if value="${servo}">
-                <joint_name>servo_conn1_joint</joint_name>
-                <joint_name>servo_conn2_joint</joint_name>
-            </xacro:if>
-            <xacro:if value="${camera == 'a010' and g_mov}">
-                <joint_name>g_mov_servo_conn_joint</joint_name>
-            </xacro:if>
+        <xacro:if value="${servo}">
+            <joint_name>servo_conn1_joint</joint_name>
+            <joint_name>servo_conn2_joint</joint_name>
+        </xacro:if>
+        <xacro:if value="${camera == 'a010' and g_mov}">
+            <joint_name>g_mov_servo_conn_joint</joint_name>
+        </xacro:if>
         </plugin>
     </gazebo>

File: orion_description/urdf/orion_macros.urdf.xacro (robot description, xacro)
@@ -36,5 +36,5 @@
                 scale="0.001 0.001 0.001"/>
             </geometry>
-            <material name="SoftBlack"/>
+            <material name="PLAWhite"/>
         </visual>
         <collision>
@@ -86,5 +86,13 @@
                 scale="0.001 0.001 0.001"/>
             </geometry>
-            <material name="PureWhite"/>
+            <xacro:if value="${color == 'mdf'}">
+                <material name="MDF"/>
+            </xacro:if>
+            <xacro:if value="${color == 'transparent'}">
+                <material name="TransparentBlack"/>
+            </xacro:if>
+            <xacro:if value="${color == 'pla'}">
+                <material name="PLAWhite"/>
+            </xacro:if>
         </visual>
         <collision>
@@ -527,5 +535,5 @@
                 scale="0.001 0.001 0.001"/>
             </geometry>
-            <material name="SoftBlack"/>
+            <material name="PLAWhite"/>
         </visual>
         <collision>
@@ -647,5 +655,5 @@
                 scale="0.001 0.001 0.001"/>
             </geometry>
-            <material name="SoftBlack"/>
+            <material name="PLAWhite"/>
         </visual>
         <collision>
@@ -722,5 +730,13 @@
                 scale="0.001 0.001 0.001"/>
             </geometry>
-            <material name="TransparentBlack"/>
+            <xacro:if value="${color == 'mdf'}">
+                <material name="MDF"/>
+            </xacro:if>
+            <xacro:if value="${color == 'transparent'}">
+                <material name="TransparentBlack"/>
+            </xacro:if>
+            <xacro:if value="${color == 'pla'}">
+                <material name="PLAWhite"/>
+            </xacro:if>
         </visual>
         <collision>
@@ -765,5 +781,13 @@
                 scale="0.001 0.001 0.001"/>
             </geometry>
-            <material name="TransparentBlack"/>
+            <xacro:if value="${color == 'mdf'}">
+                <material name="MDF"/>
+            </xacro:if>
+            <xacro:if value="${color == 'transparent'}">
+                <material name="TransparentBlack"/>
+            </xacro:if>
+            <xacro:if value="${color == 'pla'}">
+                <material name="PLAWhite"/>
+            </xacro:if>
         </visual>
         <collision>

File: orion_description/urdf/orion_materials.urdf.xacro (robot description, xacro)
@@ -22,4 +22,8 @@
         <color rgba="1.0 1.0 1.0 1.0"/>
     </material>
+    <!-- Equivalent to RGB(240, 240, 225) -->
+    <material name="PLAWhite">
+        <color rgba="0.95 0.95 0.90 1.0"/>
+    </material>
     <!-- Equivalent to RGB(181, 165, 66) -->
     <material name="Brass">
@@ -38,3 +42,7 @@
         <color rgba="0.6 0.6 0.6 1.0"/>
     </material>
+    <!-- Equivalent to RGB(187, 133, 89) -->
+    <material name="MDF">
+        <color rgba="0.72 0.52 0.35 1.0"/>
+    </material>
 </robot>

Commit message: Decription: Divided gz elements and start integrating ros2_control

File: orion_description/urdf/orion.urdf.xacro (robot description, xacro)
@@ -6,4 +6,5 @@
     <xacro:property name="rasp" default="$(arg rasp)"/>
     <xacro:property name="gazebo" default="$(arg gazebo)"/>
+    <xacro:property name="ros2_control" default="true"/>
     <!-- For colors consider mdf, transparent or pla -->
     <xacro:property name="color" default="mdf"/>
@@ -15,5 +16,6 @@
     <xacro:include filename="$(find orion_description)/urdf/orion_cameras.urdf.xacro"/>
     <xacro:if value="${gazebo}">
-        <xacro:include filename="$(find orion_description)/urdf/orion_gz.urdf.xacro"/>
+        <xacro:include filename="$(find orion_description)/urdf/orion_gz_sensors.urdf.xacro"/>
+        <xacro:include filename="$(find orion_description)/urdf/orion_gz_actuators.urdf.xacro"/>
     </xacro:if>
 </robot>

File: orion_description/urdf/orion_base.urdf.xacro (robot description, xacro)
@@ -486,13 +486,4 @@
             </gazebo>
         </xacro:if>
-        <!-- ........................ Touch sensors ........................ -->
-        <xacro:touch_sensor x="0.005" y="0.1075" z="0.0825" upper="0" side="1"
-            parent="base_l2_s2" prefix="2"/>
-        <xacro:touch_sensor x="0.005" y="-0.1075" z="0.0825" upper="0" side="2"
-            parent="base_l2_s2" prefix="2"/>
-        <xacro:touch_sensor x="0.0425" y="0.0335" z="0.0025" upper="1" side="1"
-            parent="base_l4_s2" prefix="4"/>
-        <xacro:touch_sensor x="0.0425" y="-0.0335" z="0.0025" upper="1" side="2"
-            parent="base_l4_s2" prefix="4"/>
         <!-- ........................ Wall definitions ...................... -->
         <xacro:complete_lateral_wall id="curve" parent="base_l2_s1" side="1"
@@ -544,4 +535,13 @@
         </gazebo>
     </xacro:if>
+    <!-- ........................ Touch sensors ........................ -->
+    <xacro:touch_sensor x="0.005" y="0.1075" z="0.0825" upper="0" side="1"
+        parent="base_l2_s2" prefix="2"/>
+    <xacro:touch_sensor x="0.005" y="-0.1075" z="0.0825" upper="0" side="2"
+        parent="base_l2_s2" prefix="2"/>
+    <xacro:touch_sensor x="0.0425" y="0.0335" z="0.0025" upper="1" side="1"
+        parent="base_l4_s2" prefix="4"/>
+    <xacro:touch_sensor x="0.0425" y="-0.0335" z="0.0025" upper="1" side="2"
+        parent="base_l4_s2" prefix="4"/>
     <!-- ......................... Walls definitions ............................ -->
     <xacro:complete_lateral_wall id="screen" parent="base_l3_s1" side="1"

File: orion_description/urdf/orion_gz_sensors.urdf.xacro (robot description, xacro)
@@ -10,105 +10,4 @@
 			name="gz::sim::systems::Sensors">
 			<render_engine>ogre2</render_engine>
-        </plugin>
-    </gazebo>
-    <!-- ////////////////////// JOINT PLUGINS /////////////////////////// -->
-    <!-- ...................... Diff Drive Controller ............... -->
-    <gazebo>
-        <plugin
-            filename="gz-sim-diff-drive-system"
-            name="gz::sim::systems::DiffDrive">
-            <left_joint>coupling_11_joint</left_joint>
-            <right_joint>coupling_12_joint</right_joint>
-            <wheel_separation>0.1597</wheel_separation>
-            <wheel_radius>${0.0335/2}</wheel_radius>
-            <odom_publish_frequency>1</odom_publish_frequency>
-            <max_linear_acceleration>1</max_linear_acceleration>
-            <min_linear_acceleration>-1</min_linear_acceleration>
-            <max_angular_acceleration>2</max_angular_acceleration>
-            <min_angular_acceleration>-2</min_angular_acceleration>
-            <max_linear_velocity>2.791666667</max_linear_velocity>
-            <min_linear_velocity>-2.791666667</min_linear_velocity>
-            <max_angular_velocity>2.791666667</max_angular_velocity>
-            <min_angular_velocity>-2.791666667</min_angular_velocity>
-            <odom_topic>/unused/diff_drive_odometry</odom_topic>
-            <tf_topic>/unused/diff_drive_tf</tf_topic>
-            <odom_publish_frequency>1</odom_publish_frequency>
-            <frame_id>odom_diff_drive</frame_id>
-            <child_frame_id>base_link</child_frame_id>
-        </plugin>
-    </gazebo>
-    <!-- ..................... Odometry Publisher ................. -->
-    <gazebo>
-        <plugin
-            filename="gz-sim-odometry-publisher-system"
-            name="gz::sim::systems::OdometryPublisher">
-            <odom_publish_frequency>20</odom_publish_frequency>
-            <robot_base_frame>base_link</robot_base_frame>
-            <odom_frame>odom</odom_frame>
-            <dimensions>2</dimensions>
-        </plugin>
-    </gazebo>
-    <!-- .................... Servo controllers ................ -->
-    <xacro:if value="${servo}">
-        <gazebo>
-            <plugin
-                filename="gz-sim-joint-position-controller-system"
-                name="gz::sim::systems::JointPositionController">
-                <joint_name>servo_conn1_joint</joint_name>
-                <p_gain>10</p_gain>
-                <i_gain>0.1</i_gain>
-                <d_gain>0.01</d_gain>
-                <i_max>1</i_max>
-                <i_min>-1</i_min>
-                <cmd_max>1000</cmd_max>
-                <cmd_min>-1000</cmd_min>
-            </plugin>
-        </gazebo>
-        <gazebo>
-            <plugin
-                filename="gz-sim-joint-position-controller-system"
-                name="gz::sim::systems::JointPositionController">
-                <joint_name>servo_conn2_joint</joint_name>
-                <p_gain>10</p_gain>
-                <i_gain>0.1</i_gain>
-                <d_gain>0.01</d_gain>
-                <i_max>1</i_max>
-                <i_min>-1</i_min>
-                <cmd_max>1000</cmd_max>
-                <cmd_min>-1000</cmd_min>
-            </plugin>
-        </gazebo>
-    </xacro:if>
-    <xacro:if value="${camera == 'a010' and g_mov}">
-        <gazebo>
-            <plugin
-                filename="gz-sim-joint-position-controller-system"
-                name="gz::sim::systems::JointPositionController">
-                <joint_name>g_mov_servo_conn_joint</joint_name>
-                <p_gain>10</p_gain>
-                <i_gain>0.1</i_gain>
-                <d_gain>0.01</d_gain>
-                <i_max>1</i_max>
-                <i_min>-1</i_min>
-                <cmd_max>1000</cmd_max>
-                <cmd_min>-1000</cmd_min>
-            </plugin>
-        </gazebo>
-    </xacro:if>
-        <!-- ...................... Joint state publisher ................ -->
-    <gazebo>
-        <plugin filename="gz-sim-joint-state-publisher-system"
-            name="gz::sim::systems::JointStatePublisher">
-            <joint_name>coupling_11_joint</joint_name>
-            <joint_name>coupling_12_joint</joint_name>
-            <joint_name>caster_middle_2_joint</joint_name>
-            <joint_name>caster_wheel_2_joint</joint_name>
-        <xacro:if value="${servo}">
-            <joint_name>servo_conn1_joint</joint_name>
-            <joint_name>servo_conn2_joint</joint_name>
-        </xacro:if>
-        <xacro:if value="${camera == 'a010' and g_mov}">
-            <joint_name>g_mov_servo_conn_joint</joint_name>
-        </xacro:if>
         </plugin>
     </gazebo>
@@ -156,7 +55,8 @@
         <gazebo reference="camera_link">
             <sensor name="camera" type="rgbd_camera">
-                <gz_frame_id>camera_link_optical</gz_frame_id>
+                <optical_frame_id>camera_link_optical</optical_frame_id>
                 <!-- Data based on https://store.orbbec.com/products/astra-s -->
                 <camera>
+                    <gz_frame_id>camera_link</gz_frame_id>
                     <horizontal_fov>1.1013</horizontal_fov>
                     <image>

Commit message: README: First notes about usage of ORION description package

File: orion_description/urdf/orion.urdf.xacro (robot description, xacro)
@@ -6,5 +6,5 @@
     <xacro:property name="rasp" default="$(arg rasp)"/>
     <xacro:property name="gazebo" default="$(arg gazebo)"/>
-    <xacro:property name="ros2_control" default="true"/>
+    <xacro:property name="ros2_control" default="false"/>
     <!-- For colors consider mdf, transparent or pla -->
     <xacro:property name="color" default="mdf"/>

Commit message: Description: Modified launches for param of ros2_control

File: orion_description/urdf/orion.urdf.xacro (robot description, xacro)
@@ -6,5 +6,5 @@
     <xacro:property name="rasp" default="$(arg rasp)"/>
     <xacro:property name="gazebo" default="$(arg gazebo)"/>
-    <xacro:property name="ros2_control" default="false"/>
+    <xacro:property name="ros2_control" default="$(arg ros2_control)"/>
     <!-- For colors consider mdf, transparent or pla -->
     <xacro:property name="color" default="mdf"/>

Commit message: Description: Added ros2_control plugin | Control: Finished hardware_interface | Bringup: Single bringup for diff base

File: orion_description/urdf/orion.urdf.xacro (robot description, xacro)
@@ -8,4 +8,5 @@
     <xacro:property name="ros2_control" default="$(arg ros2_control)"/>
     <xacro:property name="simplified" default="$(arg simplified)"/>
+    <xacro:property name="ctl_type" default="micro_ros"/>
     <!-- For colors consider mdf, transparent or pla -->
     <xacro:property name="color" default="mdf"/>
@@ -16,3 +17,4 @@
     <xacro:include filename="$(find orion_description)/urdf/include/orion_arms.urdf.xacro"/>
     <xacro:include filename="$(find orion_description)/urdf/include/orion_cameras.urdf.xacro"/>
+    <xacro:include filename="$(find orion_description)/urdf/include/orion_ros2_control.urdf.xacro"/>
 </robot>

Commit message: Bringup: Fixed meshes path for real robot | Description: Change of color for ORION

File: orion_description/urdf/orion.urdf.xacro (robot description, xacro)
@@ -11,5 +11,5 @@
     <xacro:property name="ctl_type" default="micro_ros"/>
     <!-- For colors consider mdf, transparent or pla -->
-    <xacro:property name="color" default="mdf"/>
+    <xacro:property name="color" default="pla"/>
     <!-- Include other files -->
     <xacro:include filename="$(find orion_description)/urdf/include/orion_materials.urdf.xacro"/>
