Commit message: Base: Fixed servo sub/pub with µ-ros | Control: Added hardware interface for servo | Description: Added ros2_control tags for servo | Bringup: Added new controllers to launch file

File: orion_description/urdf/include/orion_ros2_control.urdf.xacro (robot description, xacro)
@@ -3,5 +3,5 @@
     <xacro:if value="${ros2_control}">
         <xacro:if value="${ctl_type == 'micro_ros'}">
-            <ros2_control name="RealRobot" type="system">
+            <ros2_control name="DiffRealRobot" type="system">
                 <hardware>
                     <plugin>orion_control/DiffDriveOrion</plugin>
@@ -27,4 +27,30 @@
                 </joint>
             </ros2_control>
+            <xacro:if value="${servo}">
+                <ros2_control name="FwdLeftRealRobot" type="system">
+                    <hardware>
+                        <plugin>orion_control/ForwardOrion</plugin>
+                        <param name="feedback_topic">fwd_servo_left_feedback</param>
+                        <param name="cmd_topic">fwd_servo_left_cmd</param>
+                        <param name="servo_name">servo_conn1_joint</param>
+                    </hardware>
+                    <joint name="servo_conn1_joint">
+                        <command_interface name="position" />
+                        <state_interface name="position" />
+                    </joint>
+                </ros2_control>
+                <ros2_control name="FwdRightRealRobot" type="system">
+                    <hardware>
+                        <plugin>orion_control/ForwardOrion</plugin>
+                        <param name="feedback_topic">fwd_servo_right_feedback</param>
+                        <param name="cmd_topic">fwd_servo_right_cmd</param>
+                        <param name="servo_name">servo_conn2_joint</param>
+                    </hardware>
+                    <joint name="servo_conn2_joint">
+                        <command_interface name="position" />
+                        <state_interface name="position" />
+                    </joint>
+                </ros2_control>
+            </xacro:if>
         </xacro:if>
     </xacro:if>

Commit message: Base: Updating PlatformIO code for actuators | Description: Added new ros2_control param based on motor enc count

File: orion_description/urdf/include/orion_ros2_control.urdf.xacro (robot description, xacro)
@@ -1,4 +1,5 @@
 <?xml version="1.0"?>
 <robot xmlns:xacro="http://www.ros.org/wiki/xacro">
+    <xacro:property name="motor" value="100"/>
     <xacro:if value="${ros2_control}">
         <xacro:if value="${ctl_type == 'micro_ros'}">
@@ -8,5 +9,10 @@
                     <param name="left_wheel_name">coupling_11_joint</param>
                     <param name="right_wheel_name">coupling_12_joint</param>
-                    <param name="enc_ticks_per_rev">204</param>
+                    <xacro:if value="${motor == 1000}">
+                        <param name="enc_ticks_per_rev">204</param>
+                    </xacro:if>
+                    <xacro:if value="${motor == 100}">
+                        <param name="enc_ticks_per_rev">1250</param>
+                    </xacro:if>
                 </hardware>
                 <joint name="coupling_11_joint">
