Commit message: Assets: Modified wall batteries and base platform | Description: Updated changes based on built robot

File: orion_description/urdf/include/orion_base.urdf.xacro (robot description, xacro)
@@ -239,5 +239,5 @@
         <parent link="base_l1_s1"/>
         <child link="switch"/>
-        <origin xyz="0.025 0.074 -0.015" rpy="0 0 0"/>
+        <origin xyz="0.035 0.074 -0.015" rpy="0 0 0"/>
     </joint>
     <xacro:if value="${gazebo}">
@@ -260,6 +260,6 @@
     <!-- ///////////////// SECOND FLOOR COMPONENTS /////////////////////// -->
     <!-- ..................... Spacers for esp32 adp ..................... -->
-    <xacro:x4xmetric_spacer id="m3x10" element="esp_adapter" parent="base_l1_s1"
-        offset_x="${0.0577/2}" offset_y="${0.0607/2}" x="0" y="0" z="-0.01"/>
+    <xacro:x4xmetric_spacer id="m3x10" element="esp_adapter" parent="base_l1_s2"
+        offset_x="${0.0577/2}" offset_y="${0.0607/2}" x="0.004" y="0" z="-0.01"/>
     <!-- .......................... Esp32 Adapter ....................... -->
     <link name="esp32_adapter">
@@ -288,7 +288,7 @@
     </link>
     <joint name="esp32_adapter_joint" type="fixed">
-        <parent link="base_l1_s1"/>
+        <parent link="base_l1_s2"/>
         <child link="esp32_adapter"/>
-        <origin xyz="0 0 -0.01" rpy="0 0 0"/>
+        <origin xyz="0.004 0 -0.01" rpy="0 0 0"/>
     </joint>
     <xacro:if value="${gazebo}">
@@ -497,5 +497,5 @@
     </xacro:if>
     <!-- ////////////////// FOURTH FLOOR COMPONENTES ////////////////////// -->
-    <xacro:x4xmetric_spacer id="m3x10" element="rpi5" parent="base_l3_s2"
+    <xacro:x4xmetric_spacer id="m3x10" element="${rasp}" parent="base_l3_s2"
         offset_x="${0.049/2}" offset_y="${0.058/2}" x="0" y="0.0435" z="0.0025"/>
     <!-- Link Rasberry Pi -->
@@ -553,4 +553,80 @@
     <xacro:complete_front_wall id="rpi" parent="base_l3_s2" front="2"
         x="${0.115/2}" z="${0.082/2 + 0.0025/2}" level="3"/>
+    <!-- ............................ 2° ESP32 ................................ -->
+    <!-- ..................... Spacers for esp32 adp ..................... -->
+    <xacro:x4xmetric_spacer id="m3x10" element="esp_2_adapter" parent="base_l3_s1"
+        offset_x="${0.0577/2}" offset_y="${0.0607/2}" x="0.004" y="0" z="0.0025"/>
+    <!-- .......................... Esp32 Adapter ....................... -->
+    <link name="esp32_2_adapter">
+    <visual>
+        <origin xyz="0 0 0" rpy="0 0 0"/>
+        <geometry>
+        <mesh filename="package://orion_description/meshes/esp32_adp.stl"
+            scale="0.001 0.001 0.001"/>
+        </geometry>
+        <material name="RaspberryGreen"/>
+    </visual>
+    <collision>
+        <origin xyz="0 0 0" rpy="0 0 0"/>
+        <geometry>
+        <mesh filename="package://orion_description/meshes/esp32_adp.stl"
+            scale="0.001 0.001 0.001"/>
+        </geometry>
+    </collision>
+    <inertial>
+        <origin xyz="0 0 0" rpy="0 0 0"/>
+        <mass value="0.030"/>
+        <inertia ixx="1.1184306270694732e-05" ixy="0.0" ixz="0.0"
+                iyy="1.021680627069473e-05" iyz="0.0"
+                izz="2.0812499999999994e-05"/>
+    </inertial>
+    </link>
+    <joint name="esp32_2_adapter_joint" type="fixed">
+        <parent link="base_l3_s1"/>
+        <child link="esp32_2_adapter"/>
+        <origin xyz="0.004 0 0.0125" rpy="0 0 0"/>
+    </joint>
+    <xacro:if value="${gazebo}">
+        <gazebo reference="esp32_adapter">
+            <mu1>1.0</mu1>
+            <mu2>1.0</mu2>
+        </gazebo>
+    </xacro:if>
+    <!-- ....................... ESP32 ....................................... -->
+    <link name="esp32_2">
+    <visual>
+        <origin xyz="0 0 0" rpy="0 0 ${-pi_2}"/>
+        <geometry>
+        <mesh filename="package://orion_description/meshes/esp32.stl"
+            scale="0.001 0.001 0.001"/>
+        </geometry>
+        <material name="SoftBlack"/>
+    </visual>
+    <collision>
+        <origin xyz="0 0 0" rpy="0 0 ${-pi_2}"/>
+        <geometry>
+        <mesh filename="package://orion_description/meshes/esp32.stl"
+            scale="0.001 0.001 0.001"/>
+        </geometry>
+    </collision>
+    <inertial>
+        <origin xyz="0 0 0" rpy="0 0 ${-pi_2}"/>
+        <mass value="0.0201"/>
+        <inertia ixx="4.904162034278915e-06" ixy="0.0" ixz="0.0"
+                iyy="1.5830928543782435e-06" iyz="0.0"
+                izz="6.0040505352397235e-06"/>
+    </inertial>
+    </link>
+    <joint name="esp32_2_joint" type="fixed">
+        <parent link="esp32_2_adapter"/>
+        <child link="esp32_2"/>
+        <origin xyz="0.002 0 0.01" rpy="0 0 0"/>
+    </joint>
+    <xacro:if value="${gazebo}">
+        <gazebo reference="esp32">
+            <mu1>1.0</mu1>
+            <mu2>1.0</mu2>
+        </gazebo>
+    </xacro:if>
     <!-- .......................... Screen Sup ................................ -->
     <link name="screen_sup">

Commit message: Description: Added simplified option, to consider cases with non-functional components for desc/sim

File: orion_description/urdf/include/orion_base.urdf.xacro (robot description, xacro)
@@ -42,89 +42,90 @@
     <!-- /////////////////////// CASTER WHEEL //////////////////////////-->
     <xacro:x4xmetric_spacer id="m4x17" element="caster" parent="base_l0_s2"
-        offset_x="0.012" offset_y="0.015" x="-0.023" y="0"
-        z="${-0.001 - 0.017}"/>
+    offset_x="0.012" offset_y="0.015" x="-0.023" y="0"
+    z="${-0.001 - 0.017}"/>
     <xacro:caster_wheel parent="base_l0_s2" front="2" x="-0.023" y="0"
-        z="${-0.002 - 0.017}"/>
+    z="${-0.002 - 0.017}"/>
     <!-- //////////////// FIRST FLOOR COMPONENTS ///////////////////// -->
-    <!-- .................. Hex spacers for stack .................... -->
-    <xacro:x6xmetric_spacer id="m3x10" element="bathol" parent="base_l0_s1"
-        offset_x="${0.0855/2}" offset_y="${0.127/2}" x="0.005" y="0"
-        z="0.0025"/>
-    <!-- ..................... Battery Platform ....................... -->
-    <link name="bat_platform">
-    <visual>
-        <origin xyz="0 0 0" rpy="0 0 ${pi_2}"/>
-        <geometry>
-        <mesh filename="package://orion_description/meshes/bathold_support.stl"
-            scale="0.001 0.001 0.001"/>
-        </geometry>
-        <xacro:if value="${color == 'mdf'}">
-                <material name="MDF"/>
-            </xacro:if>
-            <xacro:if value="${color == 'transparent'}">
-                <material name="TransparentBlack"/>
-            </xacro:if>
-            <xacro:if value="${color == 'pla'}">
-                <material name="PLAWhite"/>
-            </xacro:if>
-    </visual>
-    <collision>
-        <origin xyz="0 0 0" rpy="0 0 ${pi_2}"/>
-        <geometry>
-        <mesh filename="package://orion_description/meshes/bathold_support.stl"
-            scale="0.001 0.001 0.001"/>
-        </geometry>
-    </collision>
-    <inertial>
-        <origin xyz="0 0 0" rpy="0 0 ${pi_2}"/>
-        <mass value="0.018"/>
-        <inertia ixx="1.2564374999999998e-05" ixy="0.0" ixz="0.0"
-                iyy="2.6539499999999996e-05" iyz="0.0"
-                izz="3.9091874999999996e-05"/>
-    </inertial>
-    </link>
-    <joint name="bat_platform_joint" type="fixed">
-        <parent link="base_l0_s1"/>
-        <child link="bat_platform"/>
-        <origin xyz="0.005 0 0.0125" rpy="0 0 0"/>
-    </joint>
-    <xacro:if value="${gazebo}">
-        <gazebo reference="bat_platform">
-            <mu1>1.0</mu1>
-            <mu2>1.0</mu2>
-        </gazebo>
-    </xacro:if>
-    <!-- ....................... Battery Stacks ........................ -->
-    <xacro:stack_bat parent="bat_platform" num="1" x="0" y="-0.023" z="0.0025"/>
-    <xacro:stack_bat parent="bat_platform" num="2" x="0" y="${0.023+0.02}"
-        z="0.0025"/>
-    <!-- ............... Hex spacers for Motor Driver................... -->
-    <xacro:x4xmetric_spacer id="m3x10" element="driver" parent="base_l0_s2"
+    <xacro:unless value="${simplified}">
+        <!-- .................. Hex spacers for stack .................... -->
+        <xacro:x6xmetric_spacer id="m3x10" element="bathol" parent="base_l0_s1"
+            offset_x="${0.0855/2}" offset_y="${0.127/2}" x="0.005" y="0"
+            z="0.0025"/>
+        <!-- ..................... Battery Platform ....................... -->
+        <link name="bat_platform">
+        <visual>
+            <origin xyz="0 0 0" rpy="0 0 ${pi_2}"/>
+            <geometry>
+            <mesh filename="package://orion_description/meshes/bathold_support.stl"
+                scale="0.001 0.001 0.001"/>
+            </geometry>
+            <xacro:if value="${color == 'mdf'}">
+                    <material name="MDF"/>
+                </xacro:if>
+                <xacro:if value="${color == 'transparent'}">
+                    <material name="TransparentBlack"/>
+                </xacro:if>
+                <xacro:if value="${color == 'pla'}">
+                    <material name="PLAWhite"/>
+                </xacro:if>
+        </visual>
+        <collision>
+            <origin xyz="0 0 0" rpy="0 0 ${pi_2}"/>
+            <geometry>
+            <mesh filename="package://orion_description/meshes/bathold_support.stl"
+                scale="0.001 0.001 0.001"/>
+            </geometry>
+        </collision>
+        <inertial>
+            <origin xyz="0 0 0" rpy="0 0 ${pi_2}"/>
+            <mass value="0.018"/>
+            <inertia ixx="1.2564374999999998e-05" ixy="0.0" ixz="0.0"
+                    iyy="2.6539499999999996e-05" iyz="0.0"
+                    izz="3.9091874999999996e-05"/>
+        </inertial>
+        </link>
+        <joint name="bat_platform_joint" type="fixed">
+            <parent link="base_l0_s1"/>
+            <child link="bat_platform"/>
+            <origin xyz="0.005 0 0.0125" rpy="0 0 0"/>
+        </joint>
+        <xacro:if value="${gazebo}">
+            <gazebo reference="bat_platform">
+                <mu1>1.0</mu1>
+                <mu2>1.0</mu2>
+            </gazebo>
+        </xacro:if>
+        <!-- ....................... Battery Stacks ........................ -->
+        <xacro:stack_bat parent="bat_platform" num="1" x="0" y="-0.023" z="0.0025"/>
+        <xacro:stack_bat parent="bat_platform" num="2" x="0" y="${0.023+0.02}"
+            z="0.0025"/>
+        <!-- ............... Hex spacers for Motor Driver................... -->
+        <xacro:x4xmetric_spacer id="m3x10" element="driver" parent="base_l0_s2"
         offset_x="${0.03702/2}" offset_y="${-0.0368/2}" x="-0.023453"
         y="0.031351" z="0.0025"/>
-    <!-- ......................... Motor Driver ........................ -->
-    <link name="driver">
-    <visual>
-        <origin xyz="0 0 0" rpy="0 0 0"/>
-        <geometry>
-        <mesh filename="package://orion_description/meshes/driver.stl"
-            scale="0.001 0.001 0.001"/>
-        </geometry>
-        <material name="DriverRed"/>
-    </visual>
-    <collision>
-        <origin xyz="0 0 0" rpy="0 0 0"/>
-        <geometry>
-        <mesh filename="package://orion_description/meshes/driver.stl"
-            scale="0.001 0.001 0.001"/>
-        </geometry>
-    </collision>
-    <inertial>
-        <origin xyz="0 0 0" rpy="0 0 0"/>
-        <mass value="0.026"/>
-        <inertia ixx="5.575206798350021e-06" ixy="0.0" ixz="0.0"
+        <!-- ......................... Motor Driver ........................ -->
+        <link name="driver">
+            <visual>
+                <origin xyz="0 0 0" rpy="0 0 0"/>
+                <geometry>
+                    <mesh filename="package://orion_description/meshes/driver.stl"
+                    scale="0.001 0.001 0.001"/>
+                </geometry>
+                <material name="DriverRed"/>
+            </visual>
+            <collision>
+                <origin xyz="0 0 0" rpy="0 0 0"/>
+                <geometry>
+                    <mesh filename="package://orion_description/meshes/driver.stl"
+                    scale="0.001 0.001 0.001"/>
+                </geometry>
+            </collision>
+            <inertial>
+                <origin xyz="0 0 0" rpy="0 0 0"/>
+                <mass value="0.026"/>
+                <inertia ixx="5.575206798350021e-06" ixy="0.0" ixz="0.0"
                 iyy="5.588291024131272e-06" iyz="0.0"
                 izz="8.062726989147962e-06"/>
-    </inertial>
+        </inertial>
     </link>
     <joint name="driver_joint" type="fixed">
@@ -134,96 +135,97 @@
     </joint>
     <xacro:if value="${gazebo}">
-        <gazebo reference="driver">
-            <mu1>1.0</mu1>
-            <mu2>1.0</mu2>
-        </gazebo>
-    </xacro:if>
-    <!-- ........................ Regulator Support ......................... -->
-    <link name="reg_support">
-    <visual>
-        <origin xyz="0 0 0" rpy="0 0 ${-pi_2}"/>
-        <geometry>
-        <mesh filename="package://orion_description/meshes/regulator_sup.stl"
-            scale="0.001 0.001 0.001"/>
-        </geometry>
-        <material name="PLAWhite"/>
-    </visual>
-    <collision>
-        <origin xyz="0 0 0" rpy="0 0 ${-pi_2}"/>
-        <geometry>
-        <mesh filename="package://orion_description/meshes/regulator_sup.stl"
-            scale="0.001 0.001 0.001"/>
-        </geometry>
-    </collision>
-    <inertial>
-        <origin xyz="0 0 0" rpy="0 0 ${-pi_2}"/>
-        <mass value="0.010"/>
-        <inertia ixx="2.0760416666666664e-06" ixy="0.0" ixz="0.0"
+            <gazebo reference="driver">
+                <mu1>1.0</mu1>
+                <mu2>1.0</mu2>
+            </gazebo>
+        </xacro:if>
+        <!-- ........................ Regulator Support ......................... -->
+        <link name="reg_support">
+            <visual>
+                <origin xyz="0 0 0" rpy="0 0 ${-pi_2}"/>
+                <geometry>
+                    <mesh filename="package://orion_description/meshes/regulator_sup.stl"
+                    scale="0.001 0.001 0.001"/>
+                </geometry>
+                <material name="PLAWhite"/>
+            </visual>
+            <collision>
+                <origin xyz="0 0 0" rpy="0 0 ${-pi_2}"/>
+                <geometry>
+                    <mesh filename="package://orion_description/meshes/regulator_sup.stl"
+                    scale="0.001 0.001 0.001"/>
+                </geometry>
+            </collision>
+            <inertial>
+                <origin xyz="0 0 0" rpy="0 0 ${-pi_2}"/>
+                <mass value="0.010"/>
+                <inertia ixx="2.0760416666666664e-06" ixy="0.0" ixz="0.0"
                 iyy="5.797708333333332e-06" iyz="0.0"
                 izz="3.872083333333333e-06"/>
-    </inertial>
-    </link>
-    <joint name="reg_support_joint" type="fixed">
-        <parent link="base_l0_s2"/>
-        <child link="reg_support"/>
-        <origin xyz="-0.026 -0.0275 0.0025" rpy="0 0 0"/>
-    </joint>
-    <xacro:if value="${gazebo}">
-        <gazebo reference="reg_support">
-            <mu1>1.0</mu1>
-            <mu2>1.0</mu2>
-        </gazebo>
-    </xacro:if>
-    <!-- ....................... Regulator ............................... -->
-    <link name="regulator">
-    <visual>
-        <origin xyz="0 0 0" rpy="${pi_2} 0 ${-pi_2}"/>
-        <geometry>
-        <mesh filename="package://orion_description/meshes/regulator.stl"
-            scale="0.001 0.001 0.001"/>
-        </geometry>
-        <material name="ArduinoBlue"/>
-    </visual>
-    <collision>
-        <origin xyz="0 0 0" rpy="${pi_2} 0 ${-pi_2}"/>
-        <geometry>
-        <mesh filename="package://orion_description/meshes/regulator.stl"
-            scale="0.001 0.001 0.001"/>
-        </geometry>
-    </collision>
-    <inertial>
-        <origin xyz="0 0 0" rpy="${pi_2} 0 ${-pi_2}"/>
-        <mass value="0.025"/>
-        <inertia ixx="3.4813802083333333e-06" ixy="0.0" ixz="0.0"
+            </inertial>
+        </link>
+        <joint name="reg_support_joint" type="fixed">
+            <parent link="base_l0_s2"/>
+            <child link="reg_support"/>
+            <origin xyz="-0.026 -0.0275 0.0025" rpy="0 0 0"/>
+        </joint>
+        <xacro:if value="${gazebo}">
+            <gazebo reference="reg_support">
+                <mu1>1.0</mu1>
+                <mu2>1.0</mu2>
+            </gazebo>
+        </xacro:if>
+        <!-- ....................... Regulator ............................... -->
+        <link name="regulator">
+            <visual>
+                <origin xyz="0 0 0" rpy="${pi_2} 0 ${-pi_2}"/>
+                <geometry>
+                    <mesh filename="package://orion_description/meshes/regulator.stl"
+                    scale="0.001 0.001 0.001"/>
+                </geometry>
+                <material name="ArduinoBlue"/>
+            </visual>
+            <collision>
+                <origin xyz="0 0 0" rpy="${pi_2} 0 ${-pi_2}"/>
+                <geometry>
+                    <mesh filename="package://orion_description/meshes/regulator.stl"
+                    scale="0.001 0.001 0.001"/>
+                </geometry>
+            </collision>
+            <inertial>
+                <origin xyz="0 0 0" rpy="${pi_2} 0 ${-pi_2}"/>
+                <mass value="0.025"/>
+                <inertia ixx="3.4813802083333333e-06" ixy="0.0" ixz="0.0"
                 iyy="9.114713541666667e-06" iyz="0.0"
                 izz="1.1970833333333332e-05"/>
-    </inertial>
-    </link>
-    <joint name="reg_joint" type="fixed">
-        <parent link="reg_support"/>
-        <child link="regulator"/>
-        <origin xyz="-0.0025 0 ${0.06/2}" rpy="0 0 0"/>
-    </joint>
-    <xacro:if value="${gazebo}">
-        <gazebo reference="regulator">
-            <mu1>1.0</mu1>
-            <mu2>1.0</mu2>
-        </gazebo>
-    </xacro:if>
-    <!-- ......................... Switch ........................... -->
+            </inertial>
+        </link>
+        <joint name="reg_joint" type="fixed">
+            <parent link="reg_support"/>
+            <child link="regulator"/>
+            <origin xyz="-0.0025 0 ${0.06/2}" rpy="0 0 0"/>
+        </joint>
+        <xacro:if value="${gazebo}">
+            <gazebo reference="regulator">
+                <mu1>1.0</mu1>
+                <mu2>1.0</mu2>
+            </gazebo>
+        </xacro:if>
+    </xacro:unless>
+        <!-- ......................... Switch ........................... -->
     <link name="switch">
-    <visual>
-        <origin xyz="0 0 0" rpy="${pi_2} 0 ${pi_2}"/>
-        <geometry>
-        <mesh filename="package://orion_description/meshes/switch_3s_15a.stl"
-            scale="0.001 0.001 0.001"/>
-        </geometry>
-        <material name="ArduinoBlue"/>
-    </visual>
+        <visual>
+            <origin xyz="0 0 0" rpy="${pi_2} 0 ${pi_2}"/>
+            <geometry>
+                <mesh filename="package://orion_description/meshes/switch_3s_15a.stl"
+                scale="0.001 0.001 0.001"/>
+            </geometry>
+            <material name="ArduinoBlue"/>
+        </visual>
     <collision>
-        <origin xyz="0 0 0" rpy="${pi_2} 0 ${pi_2}"/>
-        <geometry>
-        <mesh filename="package://orion_description/meshes/switch_3s_15a.stl"
-            scale="0.001 0.001 0.001"/>
+    <origin xyz="0 0 0" rpy="${pi_2} 0 ${pi_2}"/>
+    <geometry>
+    <mesh filename="package://orion_description/meshes/switch_3s_15a.stl"
+        scale="0.001 0.001 0.001"/>
         </geometry>
     </collision>
@@ -259,79 +261,81 @@
         x="${0.115/2}" z="${0.082/2 + 0.0025/2}" level="0"/>
     <!-- ///////////////// SECOND FLOOR COMPONENTS /////////////////////// -->
-    <!-- ..................... Spacers for esp32 adp ..................... -->
-    <xacro:x4xmetric_spacer id="m3x10" element="esp_adapter" parent="base_l1_s2"
+    <xacro:unless value="${simplified}">
+        <!-- ..................... Spacers for esp32 adp ..................... -->
+        <xacro:x4xmetric_spacer id="m3x10" element="esp_adapter" parent="base_l1_s2"
         offset_x="${0.0577/2}" offset_y="${0.0607/2}" x="0.004" y="0" z="-0.01"/>
-    <!-- .......................... Esp32 Adapter ....................... -->
-    <link name="esp32_adapter">
-    <visual>
-        <origin xyz="0 0 0" rpy="${pi} 0 0"/>
-        <geometry>
-        <mesh filename="package://orion_description/meshes/esp32_adp.stl"
-            scale="0.001 0.001 0.001"/>
-        </geometry>
-        <material name="RaspberryGreen"/>
-    </visual>
-    <collision>
-        <origin xyz="0 0 0" rpy="${pi} 0 0"/>
-        <geometry>
-        <mesh filename="package://orion_description/meshes/esp32_adp.stl"
-            scale="0.001 0.001 0.001"/>
-        </geometry>
-    </collision>
-    <inertial>
-        <origin xyz="0 0 0" rpy="${pi} 0 0"/>
-        <mass value="0.030"/>
-        <inertia ixx="1.1184306270694732e-05" ixy="0.0" ixz="0.0"
+        <!-- .......................... Esp32 Adapter ....................... -->
+        <link name="esp32_adapter">
+            <visual>
+                <origin xyz="0 0 0" rpy="${pi} 0 0"/>
+                <geometry>
+                    <mesh filename="package://orion_description/meshes/esp32_adp.stl"
+                    scale="0.001 0.001 0.001"/>
+                </geometry>
+                <material name="RaspberryGreen"/>
+            </visual>
+            <collision>
+                <origin xyz="0 0 0" rpy="${pi} 0 0"/>
+                <geometry>
+                    <mesh filename="package://orion_description/meshes/esp32_adp.stl"
+                    scale="0.001 0.001 0.001"/>
+                </geometry>
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
File: orion_description/urdf/orion.urdf.xacro (robot description, xacro)
@@ -7,4 +7,5 @@
     <xacro:property name="gazebo" default="$(arg gazebo)"/>
     <xacro:property name="ros2_control" default="$(arg ros2_control)"/>
+    <xacro:property name="simplified" default="$(arg simplified)"/>
     <!-- For colors consider mdf, transparent or pla -->
     <xacro:property name="color" default="mdf"/>
