Commit message: Assets: Added new regulator and microphone | Description: Adapted URDF to meshses changes and added choices to the launch files

File: orion_description/urdf/include/orion_base.urdf.xacro (robot description, xacro)
@@ -100,4 +100,56 @@
         <xacro:stack_bat parent="bat_platform" num="2" x="0" y="${0.023+0.02}"
             z="0.0025"/>
+        <!-- ........................ Additional spacers ........................-->
+        <xacro:x6xmetric_spacer id="m3x20" element="bathol_2" parent="base_l0_s1"
+            offset_x="${0.0855/2}" offset_y="${0.127/2}" x="0.005" y="0"
+            z="0.0175"/>
+        <!-- ..................... Battery Platform ....................... -->
+        <link name="bat_platform_2">
+        <visual>
+            <origin xyz="0 0 0" rpy="0 0 ${pi_2}"/>
+            <geometry>
+            <mesh filename="package://orion_description/meshes/bathold_support.stl"
+                scale="0.001 0.001 0.001"/>
+            </geometry>
+            <xacro:if value="${color == 'mdf'}">
+                    <material name="MDF"/>
+                </xacro:if>
+                <xacro:if value="${color == 'transparent'}">
+                    <material name="TransparentBlack"/>
+                </xacro:if>
+                <xacro:if value="${color == 'pla'}">
+                    <material name="PLAWhite"/>
+                </xacro:if>
+        </visual>
+        <collision>
+            <origin xyz="0 0 0" rpy="0 0 ${pi_2}"/>
+            <geometry>
+            <mesh filename="package://orion_description/meshes/bathold_support.stl"
+                scale="0.001 0.001 0.001"/>
+            </geometry>
+        </collision>
+        <inertial>
+            <origin xyz="0 0 0" rpy="0 0 ${pi_2}"/>
+            <mass value="0.018"/>
+            <inertia ixx="1.2564374999999998e-05" ixy="0.0" ixz="0.0"
+                    iyy="2.6539499999999996e-05" iyz="0.0"
+                    izz="3.9091874999999996e-05"/>
+        </inertial>
+        </link>
+        <joint name="bat_platform_2_joint" type="fixed">
+            <parent link="base_l0_s1"/>
+            <child link="bat_platform_2"/>
+            <origin xyz="0.005 0 0.0375" rpy="0 0 0"/>
+        </joint>
+        <xacro:if value="${gazebo}">
+            <gazebo reference="bat_platform_2">
+                <mu1>1.0</mu1>
+                <mu2>1.0</mu2>
+            </gazebo>
+        </xacro:if>
+        <!-- ....................... Battery Stacks ........................ -->
+        <xacro:stack_bat parent="bat_platform_2" num="3" x="0" y="-0.023" z="0.0025"/>
+        <xacro:stack_bat parent="bat_platform_2" num="4" x="0" y="${0.023+0.02}"
+            z="0.0025"/>
         <!-- ............... Hex spacers for Motor Driver................... -->
         <xacro:x4xmetric_spacer id="m3x10" element="driver" parent="base_l0_s2"
@@ -181,5 +233,5 @@
                 <origin xyz="0 0 0" rpy="${pi_2} 0 ${-pi_2}"/>
                 <geometry>
-                    <mesh filename="package://orion_description/meshes/regulator.stl"
+                    <mesh filename="package://orion_description/meshes/regulator_2.stl"
                     scale="0.001 0.001 0.001"/>
                 </geometry>
@@ -189,5 +241,5 @@
                 <origin xyz="0 0 0" rpy="${pi_2} 0 ${-pi_2}"/>
                 <geometry>
-                    <mesh filename="package://orion_description/meshes/regulator.stl"
+                    <mesh filename="package://orion_description/meshes/regulator_2.stl"
                     scale="0.001 0.001 0.001"/>
                 </geometry>
@@ -204,5 +256,5 @@
             <parent link="reg_support"/>
             <child link="regulator"/>
-            <origin xyz="-0.0025 0 ${0.06/2}" rpy="0 0 0"/>
+            <origin xyz="-0.0025 0 ${0.06/2 -0.0025}" rpy="0 0 0"/>
         </joint>
         <xacro:if value="${gazebo}">
@@ -538,4 +590,40 @@
         <xacro:if value="${gazebo}">
             <gazebo reference="${rasp}">
+                <mu1>1.0</mu1>
+                <mu2>1.0</mu2>
+            </gazebo>
+        </xacro:if>
+        <!-- .......................... Microphone .................................. -->
+        <link name="microphone">
+            <visual>
+                <origin xyz="0 0 0" rpy="0 0 ${pi}"/>
+                <geometry>
+                    <mesh filename="package://orion_description/meshes/microphone.stl"
+                    scale="0.001 0.001 0.001"/>
+                </geometry>
+                <material name="SoftBlack"/>
+            </visual>
+            <collision>
+                <origin xyz="0 0 0" rpy="0 0 ${pi}"/>
+                <geometry>
+                    <mesh filename="package://orion_description/meshes/microphone.stl"
+                    scale="0.001 0.001 0.001"/>
+                </geometry>
+            </collision>
+            <inertial>
+                <origin xyz="0 0 0" rpy="0 0 ${pi}"/>
+                <mass value="0.020"/>
+                <inertia ixx="1.0875937499999998e-05" ixy="0.0" ixz="0.0"
+                iyy="1.6950937499999996e-05" iyz="0.0"
+                izz="7.154999999999999e-06"/>
+            </inertial>
+        </link>
+        <joint name="microphone_joint" type="fixed">
+            <parent link="base_l3_s1"/>
+            <child link="microphone"/>
+            <origin xyz="-0.0275 0.0 0.06" rpy="0 0 0"/>
+        </joint>
+        <xacro:if value="${gazebo}">
+            <gazebo reference="microphone">
                 <mu1>1.0</mu1>
                 <mu2>1.0</mu2>

File: orion_description/urdf/include/orion_macros.urdf.xacro (robot description, xacro)
@@ -849,4 +849,10 @@
                         iyy="8.960721799390997e-09" iyz="0"
                         izz="4.443388969597693e-09"/>
+            </xacro:if>
+            <xacro:if value="${id == 'm3x20'}">
+                <mass value="0.0024"/>
+                <inertia ixx="8.5251996963501e-08" ixy="0" ixz="0"
+                        iyy="8.648216387229408e-08" iyz="0"
+                        izz="1.333016690879308e-08"/>
             </xacro:if>
         </inertial>

Commit message: Description: Fixing tf issues related with odometry

File: orion_description/urdf/include/orion_base.urdf.xacro (robot description, xacro)
@@ -4,17 +4,24 @@
     <!-- ////////////////////////// BASE LINK //////////////////////////////-->
     <link name="base_link"/>
+    <!-- .................... Middle frame ......................... -->
+    <link name="middle_base"/>
+    <joint name="to_footprint" type="fixed">
+        <origin xyz="-0.05 0.0 0.0" rpy="0.0 0.0 0.0"/>
+        <parent link="base_link"/>
+        <child link="middle_base"/>
+    </joint>
     <!-- ///////////////////////// PROPERTIES //////////////////////////////-->
     <xacro:property name="level_height" value="0.08"/>
     <xacro:property name="thickness" value="0.0025"/>
     <!-- /////////////////////////// LEVELS ///////////////////////////////-->
-    <xacro:com_base level="0" parent="base_link" x="0" y="0"
+    <xacro:com_base level="0" parent="middle_base" x="0" y="0"
         z="${level_height*0+ thickness*0}"/>
-    <xacro:com_base level="1" parent="base_link" x="0" y="0"
+    <xacro:com_base level="1" parent="middle_base" x="0" y="0"
         z="${level_height*1 + thickness*1}"/>
-    <xacro:com_base level="2" parent="base_link" x="0" y="0"
+    <xacro:com_base level="2" parent="middle_base" x="0" y="0"
         z="${level_height*2 + thickness*2}"/>
-    <xacro:com_base level="3" parent="base_link" x="0" y="0"
+    <xacro:com_base level="3" parent="middle_base" x="0" y="0"
         z="${level_height*3 + thickness*3}"/>
-    <xacro:half_base level="4" side="2" parent="base_link" x="0" y="0"
+    <xacro:half_base level="4" side="2" parent="middle_base" x="0" y="0"
         z="${level_height*4 + thickness*4}"/>
     <!-- /////////////////////// LEVEL's SPACERS//////////////////////////-->

File: orion_description/urdf/include/orion_macros.urdf.xacro (robot description, xacro)
@@ -123,7 +123,7 @@
     <!-- ...................... Complete base ............................ -->
     <xacro:macro name="com_base" params="level parent x y z">
-        <xacro:half_base level="${level}" side="1" parent="base_link" x="${x}"
+        <xacro:half_base level="${level}" side="1" parent="middle_base" x="${x}"
             y="${y}" z="${z}"/>
-        <xacro:half_base level="${level}" side="2" parent="base_link" x="${x}"
+        <xacro:half_base level="${level}" side="2" parent="middle_base" x="${x}"
             y="${y}" z="${z}"/>
     </xacro:macro>
@@ -293,6 +293,7 @@
             <origin xyz="0 0 0" rpy="0 ${pi_2*muls} 0"/>
             <geometry>
-            <mesh filename="package://orion_description/meshes/neumatic.stl"
-                scale="0.001 0.001 0.001"/>
+            <sphere radius="0.033675"/>
+            <!--mesh filename="package://orion_description/meshes/neumatic.stl"
+                scale="0.001 0.001 0.001"/-->
             </geometry>
         </collision>
@@ -312,5 +313,5 @@
         <gazebo reference="neumatic_${front}${side}">
             <mu1>1.0</mu1>
-            <mu2>1.0</mu2>
+            <mu2>0.8</mu2>
         </gazebo>
     </xacro:macro>
@@ -375,5 +376,5 @@
         <inertial>
             <origin xyz="0 0 0" rpy="0 0 ${-pi_2}"/>
-            <mass value="0.01633"/>
+            <mass value="0.001"/>
             <inertia ixx="1.6321007868011535e-06" ixy="0.0" ixz="0.0"
                     iyy="1.3901075509910613e-06" iyz="0.0"
@@ -386,8 +387,11 @@
             <child link="caster_middle_${front}"/>
             <origin xyz="0 0 -0.002" rpy="${pi} 0 0"/>
+            <dynamics damping="0.05" friction="0.0"/>
         </joint>
         <gazebo reference="caster_middle_${front}">
-            <mu1>1.0</mu1>
-            <mu2>1.0</mu2>
+            <mu1>0.01</mu1>
+            <mu2>0.01</mu2>
+            <kp>100000.0</kp>
+            <kd>10.0</kd>
         </gazebo>
         <!-- Caster wheel definition-->
@@ -410,5 +414,5 @@
         <inertial>
             <origin xyz="0 0 0" rpy="${pi_2} 0 0"/>
-            <mass value="0.00794"/>
+            <mass value="0.001"/>
             <inertia ixx="5.723473258925721e-07" ixy="0.0" ixz="0.0"
                     iyy="8.268436933141506e-07" iyz="0.0"
@@ -421,8 +425,11 @@
             <child link="caster_wheel_${front}"/>
             <origin xyz="-0.0108 0 0.0185" rpy="${pi_2} 0 0"/>
+            <dynamics damping="0.05" friction="0.0"/>
         </joint>
         <gazebo reference="caster_wheel_${front}">
-            <mu1>0.001</mu1>
-            <mu2>0.001</mu2>
+            <mu1>0.01</mu1>
+            <mu2>0.01</mu2>
+            <kp>100000.0</kp>
+            <kd>10.0</kd>
         </gazebo>
     </xacro:macro>

Commit message: Description: Fix, change footprint name to base_link

File: orion_description/urdf/include/orion_base.urdf.xacro (robot description, xacro)
@@ -6,5 +6,5 @@
     <!-- .................... Middle frame ......................... -->
     <link name="middle_base"/>
-    <joint name="to_footprint" type="fixed">
+    <joint name="to_middle_base" type="fixed">
         <origin xyz="-0.05 0.0 0.0" rpy="0.0 0.0 0.0"/>
         <parent link="base_link"/>
