Commit message: Description: Added motors limits | Control: Fixing mobile base params

File: orion_description/urdf/include/orion_macros.urdf.xacro (robot description, xacro)
@@ -239,4 +239,5 @@
             <parent link="motor_support_${front}${side}"/>
             <child link="coupling_${front}${side}"/>
+            <limit effort="0.40964" velocity="104.97"/>
             <origin xyz="0 ${(0.01120 + 0.000325)*muls} 0" rpy="${-pi_2*muls+orin} 0 0"/>
         </joint>
@@ -625,5 +626,5 @@
             <child link="servo_conn_${side}"/>
             <origin xyz="0.01 ${0.0406*inv} 0" rpy="${-pi_2*inv} 0 0"/>
-            <limit lower="${-pi_2}" upper="${pi_2}" effort="0.92" velocity="6.0"/>
+            <limit lower="${-pi_2}" upper="${pi_2}" effort="1.08" velocity="5.24"/>
             <dynamics damping="0.05" friction="0.002"/>
         </joint>

File: orion_description/urdf/include/orion_ros2_control.urdf.xacro (robot description, xacro)
@@ -8,5 +8,5 @@
                     <param name="left_wheel_name">coupling_11_joint</param>
                     <param name="right_wheel_name">coupling_12_joint</param>
-                    <param name="enc_ticks_per_rev">220</param>
+                    <param name="enc_ticks_per_rev">204</param>
                 </hardware>
                 <joint name="coupling_11_joint">

Commit message: Description: Added change of joint when using real robot for caster | Base: Updating servo mangement and limits

File: orion_description/urdf/include/orion_macros.urdf.xacro (robot description, xacro)
@@ -316,6 +316,8 @@
     </xacro:macro>
     <!--////////////////////////// CASTER WHEEL ////////////////////////////-->
-    <!--xacro:property name="caster_type" value="continuous"/-->
-    <xacro:property name="caster_type" value="continuous"/>
+    <xacro:property name="caster_type" value="fixed"/>
+    <xacro:if value="${gazebo}">
+        <xacro:property name="caster_type" value="continuous"/>
+    </xacro:if>
     <!-- ......................... Macro for caster ....................... -->
     <xacro:macro name="caster_wheel" params="parent front x y z">
@@ -626,5 +628,5 @@
             <child link="servo_conn_${side}"/>
             <origin xyz="0.01 ${0.0406*inv} 0" rpy="${-pi_2*inv} 0 0"/>
-            <limit lower="${-pi_2}" upper="${pi_2}" effort="1.08" velocity="5.24"/>
+            <limit lower="${-pi/3}" upper="${pi/3}" effort="1.08" velocity="5.24"/>
             <dynamics damping="0.05" friction="0.002"/>
         </joint>

Commit message: Description: Allowing change of motor and updating args

File: orion_description/urdf/include/orion_macros.urdf.xacro (robot description, xacro)
@@ -239,5 +239,10 @@
             <parent link="motor_support_${front}${side}"/>
             <child link="coupling_${front}${side}"/>
-            <limit effort="0.40964" velocity="104.97"/>
+            <xacro:if value="${motor == 1000}">
+                <limit effort="0.01079" velocity="104.97"/>
+            </xacro:if>
+            <xacro:if value="${motor == 100}">
+                <limit effort="0.08336" velocity="10.47"/>
+            </xacro:if>
             <origin xyz="0 ${(0.01120 + 0.000325)*muls} 0" rpy="${-pi_2*muls+orin} 0 0"/>
         </joint>

File: orion_description/urdf/include/orion_ros2_control.urdf.xacro (robot description, xacro)
@@ -1,5 +1,4 @@
 <?xml version="1.0"?>
 <robot xmlns:xacro="http://www.ros.org/wiki/xacro">
-    <xacro:property name="motor" value="100"/>
     <xacro:if value="${ros2_control}">
         <xacro:if value="${ctl_type == 'micro_ros'}">

File: orion_description/urdf/orion.urdf.xacro (robot description, xacro)
@@ -8,4 +8,5 @@
     <xacro:property name="ros2_control" default="$(arg ros2_control)"/>
     <xacro:property name="simplified" default="$(arg simplified)"/>
+    <xacro:property name="motor" value="$(arg motor)"/>
     <xacro:property name="ctl_type" default="micro_ros"/>
     <!-- For colors consider mdf, transparent or pla -->
